File: Electrocity_Manager/Electrocity_Manager.kicad_pcb (KiCad board)
At the start: 2 copper layers, 100 x 77 mm, 197 parts, among them IC2 MAIN_SHUTDOWN, IC3 RELAY_STATE, IC4 ADC_RST, J1 SERIAL, P1 SWD, P10 EMERGENCY, P11 EMERGENCY, P12 FRAME_GRAND, P13 BATT_IN, P14 OUT_A, P15 OUT_B, P16 BATT_IN, P17 OUT_A, P18 OUT_B, P2 CAN, P3 CAN, P4 EMERGENCY_SIGNAL, P5 EMERGENCY_SIGNAL, P6 12V_OUT, P7 12V_OUT, P9 MAIN_SW, Q1 FET_N, Q2 NPN, Q3 NPN, Q7 FET_N, SW1 RST, SW2 SW0, SW3 SW1, U1 MAX3051, U10 BD9G101G, U11 ACS781, U11 OUTA_CHECK, U12 V23134J1052D642, U13 ACS70331, U14 ACS781, U14 OUTA_CHECK, U15 BD33FA1, U16 LOGO, U17 LOGO, U18 LOGO, U19 MCP2221A, U2 STM32F405RG, U20 OSRB38C9AA, U21 OSRB38C9AA, U22 HSIN_946, U23 LOGO, U24 LOGO, U25 LOGO, U26 LOGO, U3 FULL COLOR, U4 AQM0802_BL, U5 AP3211, U6 SI8900, U7 AZ1086H, U8 V23134J1052D642, U9 RPA60-12FW/N, X1 8MHz

Commit message: mainと電源が仮完成.
Parts:
- removed C39: 1u, Mizz_lib:C_0603
- removed C40: 0.1u, Mizz_lib:C_0603
- removed P14: OUT_A, RP_KiCAD_Connector:XT60_F
- removed P18: OUT_B, RP_KiCAD_Connector:XT60_M
- removed the R40 at (111.0, 128.0)
- removed the R44 at (111.0, 126.2)
- removed R9: 4.7k, Mizz_lib:R_0603
- removed the U11 at (73.2, 113.2)
- removed the U14 at (98.8, 113.2)
- removed the U14 at (105.5, 93.2)
- removed U26: LOGO, Mizz_lib:PiOtyu_silk_21.3x6.8
- added AMP1: TSC103, Package_SO:SO-8_3.9x4.9mm_P1.27mm, F.Cu at (74.0, 110.2)
- added AMP2: TSC103, Package_SO:SO-8_3.9x4.9mm_P1.27mm, F.Cu at (97.2, 110.2)
- added Q4: FET_N, Mizz_lib:SOT-23, B.Cu at (133.8, 156.8)
- added R54: 10k, Mizz_lib:R_0603, B.Cu at (134.5, 154.2)
- added R55: 2m, Mizz_lib:WSHP2818, B.Cu at (64.8, 112.5)
- added R56: 2m, Mizz_lib:WSHP2818, B.Cu at (70.0, 112.5)
- added R57: 2m, Mizz_lib:WSHP2818, B.Cu at (87.8, 112.5)
- added R60: 2m, Mizz_lib:WSHP2818, B.Cu at (93.2, 112.5)
- added U14: OUTB_CHECK, Package_SO:SOIC-4_4.55x2.6mm_P1.27mm, F.Cu at (108.0, 126.2)
- C33: value 1u -> 0.1u; moved to F.Cu
- D19: value +12P -> +8V5P
- D20: value +3.3P -> +3V3P
- Q2, Q3: footprint Mizz_lib:SOT-123 -> Package_TO_SOT_SMD:SOT-23W
- R40, R44, R49, R50: moved to B.Cu
- U24: footprint Mizz_lib:Pikatyuu_15x15 -> Mizz_lib:Dodaitos_15x15_silk
- moved C33 49.1 mm to (72.5, 106.8)
- moved R44 43.9 mm to (103.8, 134.0)
- moved R40 42.5 mm to (111.7, 130.8), turned to 270 degrees
- moved U11 42.3 mm to (108.0, 131.2)
- moved R49 39.7 mm to (111.8, 127.8), turned to 90 degrees
- moved R50 36.4 mm to (103.8, 129.0)
- moved C34 8.49 mm to (95.8, 106.8), turned to 0 degrees
- moved P15 7.50 mm to (82.8, 106.0)
- moved D17 7.25 mm to (90.0, 106.0)
- moved R36 7.25 mm to (90.0, 108.0)
- moved D16 6.75 mm to (67.0, 106.0)
- moved P17 6.75 mm to (60.0, 106.0)
- moved R35 6.75 mm to (67.0, 108.2)
- moved U25 1.35 mm to (83.0, 170.5)
- moved U24 0.50 mm to (93.5, 164.0)
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Connections:
- net /PB2 renamed Net-(U2-Pad28)
- C30 pad 2: +12C -> +8V
- C33 pad 1: /ADC12_IN1 -> 3V3
- C33 pad 2: GND -> GNDPWR
- C34 pad 1: +3.3V -> 3V3
- C34 pad 2: GND -> GNDPWR
- C37 pad 2: +12C -> +8V
- C46 pad 1: +12C -> +8V
- IC2 pad 4: Net-(IC2-Pad4) -> +8V
- L2 pad 2: +12C -> +8V
- P10 pad 1: +12C -> +8V
- R38 pad 2: +12C -> +8V
- R40 pad 2: Net-(R40-Pad2) -> /PA1
- R41 pad 1: +12C -> +8V
- R49 pad 2: Net-(R49-Pad2) -> /PA0
- U11 pad 3: Net-(R40-Pad2) -> /PA1
- U11 pad 4: Net-(U11-Pad4) -> +3.3V
- U12 pad 87: Net-(U12-Pad87) -> /To_CurrentB
- U15 pad 3: +12C -> +8V
- U2 pad 14: /ADC12_IN2 -> /PA0
- U2 pad 15: /ADC12_IN1 -> /PA1
- U2 pad 50: Net-(U2-Pad50) -> /CoilReadPin_PA15
- U22 pad 1: Net-(U22-Pad1) -> Net-(P11-Pad2)
- U6 pad 3: /OUTB_Current -> /OUTA_Current
- U6 pad 4: /OUTA_Current -> /OUTB_Current
- U8 pad 87: Net-(U8-Pad87) -> /To_CurrentA
Routing:
- net +8V: track 0.00 -> 98.0 mm, vias 0 -> 5
- net +12C: track 78.2 -> 0.00 mm, vias 3 -> 0
- net /OUTA_Current: track 0.00 -> 61.2 mm, vias 0 -> 2
- net 3V3: track 54.2 -> 107.3 mm, vias 4 -> 5
- net OUT_A: track 7.19 -> 57.0 mm, vias 0 -> 1
- net Net-(R40-Pad2): track 43.6 -> 0.00 mm, vias 1 -> 0
- net /OUTB_Current: track 0.00 -> 41.1 mm, vias 0 -> 2
- net +3.3V: track 277.6 -> 240.3 mm
- net GND: track 46.1 -> 11.1 mm, vias 114 -> 135
- net GNDPWR: track 9.14 -> 42.7 mm, vias 245 -> 288
- net OUT_B: track 7.30 -> 31.1 mm, vias 0 -> 2
- net /PA0: track 0.00 -> 22.1 mm, vias 0 -> 1
- net /ADC12_IN2: track 21.3 -> 0.00 mm, vias 1 -> 0
- net /ADC12_IN1: track 19.7 -> 0.00 mm, vias 2 -> 0
- net /PA1: track 0.00 -> 19.1 mm, vias 0 -> 1
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- added copper zone on B.Cu, net /To_CurrentA
- added copper zone on B.Cu, net /To_CurrentB
- removed copper zone on B.Cu, net Net-(U11-Pad5)
- removed copper zone on B.Cu, net Net-(U12-Pad87)
Other:
- board text added: "Designed by A.Mizuta in 2019/11/05."
- board text added: "Electrocity Manager ver.2.0"
- board text added: "Libra Zubenelgenubi"
- board text added: "Lithium polymer 3s-6s"
- board text added: "Pocket Monster "Dodaitos""
- board text added: "Range of use:"
- board text removed: "Designed by A.Mizuta in 2019/10/10."
- board text removed: "Electrocity Manager ver.2.0 for ROBO RUGBY 7s."
- board text removed: "Pocket Monster "Pikachu""
