File: Electrocity_Manager/Electrocity_Manager.sch (KiCad schematic (older format))
At the start: 187 parts, among them IC2 MAIN_SHUTDOWN, IC3 RELAY_STATE, IC4 ADC_RST, J1 SERIAL, P1 SWD, P10 EMERGENCY, P11 EMERGENCY, P12 FRAME_GRAND, P13 BATT_IN, P15 OUT_B, P16 BATT_IN, P17 OUT_A, P2 CAN, P3 CAN, P4 EMERGENCY_SIGNAL, P5 EMERGENCY_SIGNAL, P6 12V_OUT, P7 12V_OUT, P9 MAIN_SW, Q1 FET_N, Q2 NPN, Q3 NPN, Q7 FET_N, SW1 RST, SW2 SW0, SW3 SW1, U1 MAX3051, U10 BD9G101G, U11 OUTA_CHECK, U12 V23134J1052D642, U13 ACS70331, U14 OUTA_CHECK, U15 BD33FA1, U16 LOGO, U17 LOGO, U18 LOGO, U19 MCP2221A, U2 STM32F405RG, U20 OSRB38C9AA, U21 OSRB38C9AA, U22 HSIN_946, U23 LOGO, U24 LOGO, U25 LOGO, U26 LOGO, U3 FULL COLOR, U4 AQM0802_BL, U5 AP3211, U6 SI8900, U7 AZ1086H, U8 V23134J1052D642, U9 RPA60-12FW/N, X1 8MHz

Commit message: mainと電源が仮完成.
Parts:
- removed R9: 4.7k, Mizz_lib:R_0603, symbol Electrocity_Manager-rescue:R-device
- removed U26: LOGO, Mizz_lib:PiOtyu_silk_21.3x6.8, symbol Electrocity_Manager-rescue:LOGO-myDevice-Electrocity_Manager-rescue
- added AMP1, AMP2: TSC103, Package_SO:SO-8_3.9x4.9mm_P1.27mm, symbol Miz:TSC103
- added C33, C34: 0.1u, Mizz_lib:C_0603, symbol Electrocity_Manager-rescue:C-device
- added Q4: FET_N, Mizz_lib:SOT-23, symbol Electrocity_Manager-rescue:MOSFET_N_123-Hori_lib-Electrocity_Manager-rescue
- added R54: 10k, Mizz_lib:R_0603, symbol Electrocity_Manager-rescue:R-device
- added R55, R56, R57, R60: 2m, Mizz_lib:WSHP2818, symbol Device:R
- D19: value +12P -> +8V5P
- D20: value +3.3P -> +3V3P
- Q2, Q3: footprint Mizz_lib:SOT-123 -> Package_TO_SOT_SMD:SOT-23W
- U14: value OUTA_CHECK -> OUTB_CHECK
- U24: footprint Mizz_lib:Pikatyuu_15x15 -> Mizz_lib:Dodaitos_15x15_silk
Connections:
- net +12C is gone; now on net +8V: C30.2, C37.2, C46.1, L2.2, P10.1 (P1), R38.2, R41.1, U15.3 (Vcc)
- net ADC12_IN1 is gone; now on net PA1: U2.15 (UART4_RX/ADC12_IN1/TIM5_CH2/TIM2_CH2/PA1)
- net ADC12_IN2 is gone; now on net PA0: U2.14 (UART4_TX/TIM2_CH1_ETR/ADC12_IN0/TIM5_CH1/PA0)
- net +3.3V: now also R54.2
- net 3V3: now also AMP1.5 (VCC), AMP2.5 (VCC), C33.1, C34.1
- net GND: now also Q4.2 (S)
- net GNDPWR: now also AMP1.2 (SEL1), AMP1.3 (SEL2), AMP1.6 (GND), AMP1.7 (VCC-), AMP2.2 (SEL1), AMP2.3 (SEL2), AMP2.6 (GND), AMP2.7 (VCC-), C33.2, C34.2
- net OUTA_Current: now also U6.3 (AIN0), AMP1.4 (Out); no longer U6.4 (AIN1)
- net OUTB_Current: now also U6.4 (AIN1), AMP2.4 (Out); no longer U6.3 (AIN0)
- net OUT_A: now also AMP1.1 (Vm), R55.2, R56.2; no longer U14.1
- net OUT_B: now also U14.1, AMP2.1 (Vm), R57.2, R60.2
- net Relay_state: now also Q4.1 (G)
- net CoilReadPin_PA15: now reaches U2.50 (TIM2_CH1_ETR/PA15)
- net CoilReadPin_PA15: now also Q4.3 (D), R54.1
- net To_CurrentA: now reaches U8.87
- net To_CurrentA: now also AMP1.8 (Vp), R55.1, R56.1
- net To_CurrentB: now reaches U12.87
- net To_CurrentB: now also AMP2.8 (Vp), R57.1, R60.1
- net +8V: now reaches IC2.4
- net PA1: now reaches R40.2, U11.3
- net PA0: now reaches R49.2, U14.3
- net PB2: no longer names the net of U2.28 (BOOT1/PB2)
Other:
- moved on the sheet: C19, C20, C21, D2, D22, D3, D4, Q3, R2, R26, R27, R28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
