File: F4_CAN_DCMD/CAN_DCMD.kicad_pcb (KiCad board)
At the start: 2 copper layers, 75 x 88 mm, 198 parts, among them P1 SWD, P10 OUT_1, P11 ENC_0, P13 ENC_1, P14 I/O_1, P15 OUT_0, P3 CAN, P4 CAN, P5 SERIAL, P6 I/O_0, P7 FAN, P8 BATT_IN, P9 BATT_IN, Q1 MOSFET_N, Q2 MOSFET_N, Q3 MOSFET_N, Q4 MOSFET_N, Q5 MOSFET_N, Q6 MOSFET_N, Q7 MOSFET_N, Q8 MOSFET_N, SW1 RST, SW3 SW0, SW4 SW1, U1 MAX3051, U10 ACS758, U11 POWER_ON, U12 SI8274, U13 ACS758, U14 SI8274, U15 AZ1086H, U16 LOGO, U19 ADRESS, U2 AP3211, U3 STM32F405RG, U4 SI8274, U5 SI8900, U6 ADC_~RST, U7 BD9G101G, U8 SI8274, U9 BD33FA1, Y1 8MHz

Commit message: MD関連
Parts:
- added C53: 0.1u, Capacitor_SMD:C_0603_1608Metric, F.Cu at (123.0, 44.8)
- added C54: 0.1u, Capacitor_SMD:C_0603_1608Metric, F.Cu at (127.0, 44.8)
- Q1, Q2, Q3, Q4, Q5, Q6, Q7, Q8: footprint Mizz_lib:HSOF-8-1 -> Mizz_lib:D2-PAK_compact
Connections:
- U3 pad 25: /LED3 -> Net-(U3-Pad25)
- U3 pad 26: /LED4 -> /LED3
- U3 pad 27: /SW0 -> /LED4
- U3 pad 29: /SW1 -> Net-(U3-Pad29)
- U3 pad 30: Net-(U3-Pad30) -> /SW1
- U3 pad 33: /MODE -> /SW0
Routing:
- net +3V3: track 44.6 -> 31.3 mm, vias 6 -> 4
- net /MOTOR0_BATT: track 4.09 -> 0.04 mm
- net GND: vias 76 -> 75
- removed copper zone on B.Cu, net /MOTOR0_BATT
- removed copper zone on B.Cu, net /MOTOR1_BATT
- removed copper zone on B.Cu, net /OUT0_L
- removed copper zone on B.Cu, net /OUT0_R
- removed copper zone on B.Cu, net /OUT1_L
- removed copper zone on B.Cu, net /OUT1_R
Other:
- board text added: "CAN DC-MotroDriver "Leo Regulus" ver.0.0"
- board text removed: "CAN DC-MotroDriver "Aqualius Sadalsuud" ver.0.0"
