File: F4_CAN_DCMD/CAN_DCMD.sch (KiCad schematic (older format))
At the start: 198 parts, among them P1 SWD, P10 OUT_1, P11 ENC_0, P13 ENC_1, P14 I/O_1, P15 OUT_0, P3 CAN, P4 CAN, P5 SERIAL, P6 I/O_0, P7 FAN, P8 BATT_IN, P9 BATT_IN, Q1 MOSFET_N, Q2 MOSFET_N, Q3 MOSFET_N, Q4 MOSFET_N, Q5 MOSFET_N, Q6 MOSFET_N, Q7 MOSFET_N, Q8 MOSFET_N, SW1 RST, SW3 SW0, SW4 SW1, U1 MAX3051, U10 ACS758, U11 POWER_ON, U12 SI8274, U13 ACS758, U14 SI8274, U15 AZ1086H, U16 LOGO, U19 ADRESS, U2 AP3211, U3 STM32F405RG, U4 SI8274, U5 SI8900, U6 ADC_~RST, U7 BD9G101G, U8 SI8274, U9 BD33FA1, Y1 8MHz

Commit message: MD関連
Parts:
- added C53, C54: 0.1u, Capacitor_SMD:C_0603_1608Metric, symbol CAN_DCMD-rescue:C-Device-MD_Enbarr_x2-rescue-F4_CAN_DCMD-rescue-SteerMD-rescue
- C1, C10, C11, C12, C13, C14, C15, C16, C17, C18, C19, C2, C20, C21, C22, C23, C24, C26, C27, C28, C29, C3, C30, C31, C32, C35, C36, C37, C38, C39, C4, C40, C41, C42, C43, C44, C45, C46, C47, C48, C49, C5, C50, C51, C52, C55, C56, C57, C6, C7, C8, C9: symbol SteerMD-rescue:C-Device-MD_Enbarr_x2-rescue-F4_CAN_DCMD-rescue -> CAN_DCMD-rescue:C-Device-MD_Enbarr_x2-rescue-F4_CAN_DCMD-rescue-SteerMD-rescue
- C25, C33, C34: symbol SteerMD-rescue:CP1-Device-MD_Enbarr_x2-rescue-F4_CAN_DCMD-rescue -> CAN_DCMD-rescue:CP1-Device-MD_Enbarr_x2-rescue-F4_CAN_DCMD-rescue-SteerMD-rescue
- D1, D11, D13, D14, D15, D16, D17, D18, D19, D2, D20, D24, D26, D3, D4, D47, D5: symbol SteerMD-rescue:DIODE-device-MD_Enbarr_x2-rescue-F4_CAN_DCMD-rescue -> CAN_DCMD-rescue:DIODE-device-MD_Enbarr_x2-rescue-F4_CAN_DCMD-rescue-SteerMD-rescue
- D21, D22, D23, D27, D32, D33, D34, D39, D7, D8, D9: symbol SteerMD-rescue:LED-Device-MD_Enbarr_x2-rescue-F4_CAN_DCMD-rescue -> CAN_DCMD-rescue:LED-Device-MD_Enbarr_x2-rescue-F4_CAN_DCMD-rescue-SteerMD-rescue
- JP1, JP2: symbol SteerMD-rescue:Jumper-Device-MD_Enbarr_x2-rescue-F4_CAN_DCMD-rescue -> CAN_DCMD-rescue:Jumper-Device-MD_Enbarr_x2-rescue-F4_CAN_DCMD-rescue-SteerMD-rescue
- L1, L2: symbol SteerMD-rescue:INDUCTOR-pspice-MD_Enbarr_x2-rescue-F4_CAN_DCMD-rescue -> CAN_DCMD-rescue:INDUCTOR-pspice-MD_Enbarr_x2-rescue-F4_CAN_DCMD-rescue-SteerMD-rescue
- P1: symbol SteerMD-rescue:CONN_01X06-conn-MD_Enbarr_x2-rescue-F4_CAN_DCMD-rescue -> CAN_DCMD-rescue:CONN_01X06-conn-MD_Enbarr_x2-rescue-F4_CAN_DCMD-rescue-SteerMD-rescue
- P10, P15, P7, P8, P9: symbol SteerMD-rescue:CONN_01X02-conn-MD_Enbarr_x2-rescue-F4_CAN_DCMD-rescue -> CAN_DCMD-rescue:CONN_01X02-conn-MD_Enbarr_x2-rescue-F4_CAN_DCMD-rescue-SteerMD-rescue
- P11, P13, P3, P4, P5: symbol SteerMD-rescue:CONN_01X04-conn-MD_Enbarr_x2-rescue-F4_CAN_DCMD-rescue -> CAN_DCMD-rescue:CONN_01X04-conn-MD_Enbarr_x2-rescue-F4_CAN_DCMD-rescue-SteerMD-rescue
- P14, P6: symbol SteerMD-rescue:CONN_01X03-conn-MD_Enbarr_x2-rescue-F4_CAN_DCMD-rescue -> CAN_DCMD-rescue:CONN_01X03-conn-MD_Enbarr_x2-rescue-F4_CAN_DCMD-rescue-SteerMD-rescue
- Q1, Q2, Q3, Q4, Q5, Q6, Q7, Q8: footprint Mizz_lib:HSOF-8-1 -> Mizz_lib:D2-PAK_compact; symbol SteerMD-rescue:MOSFET_N-Miz-F4_CAN_DCMD-rescue -> CAN_DCMD-rescue:MOSFET_N-Miz-F4_CAN_DCMD-rescue-SteerMD-rescue
- R1, R10, R11, R12, R13, R14, R15, R16, R17, R18, R19, R2, R20, R21, R22, R23, R24, R25, R26, R27, R28, R29, R3, R30, R31, R32, R33, R34, R35, R36, R37, R38, R39, R4, R40, R41, R42, R43, R44, R45, R46, R47, R48, R49, R5, R50, R51, R53, R54, R55, R56, R57, R58, R59, R6, R60, R61, R62, R63, R64, R65, R66, R67, R68, R7, R8, R9: symbol SteerMD-rescue:R-Device-MD_Enbarr_x2-rescue-F4_CAN_DCMD-rescue -> CAN_DCMD-rescue:R-Device-MD_Enbarr_x2-rescue-F4_CAN_DCMD-rescue-SteerMD-rescue
- SW1, SW3, SW4: symbol SteerMD-rescue:SW_PUSH-device-MD_Enbarr_x2-rescue-F4_CAN_DCMD-rescue -> CAN_DCMD-rescue:SW_PUSH-device-MD_Enbarr_x2-rescue-F4_CAN_DCMD-rescue-SteerMD-rescue
- U1: symbol SteerMD-rescue:MAX3051-Interface_UART-MD_Enbarr_x2-rescue-F4_CAN_DCMD-rescue -> CAN_DCMD-rescue:MAX3051-Interface_UART-MD_Enbarr_x2-rescue-F4_CAN_DCMD-rescue-SteerMD-rescue
- U11, U6: symbol SteerMD-rescue:TLP291-Isolator-MD_Enbarr_x2-rescue-F4_CAN_DCMD-rescue -> CAN_DCMD-rescue:TLP291-Isolator-MD_Enbarr_x2-rescue-F4_CAN_DCMD-rescue-SteerMD-rescue
- U12, U14, U4, U8: symbol SteerMD-rescue:SI8274-Miz-F4_CAN_DCMD-rescue -> CAN_DCMD-rescue:SI8274-Miz-F4_CAN_DCMD-rescue-SteerMD-rescue
- U15: symbol SteerMD-rescue:AZ1086H-myDevice-MD_Enbarr_x2-rescue-MD_Enbarr_x2-rescue-F4_CAN_DCMD-rescue -> CAN_DCMD-rescue:AZ1086H-myDevice-MD_Enbarr_x2-rescue-MD_Enbarr_x2-rescue-F4_CAN_DCMD-rescue-SteerMD-rescue
- U16: symbol SteerMD-rescue:LOGO-myDevice-MD_Enbarr_x2-rescue-F4_CAN_DCMD-rescue -> CAN_DCMD-rescue:LOGO-myDevice-MD_Enbarr_x2-rescue-F4_CAN_DCMD-rescue-SteerMD-rescue
- U19: symbol SteerMD-rescue:SW_ROTARY_16-Miz-F4_CAN_DCMD-rescue -> CAN_DCMD-rescue:SW_ROTARY_16-Miz-F4_CAN_DCMD-rescue-SteerMD-rescue
- U3: symbol SteerMD-rescue:STM32F405RG_excerpt-stm32f405rg_excerpt-Miz-MD_Enbarr_x2-rescue-F4_CAN_DCMD-rescue -> CAN_DCMD-rescue:STM32F405RG_excerpt-stm32f405rg_excerpt-Miz-MD_Enbarr_x2-rescue-F4_CAN_DCMD-rescue-SteerMD-rescue
- U5: symbol SteerMD-rescue:SI8900-Hori_lib-MD_Enbarr_x2-rescue-F4_CAN_DCMD-rescue -> CAN_DCMD-rescue:SI8900-Hori_lib-MD_Enbarr_x2-rescue-F4_CAN_DCMD-rescue-SteerMD-rescue
- U7: symbol SteerMD-rescue:BD9G101G-myDevice-MD_Enbarr_x2-rescue-F4_CAN_DCMD-rescue -> CAN_DCMD-rescue:BD9G101G-myDevice-MD_Enbarr_x2-rescue-F4_CAN_DCMD-rescue-SteerMD-rescue
- Y1: symbol SteerMD-rescue:Crystal-Device-MD_Enbarr_x2-rescue-F4_CAN_DCMD-rescue -> CAN_DCMD-rescue:Crystal-Device-MD_Enbarr_x2-rescue-F4_CAN_DCMD-rescue-SteerMD-rescue
Connections:
- net labels removed: MODE
- wire segments 300 -> 306
Other:
- moved on the sheet: TH1, TH2
