File: SteerMD/SteerMD.kicad_pcb (KiCad board)
At the start: 2 copper layers, 75 x 88 mm, 198 parts, among them P1 SWD, P10 OUT_1, P11 ENC_0, P13 ENC_1, P14 I/O_1, P15 OUT_0, P3 CAN, P4 CAN, P5 SERIAL, P6 I/O_0, P7 FAN, P8 BATT_IN, P9 BATT_IN, Q1 MOSFET_N, Q2 MOSFET_N, Q3 MOSFET_N, Q4 MOSFET_N, Q5 MOSFET_N, Q6 MOSFET_N, Q7 MOSFET_N, Q8 MOSFET_N, SW1 RST, SW3 SW0, SW4 SW1, U1 MAX3051, U10 ACS758, U11 POWER_ON, U12 SI8274, U13 ACS758, U14 SI8274, U15 AZ1086H, U16 LOGO, U19 ADRESS, U2 AP3211, U3 STM32F405RG, U4 SI8274, U5 SI8900, U6 ADC_~RST, U7 BD9G101G, U8 SI8274, U9 BD33FA1, Y1 8MHz

Commit message: 2019/12/8
Parts:
- moved R67 106.9 mm to (99.5, 81.1)
- moved TH1 37.9 mm to (99.7, 77.5)
Changed lines of the file:
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@@
   )
   (setup
-    (last_trace_width 1)
+    (last_trace_width 0.25)
     (user_trace_width 0.3)
     (user_trace_width 0.5)
@@
   )
   (module Resistor_SMD:R_0603_1608Metric (layer F.Cu)
-    (at 183.205001 14.665001)
+    (at 99.5 81.1)
     (descr "Resistor SMD 0603 (1608 Metric), square (rectangular) end terminal, IPC_7351 nominal, (Body size source: http://www.tortai-tech.com/upload/download/2011102023233369053.pdf), generated with kicad-footprint-generator")
     (tags resistor)
     (attr smd)
-    (fp_text reference R67 (at 0 -1.43) (layer F.SilkS)
+    (fp_text reference R67 (at 0 -1.43) (layer F.SilkS) hide
       (effects (font (size 1 1) (thickness 0.15)))
     )
-    (fp_text value 10k (at 0 1.43) (layer F.Fab)
-      (effects (font (size 1 1) (thickness 0.15)))
+    (fp_text value 10k (at 0 1.43) (layer F.SilkS)
+      (effects (font (size 0.8 0.8) (thickness 0.15)))
     )
     (fp_line (start -0.8 0.4) (end -0.8 -0.4) (layer F.Fab) (width 0.1))
@@
     (tags resistor)
     (attr smd)
-    (fp_text reference R68 (at 0 -1.43) (layer F.SilkS)
+    (fp_text reference R68 (at 0 -1.43) (layer F.SilkS) hide
       (effects (font (size 1 1) (thickness 0.15)))
     )
@@
   )
   (module Capacitor_SMD:C_0603_1608Metric (layer F.Cu)
-    (at 63.05 87.5)
+    (at 99.65 77.5)
     (descr "Capacitor SMD 0603 (1608 Metric), square (rectangular) end terminal, IPC_7351 nominal, (Body size source: http://www.tortai-tech.com/upload/download/2011102023233369053.pdf), generated with kicad-footprint-generator")
     (tags capacitor)
@@
     (tags capacitor)
     (attr smd)
-    (fp_text reference C4 (at 0 -1.43) (layer F.SilkS)
+    (fp_text reference C4 (at 0 -1.43) (layer F.SilkS) hide
       (effects (font (size 1 1) (thickness 0.15)))
     )
-    (fp_text value 0.1u (at 0 1.43) (layer F.Fab)
-      (effects (font (size 1 1) (thickness 0.15)))
+    (fp_text value 0.1u (at 0 1.43) (layer F.SilkS)
+      (effects (font (size 0.8 0.8) (thickness 0.15)))
     )
     (fp_text user %R (at 0 0) (layer F.Fab)
@@
     (tags capacitor)
     (attr smd)
-    (fp_text reference C21 (at 0 -1.43) (layer F.SilkS)
+    (fp_text reference C21 (at 0 -1.43) (layer F.SilkS) hide
       (effects (font (size 1 1) (thickness 0.15)))
     )
-    (fp_text value 0.1u (at 0 1.43) (layer F.Fab)
-      (effects (font (size 1 1) (thickness 0.15)))
+    (fp_text value 0.1u (at 0 1.43) (layer F.SilkS)
+      (effects (font (size 0.8 0.8) (thickness 0.15)))
     )
     (fp_line (start -0.8 0.4) (end -0.8 -0.4) (layer F.Fab) (width 0.1))
@@
     (tags capacitor)
     (attr smd)
-    (fp_text reference C52 (at 0 -1.43) (layer F.SilkS)
+    (fp_text reference C52 (at 0 -1.43) (layer F.SilkS) hide
       (effects (font (size 1 1) (thickness 0.15)))
     )
-    (fp_text value 0.1u (at 0 1.43) (layer F.Fab)
+    (fp_text value 0.1u (at 0 1.43) (layer F.SilkS)
       (effects (font (size 1 1) (thickness 0.15)))
     )
@@
     (tags resistor)
     (attr smd)
-    (fp_text reference R2 (at 0 -1.43) (layer F.SilkS)
+    (fp_text reference R2 (at 0 -1.43) (layer F.SilkS) hide
       (effects (font (size 1 1) (thickness 0.15)))
     )
-    (fp_text value 10k (at 0 1.43) (layer F.Fab)
-      (effects (font (size 1 1) (thickness 0.15)))
+    (fp_text value 10k (at 0 1.43) (layer F.SilkS)
+      (effects (font (size 0.8 0.8) (thickness 0.15)))
     )
     (fp_line (start -0.8 0.4) (end -0.8 -0.4) (layer F.Fab) (width 0.1))
@@
     (tags resistor)
     (attr smd)
-    (fp_text reference R13 (at 0 -1.43) (layer F.SilkS)
+    (fp_text reference R13 (at 0 -1.43) (layer F.SilkS) hide
       (effects (font (size 1 1) (thickness 0.15)))
     )
-    (fp_text value 100k (at 0 1.43) (layer F.Fab)
+    (fp_text value 100k (at 0 1.43) (layer F.SilkS)
       (effects (font (size 1 1) (thickness 0.15)))
     )
@@
     (tags resistor)
     (attr smd)
-    (fp_text reference R53 (at 0 -1.43) (layer F.SilkS)
+    (fp_text reference R53 (at 0 -1.43) (layer F.SilkS) hide
       (effects (font (size 1 1) (thickness 0.15)))
     )
-    (fp_text value FILTER (at 0 1.43) (layer F.Fab)
-      (effects (font (size 1 1) (thickness 0.15)))
+    (fp_text value FILTER (at 0 1.43) (layer F.SilkS)
+      (effects (font (size 0.8 0.8) (thickness 0.15)))
     )
     (fp_text user %R (at 0 0) (layer F.Fab)
@@
     (tags resistor)
     (attr smd)
-    (fp_text reference R54 (at 0 -1.43) (layer F.SilkS)
+    (fp_text reference R54 (at 0 -1.43) (layer F.SilkS) hide
       (effects (font (size 1 1) (thickness 0.15)))
     )
-    (fp_text value FILTER (at 0 1.43) (layer F.Fab)
-      (effects (font (size 1 1) (thickness 0.15)))
+    (fp_text value FILTER (at 0 1.43) (layer F.SilkS)
+      (effects (font (size 0.8 0.8) (thickness 0.15)))
     )
     (fp_line (start -0.8 0.4) (end -0.8 -0.4) (layer F.Fab) (width 0.1))
@@
     (tags resistor)
     (attr smd)
-    (fp_text reference R63 (at 0 -1.43) (layer F.SilkS)
+    (fp_text reference R63 (at 0 -1.43) (layer F.SilkS) hide
       (effects (font (size 1 1) (thickness 0.15)))
     )
-    (fp_text value FILTER (at 0 1.43) (layer F.Fab)
-      (effects (font (size 1 1) (thickness 0.15)))
+    (fp_text value FILTER (at 0 1.43) (layer F.SilkS)
+      (effects (font (size 0.8 0.8) (thickness 0.15)))
     )
     (fp_line (start -0.8 0.4) (end -0.8 -0.4) (layer F.Fab) (width 0.1))
@@
     (tags resistor)
     (attr smd)
-    (fp_text reference R64 (at 0 -1.43) (layer F.SilkS)
+    (fp_text reference R64 (at 0 -1.43) (layer F.SilkS) hide
       (effects (font (size 1 1) (thickness 0.15)))
     )
-    (fp_text value FILTER (at 0 1.43) (layer F.Fab)
-      (effects (font (size 1 1) (thickness 0.15)))
+    (fp_text value FILTER (at 0 1.43) (layer F.SilkS)
+      (effects (font (size 0.8 0.8) (thickness 0.15)))
     )
     (fp_text user %R (at 0 0) (layer F.Fab)
@@
     (tags resistor)
     (attr smd)
-    (fp_text reference R65 (at 0 -1.43) (layer F.SilkS)
+    (fp_text reference R65 (at 0 -1.43) (layer F.SilkS) hide
       (effects (font (size 1 1) (thickness 0.15)))
     )
-    (fp_text value 100k (at 0 1.43) (layer F.Fab)
-      (effects (font (size 1 1) (thickness 0.15)))
+    (fp_text value 100k (at 0 1.43) (layer F.SilkS)
+      (effects (font (size 0.8 0.8) (thickness 0.15)))
     )
     (fp_line (start -0.8 0.4) (end -0.8 -0.4) (layer F.Fab) (width 0.1))
@@
     (tags resistor)
     (attr smd)
-    (fp_text reference R66 (at 0 -1.43) (layer F.SilkS)
+    (fp_text reference R66 (at 0 -1.43) (layer F.SilkS) hide
       (effects (font (size 1 1) (thickness 0.15)))
     )
-    (fp_text value 10k (at 0 1.43) (layer F.Fab)
+    (fp_text value 10k (at 0 1.43) (layer F.SilkS)
       (effects (font (size 1 1) (thickness 0.15)))
     )

Commit message: 2019/12/12途中(内職)
Parts:
- added R52: FILTER, Resistor_SMD:R_0603_1608Metric, F.Cu at (182.4, 98.6)
- added R69: FILTER, Resistor_SMD:R_0603_1608Metric, F.Cu at (182.4, 101.1)
- added TH3: Thermistor, Capacitor_SMD:C_0603_1608Metric, F.Cu at (104.9, 74.9)
- added TH4: Thermistor, Capacitor_SMD:C_0603_1608Metric, F.Cu at (125.8, 75.0)
- P11, P13, P3, P4: footprint Mizz_lib:XA_4LC -> Mizz_lib:XA_4L
- P5: footprint Mizz_lib:XA_4LC -> Mizz_lib:XA_4P
- R67, R68: value 10k -> FILTER
- moved TH2 82.0 mm to (115.3, 75.0)
- moved R53 49.5 mm to (111.3, 75.8), turned to 270 degrees
- moved R63 49.1 mm to (122.0, 75.8), turned to 270 degrees
- moved R64 40.4 mm to (128.3, 60.0), turned to 270 degrees
- moved R54 35.0 mm to (111.7, 60.0), turned to 270 degrees
- moved R22 10.6 mm to (133.9, 92.5)
- moved R23 10.6 mm to (135.5, 92.5)
- moved C6 10.2 mm to (122.5, 118.0)
- moved C8 9.99 mm to (117.0, 111.0)
- moved P5 9.65 mm to (113.8, 135.7), turned to 180 degrees
- moved R9 8.92 mm to (119.7, 119.2), turned to 45 degrees
- moved R30 8.10 mm to (100.8, 75.8)
- moved R1 6.80 mm to (109.2, 112.3)
- moved TH1 5.81 mm to (94.5, 74.9)
- moved C15 5.40 mm to (108.8, 132.6), turned to 270 degrees
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Connections:
- net /Motor0_Tmp renamed /Motor0L_Tmp
- R68 pad 1: /Motor1_Tmp -> /Motor1L_Tmp
- TH2 pad 2: /Motor1_Tmp -> /Motor1L_Tmp
Routing:
- net /CounterVoltage0: track 74.2 -> 21.3 mm, vias 2 -> 0
- net /CounterVoltage1: track 53.8 -> 3.53 mm, vias 1 -> 0
- net /batt: track 26.9 -> 39.9 mm
- net Net-(Q6-PadG): track 0.00 -> 10.3 mm, vias 0 -> 1
- net +BATT: track 107.6 -> 98.4 mm, vias 40 -> 38
- net GNDPWR: track 64.2 -> 57.4 mm, vias 30 -> 33
- net /OUT1_R: track 4.23 -> 10.9 mm
- net /ADR_8: track 5.73 -> 0.00 mm
- net Net-(Q2-PadG): track 0.00 -> 4.22 mm, vias 0 -> 1
- net Net-(R66-Pad2): track 3.70 -> 0.00 mm
- net /Voltage: track 11.1 -> 7.86 mm
- net +5V: track 109.3 -> 107.2 mm, vias 2 -> 3
- net Net-(D47-Pad2): track 1.31 -> 0.00 mm
- net +3V3: track 44.6 -> 45.4 mm, vias 6 -> 8
- net Net-(Q8-PadG): vias 0 -> 1
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