File: stm32f4_Centaurus_ver.2.0/stm32f4_Centaurus_ver.2.0/stm32f4_Centaurus.sch (KiCad schematic (older format))
At the start: 207 parts, among them IC1 PIC24FJ64GB004, P1 PICKit3, P10 XA2_12V, P11 CAN0, P12 CAN1, P13 CAN0, P14 CAN1, P15 SERIAL2, P16 SERIAL0, P17 XA2_5V, P18 SWD, P2 SERIAL5_SBDBT, P23 A/D, P24 PWM, P25 A/D_batt, P26 PWM_batt, P27 EMERGENCY_CHECK, P28 I/O_5V, P29 I/O_Variable, P3 ENC0, P30 I/O_5V_batt, P31 I/O_Variable, P4 ENC2, P5 SERIAL1, P6 ENC3, P7 ENC1, P8 SERIAL4, P9 SERIAL3, Q1 FET_P, Q2 FET_P, Q3 FET_P, Q4 NPN, Q5 NPN, Q6 FET_P, Q7 FET_N, SW1 Main_POWER, SW2 SW1, SW3 SW0, SW4 SW2, SW5 SW3, U1 STM32F407VG, U10 LOGO, U12 25LC010A, U13 LOGO, U2 AZ1086H, U3 MCP2221A, U4 AP3211, U5 MAX3051, U6 MAX3051, U7 AQM1602_BL, U8 OSTBABS4C2B, U9 LOGO, X1 8MHz

Commit message: mainと電源が仮完成.
Parts:
- U13: footprint Mizz_lib:Robocon2019_30.0x30.0_silk -> Mizz_lib:Robocon2020_30.0x12.5_silk
Connections:
- net OSC_IN: now also C13.1
- net OSC_OUT: now also C11.1
Changed lines of the file:
@@
 F 0 "U13" H 20678 1253 60  0000 L CNN
 F 1 "LOGO" H 20678 1147 60  0000 L CNN
-F 2 "Mizz_lib:Robocon2019_30.0x30.0_silk" H 20400 1200 60  0001 C CNN
+F 2 "Mizz_lib:Robocon2020_30.0x12.5_silk" H 20400 1200 60  0001 C CNN
 F 3 "" H 20400 1200 60  0000 C CNN
 	1    20400 1200
@@
 	13075 15025 13100 15025
 Wire Wire Line
-	2125 7675 2175 7675
-Wire Wire Line
-	1475 7675 1525 7675
+	2125 7675 2150 7675
+Wire Wire Line
+	1475 7675 1500 7675
 Wire Wire Line
 	1425 6625 1425 6825
@@
 	17900 10450 17675 10450
 $Comp
-L power:+3.3V #PWR?
+L power:+3.3V #PWR0159
 U 1 1 5D5C8490
 P 17675 10050
-F 0 "#PWR?" H 17675 10010 30  0001 C CNN
+F 0 "#PWR0159" H 17675 10010 30  0001 C CNN
 F 1 "+3.3V" H 17684 10188 30  0000 C CNN
 F 2 "" H 17675 10050 60  0000 C CNN
@@
 Wire Wire Line
 	13100 15025 13250 15025
+Connection ~ 2150 7675
+Wire Wire Line
+	2150 7675 2175 7675
+Connection ~ 1500 7675
+Wire Wire Line
+	1500 7675 1525 7675
 $EndSCHEMATC

Commit message: main基板のdcdc改善
Parts:
- R35: value 50k -> 3.9k
- R36: value 10k -> 680
- U4: value AP3211 -> BD9G101G
Changed lines of the file:
@@
 P 5075 3525
 F 0 "U4" H 5075 3990 50  0000 C CNN
-F 1 "AP3211" H 5075 3899 50  0000 C CNN
+F 1 "BD9G101G" H 5075 3899 50  0000 C CNN
 F 2 "Mizz_lib:TSOT-6-MK06A" H 5075 3525 50  0001 C CNN
 F 3 "" H 5075 3525 50  0001 C CNN
@@
 P 5950 3475
 F 0 "R35" H 6028 3513 40  0000 L CNN
-F 1 "50k" H 6028 3437 40  0000 L CNN
+F 1 "3.9k" H 6028 3437 40  0000 L CNN
 F 2 "Mizz_lib:R_0603" V 5880 3475 30  0001 C CNN
 F 3 "" H 5950 3475 30  0000 C CNN
@@
 P 5950 3825
 F 0 "R36" H 6028 3863 40  0000 L CNN
-F 1 "10k" H 6028 3787 40  0000 L CNN
+F 1 "680" H 6028 3787 40  0000 L CNN
 F 2 "Mizz_lib:R_0603" V 5880 3825 30  0001 C CNN
 F 3 "" H 5950 3825 30  0000 C CNN

Commit message: パワー系の配線完了かな
Parts:
- R53: value 120 -> 10
Connections:
- net CAN0_BUS_Vdd: now also C22.2
- net CAN1_BUS_Vdd: now also C23.2
- net at R71.1: now also P27.4 (P4), Q7.1 (G)
Changed lines of the file:
@@
 P 20925 3650
 F 0 "R53" H 21003 3688 40  0000 L CNN
-F 1 "120" H 21003 3612 40  0000 L CNN
+F 1 "10" H 21003 3612 40  0000 L CNN
 F 2 "Mizz_lib:R_0603" V 20855 3650 30  0001 C CNN
 F 3 "" H 20925 3650 30  0000 C CNN
@@
 $EndComp
 Wire Wire Line
-	20625 7500 20625 7725
-Wire Wire Line
-	20625 8450 20625 8675
+	20625 7500 20625 7625
+Wire Wire Line
+	20625 8450 20625 8575
 Wire Wire Line
 	11775 14000 11800 14000
@@
 	16150 3250 16150 3450
 Wire Wire Line
-	16250 3750 16600 3750
+	16250 3750 16575 3750
 Connection ~ 5950 3325
 Wire Wire Line
@@
 Wire Wire Line
 	1500 7675 1525 7675
+Connection ~ 16575 3750
+Wire Wire Line
+	16575 3750 16600 3750
+Connection ~ 20625 7625
+Wire Wire Line
+	20625 7625 20625 7725
+Connection ~ 20625 8575
+Wire Wire Line
+	20625 8575 20625 8675
 $EndSCHEMATC
