File: Electricity_Manager/Electricity_Manager.kicad_pcb (KiCad board)
At the start: 2 copper layers, 100 x 77 mm, 197 parts, among them IC2 MAIN_SHUTDOWN, IC3 RELAY_STATE, IC4 ADC_RST, J1 SERIAL, P1 SWD, P10 EMERGENCY, P11 EMERGENCY, P12 FRAME_GRAND, P13 BATT_IN, P15 OUT_B, P16 BATT_IN, P17 OUT_A, P2 CAN, P3 CAN, P4 EMERGENCY_SIGNAL, P5 EMERGENCY_SIGNAL, P6 12V_OUT, P7 12V_OUT, P9 MAIN_SW, Q1 FET_N, Q2 NPN, Q3 NPN, Q4 FET_N, Q7 FET_N, SW1 RST, SW2 SW0, SW3 SW1, U1 MAX3051, U10 BD9G101G, U11 OUTA_CHECK, U12 LOGO, U13 LOGO, U14 OUTB_CHECK, U15 BD33FA1, U16 LOGO, U17 LOGO, U18 LOGO, U19 MCP2221A, U2 STM32F405RG, U20 OSRB38C9AA, U21 OSRB38C9AA, U22 HSIN_946, U23 LOGO, U25 LOGO, U3 FULL COLOR, U4 AQM0802_BL, U5 AP3211, U6 SI8900, U7 AZ1086H, U8 ACS70331, U9 LOGO, X1 8MHz

Commit message: electrocity -> electricity
Parts:
- removed DCDC1: MGFS402412, Mizz_lib:MGFS402412
- removed RL1, RL2: 7-1393302-7, Mizz_lib:7-1393302-7
- added U24: LOGO, Mizz_lib:Dodaitos_15x15_silk, B.Cu at (93.5, 164.0)
- C32: footprint Capacitor_THT:CP_Radial_D8.0mm_P2.50mm -> Capacitors_ThroughHole:C_Radial_D6.3_L11.2_P2.5
- C35: value 470u -> 100u; footprint Capacitor_THT:CP_Radial_D8.0mm_P3.50mm -> Capacitors_ThroughHole:C_Radial_D6.3_L11.2_P2.5
- D26: value TX -> RX
- D27: value RX -> TX
- R52: value 10k -> 49.9k
- R53: value 1k -> 10k
- U12: value LOGO -> V23134J1052D642; footprint Mizz_lib:Libra_15x15_silk -> Mizz_lib:V23134J1052D642
- U13: value LOGO -> ACS70331; footprint Mizz_lib:RP_KIT_Logo_mask_15.0x15.0 -> Mizz_lib:ALLEGRO_ACS70331EESATR-005U3
- U8: value ACS70331 -> V23134J1052D642; footprint Mizz_lib:ALLEGRO_ACS70331EESATR-005U3 -> Mizz_lib:V23134J1052D642
- U9: value LOGO -> RPA60-12FW/N; footprint Mizz_lib:Mega_Fusigibana_15x9_silk -> Mizz_lib:RPA60-24xxSFW; moved to F.Cu
- moved U8 73.5 mm to (62.5, 127.2), turned to 0 degrees
- moved U13 50.6 mm to (125.0, 166.0), turned to 90 degrees
- moved U12 30.8 mm to (89.2, 127.2)
- moved C32 18.8 mm to (66.2, 170.2)
- moved U9 18.4 mm to (95.2, 162.0), turned to 0 degrees
- moved U25 15.3 mm to (83.0, 170.5)
- moved D24 7.81 mm to (77.2, 151.2)
- moved D21 5.39 mm to (78.8, 166.5), turned to 90 degrees
- moved C35 5.35 mm to (124.0, 170.2)
- moved P16 3.25 mm to (58.8, 149.8)
- moved IC3 2.75 mm to (108.0, 160.8)
- moved P13 2.75 mm to (58.8, 160.0)
- moved R11 2.26 mm to (102.0, 159.5)
- moved C37 1.75 mm to (91.0, 155.8)
- moved C43 1.75 mm to (97.8, 155.5)
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Routing:
- net /24V: track 40.4 -> 27.4 mm
- net Net-(C35-Pad1): track 17.3 -> 9.71 mm
- net /Relay_Out: track 109.0 -> 115.4 mm
- net /Coil: track 129.5 -> 126.6 mm
- net +8V: track 100.6 -> 98.0 mm
- net 3V3: track 105.7 -> 107.3 mm
- net Net-(C36-Pad2): track 8.48 -> 9.63 mm
- net /Relay_state: track 47.8 -> 46.6 mm
- net Net-(IC4-Pad2): track 1.71 -> 2.46 mm
- net +BATT: track 17.1 -> 17.7 mm
- net GNDPWR: vias 297 -> 288
- net GND: vias 129 -> 135
Other:
- board text added: "Designed by A.Mizuta in 2019/11/05."
- board text added: "Electricity Manager ver.2.0"
- board text added: "Libra Zubenelgenubi"
- board text added: "Pocket Monster "Dodaitos""
- board text removed: "Designed by A.Mizuta in 2019/11/18."
- board text removed: "Electrocity Manager_40W"
- board text removed: "Libra Zubeneschamali"
- board text removed: "Pocket Monster "Mega Fushigibana""
