File: CAN_BLDCMD/CAN_BLDCMD.sch (KiCad schematic (older format))
At the start: 111 parts

Commit message: 何変更したか忘れた
Parts:
- added C? (x2): 4.7u, symbol Device:C
- added R? (x6): R, symbol Device:R
- added R?: 4.7k, symbol Device:R
- added R?: 10k, symbol Device:R
- added U?: BD33FA1, symbol Miz:BD33FA1
- added U?: POWER_ON, Package_SO:SOIC-4_4.55x2.6mm_P1.27mm, symbol Isolator:TLP291
Connections:
- net +3.3VP: now also U?.1 (Vo)
- net +3V3: now also U?.4
- net +BATT: now also U?.1
- net GND: now also R?.1
- net GNDPWR: now also R?.1, R?.2, R?.2, R?.2
- net OUT_U: now also R?.1
- net OUT_V: now also R?.1
- net OUT_W: now also R?.1
- net USARTx_RX: now reaches U?.12 (TX)
- net USARTx_TX: now reaches U?.13 (RX)
- new net: R?.2, U?.2
- new net POWER_ON: R?.2, U?.3
Other:
- moved on the sheet: C?, D?, J?, L?, Q?, R?, U?

Commit message: BLDCの設計を進めた
Parts:
- removed D?: DIODE, symbol pspice:DIODE
- added C? (x12): 0.1u, symbol Device:C
- added C?: 1u, symbol Device:C
- added C?: 4.7u, symbol Device:C
- added C?: 22u, symbol Device:C
- added C?: 10u, symbol Device:C
- added D? (x4): DIODE, symbol Miz:DIODE_rev
- added D?: 12VP, symbol Device:LED
- added D?: 3V3P, symbol Device:LED
- added D?: BATT, symbol Device:LED
- added D?: MAIN_BATT, symbol Device:LED
- added D?: 12V, symbol Device:LED
- added D?: 5V, symbol Device:LED
- added D?: 3V3, symbol Device:LED
- added D? (x3): LED, symbol Device:LED
- added D?: DIODE, symbol Miz:PWR_DIODE
- added J?: SWD, symbol Connector_Generic:Conn_01x06
- added J?: SERIAL, symbol Connector_Generic:Conn_01x04
- added J?: EX_SIGNAL_IN, symbol Connector_Generic:Conn_01x04
- added J?: FAN, symbol Connector_Generic:Conn_01x02
- added JP?: SWD_Vdd, symbol Device:Jumper
- added R? (x9): 10k, symbol Device:R
- added R? (x2): 4.7k, symbol Device:R
- added R?: 2.2k, symbol Device:R
- added R?: 330, symbol Device:R
- added R? (x3): 240, symbol Device:R
- added R?: 47, symbol Device:R
- added SW?: RST, symbol Switch:SW_Push
- added SW?: SW0, symbol Switch:SW_Push
- added SW?: SW1, symbol Switch:SW_Push
- added SW?: MODE, symbol Switch:SW_DPDT_x2
- added TH? (x4): Thermistor, symbol Device:Thermistor
- added U? (x2): LTC2644, symbol Miz:LTC2644
- added U?: AZ1086H, symbol Miz:AZ1086H
- C?: value 1500u -> 2200u
- R? (x2): value 100 -> 4.7k
- R? (x3): value R -> 10k
- R? (x3): value R -> 1k
Connections:
- net +12P: now also C?.1, U?.3 (Vcc), R?.2
- net +12V: now also D?.2 (A)
- net +3.3VP: now also C?.1, C?.1, C?.1, C?.1, C?.1, C?.1, C?.1, R?.2, U?.1 (Vcc), U?.1 (Vcc), U?.10 (REF), U?.10 (REF), U?.4 (IDLSEL), U?.4 (IDLSEL), U?.5 (IOVcc), U?.5 (IOVcc), U?.7 (~PD), U?.7 (~PD)
- net +3V3: now also C?.1, C?.1, C?.1, C?.1, C?.1, C?.1, C?.1, D?.1 (K), D?.2 (A), R?.1, R?.2, R?.2, TH?.1, TH?.1, TH?.1, TH?.1, U?.2 (V_OUT); no longer R?.2, R?.2
- net +5V: now also R?.2, R?.2, C?.1, C?.1, D?.2 (A), J?.2 (Pin_2), U?.3 (V_IN)
- net +BATT: now also D?.2 (A), R?.2
- net BATT: now also D?.1 (K), R?.2, R?.2
- net GND: now also C?.1, C?.2, C?.2, C?.2, C?.2, C?.2, C?.2, C?.2, C?.2, C?.2, D?.1 (K), D?.1 (K), D?.1 (K), D?.1 (K), D?.1 (K), D?.1 (K), J?.1 (Pin_1), J?.1 (Pin_1), J?.1 (Pin_1), R?.1, R?.1, R?.1, R?.1, R?.1, R?.1, SW?.1, SW?.1, SW?.1 (A), SW?.2, U?.1 (GND)
- net GNDPWR: now also C?.2, C?.2, U?.2 (GND), C?.2, C?.2, C?.2, C?.2, C?.2, C?.2, D?.1 (K), D?.1 (K), D?.1 (K), D?.1 (K), J?.1 (Pin_1), U?.11 (REFSEL), U?.11 (REFSEL), U?.12 (GND), U?.12 (GND), U?.6 (GND), U?.6 (GND)
- net PWM_U: now also D?.1 (K)
- net PWM_V: now also D?.1 (K)
- net PWM_W: now also D?.1 (K)
- net TIMx_CH1: now also R?.2; no longer R?.1
- net TIMx_CH2: now also R?.2; no longer R?.1
- net ~RST: now also C?.2, J?.5 (Pin_5), SW?.1
- net at U?.28 (BOOT1/PB2): now also R?.1
- net SWDIO: now reaches U?.46 (SWDIO/PA13)
- net SWDIO: now also J?.3 (Pin_3)
- net SWCLK: now reaches U?.49 (SWCLK/PA14)
- net SWCLK: now also J?.4 (Pin_4)
- net at J?.3 (Pin_3), R?.1: now also R?.1
- net at J?.4 (Pin_4), R?.1: now also R?.1
- net OUT_U_Voltage_DAC: now reaches U?.3 (AIN0)
- net OUT_U_Voltage_DAC: now also U?.2 (VoutA)
- net OUT_V_Voltage_DAC: now reaches U?.4 (AIN1)
- net OUT_V_Voltage_DAC: now also U?.3 (VoutB)
- net OUT_W_Voltage_DAC: now reaches U?.5 (AIN2)
- net OUT_W_Voltage_DAC: now also U?.2 (VoutA)
- net OUT_W_Voltage: now reaches R?.2
- net OUT_W_Voltage: now also R?.1, U?.9 (INA)
- net OUT_V_Voltage: now reaches R?.2
- net OUT_V_Voltage: now also R?.1, U?.8 (INB)
- net OUT_U_Voltage: now reaches R?.2
- net OUT_U_Voltage: now also R?.1, U?.9 (INA)
- new net: J?.2 (Pin_2), JP?.1
- new net: D?.2 (A), JP?.2
- new net: D?.2 (A), R?.1 (x7)
- new net: D?.2 (A), J?.2 (Pin_2)
- new net: D?.2 (A), J?.3 (Pin_3)
- new net: D?.2 (A), J?.4 (Pin_4)
- new net: J?.2 (Pin_2), R?.1
- new net LED0: R?.2
- new net LED1: R?.2
- new net LED2: R?.2
- new net OUT_U_Temp: R?.2, TH?.2
- new net OUT_V_Temp: R?.2, TH?.2
- new net OUT_W_Temp: R?.2, TH?.2
- new net SW0: R?.1, SW?.2
- new net SW1: R?.1, SW?.2
- new net USARTX_RX: J?.4 (Pin_4)
- new net USARTX_TX: J?.3 (Pin_3)
- new net mode_SW: R?.2, SW?.2 (B)
- new net substrateTemp: R?.2, TH?.2
- no-connect marks 12 -> 16
Other:
- note added: "TIM8:MotorDrive"
- moved on the sheet: C?, D?, J?, JP?, L?, R?, U?, Y?

Commit message: Main typeC化
Parts:
- added D2, D3, D4, D5: DIODE, Diode_SMD:D_0603_1608Metric, symbol Miz:DIODE_rev
- added J10: HALL_IN, symbol Connector_Generic:Conn_01x06
- added J11, J12, J13: Conn_01x01, symbol Connector_Generic:Conn_01x01
- added R11: 1.2k, Mizz_lib:1608_WP, symbol Device:R
- added R12: 510, Mizz_lib:1608_WP, symbol Device:R
- added R13: 330, Mizz_lib:1608_WP, symbol Device:R
- added R63, R64, R65: 10k, Mizz_lib:1608_WP, symbol Device:R
- added U19: ADRESS, symbol Miz:SW_ROTARY_16
- C1, C10, C12, C13, C14, C16, C17, C18, C19, C2, C20, C21, C22, C23, C24, C25, C26, C27, C28, C29, C3, C30, C31, C37, C38, C39, C4, C40, C41, C42, C43, C44, C45, C5, C6, C7, C8: renamed from C?; footprint (none) -> Mizz_lib:1608_WP
- C15, C32, C34, C36, C47, C48, C55, C9: renamed from C?; footprint (none) -> Capacitor_SMD:C_0805_2012Metric
- C46: renamed from C?; footprint (none) -> Mizz_lib:C_Radial_D13mm_H25.0mm_P5.00mm
- C49, C50, C51, C52, C53, C54: renamed from C?; footprint (none) -> Capacitor_SMD:C_1206_3216Metric
- D1, D19, D20, D6, D7, D8: renamed from D?; footprint (none) -> Diode_SMD:D_SOD-123
- D10, D11, D9: renamed from D?; footprint (none) -> Diode_SMD:D_0603_1608Metric
- D12, D13, D14, D15, D16, D17, D27, D28, D29, D30: renamed from D?; footprint (none) -> LED_SMD:LED_0603_1608Metric
- D18: renamed from D?; footprint (none) -> Diode_SMD:D_SMA
- D21, D22, D23, D24, D25, D26: renamed from D?; footprint (none) -> Mizz_lib:1608_WP
- J1: renamed from J?; footprint (none) -> Mizz_lib:XA_6LC
- J8: renamed from J?; footprint (none) -> Mizz_lib:XT60_F
- J9: renamed from J?; footprint (none) -> Mizz_lib:XT60_M
- JP1: renamed from JP?; footprint (none) -> Mizz_lib:GS2
- L1, L2: renamed from L?; footprint (none) -> Mizz_lib:Inductor_Taiyo-Yuden_NR-50xx_HandSoldering
- Q1, Q2, Q3, Q4, Q5, Q6: renamed from Q?; footprint (none) -> Mizz_lib:HSOF-8-1
- R1, R10, R14, R15, R16, R17, R18, R19, R2, R20, R21, R22, R23, R24, R25, R26, R27, R28, R29, R3, R30, R32, R33, R34, R35, R36, R37, R38, R39, R4, R40, R41, R42, R43, R44, R45, R46, R47, R48, R49, R5, R50, R51, R52, R53, R54, R55, R56, R57, R58, R59, R6, R60, R61, R62, R7, R8, R9: renamed from R?; footprint (none) -> Mizz_lib:1608_WP
- R31: renamed from R?; footprint (none) -> Mizz_lib:R_2812
- SW2: renamed from SW?; footprint (none) -> Mizz_lib:SW_Micro_SPST
- TH1, TH2, TH3, TH4: renamed from TH?; footprint (none) -> Mizz_lib:1608_WP
- U12, U13, U14: renamed from U?; footprint (none) -> Package_SO:SOP-16_4.4x10.4mm_P1.27mm
- U15, U16, U17: renamed from U?; footprint (none) -> Mizz_lib:ACS785xCB
- U18: renamed from U?; footprint (none) -> Mizz_lib:Mini_Monster
- U5: renamed from U?; footprint (none) -> Package_SO:SOIC-16W_7.5x10.3mm_P1.27mm
- Y1: renamed from Y?; footprint (none) -> Mizz_lib:Crystal_SMD_5032_2Pads
- gave numbers to parts that had none: 23
Connections:
- net +12V: now also R11.2; no longer D12.2 (A)
- net +3V3: now also R13.2; no longer D14.2 (A)
- net +5V: now also J10.6 (Pin_6), R12.2, R63.1, R64.1, R65.1; no longer D13.2 (A)
- net ADC_~RST~_PIN: now also U4.44 (CAN1_RX/TIM1_CH4/PA11)
- net CAN1_RX: now also U4.61 (TIM4_CH3/TIM10_CH1/CAN1_RX/PB8)
- net CAN1_TX: now also U4.62 (TIM4_CH4/TIM11_CH1/CAN1_TX/PB9)
- net Current_U: now also U4.25 (PC5/ADC12_IN15)
- net Current_V: now also U4.26 (ADC12_IN8/TIM1_CH2N/TIM8_CH2N/TIM3_CH3/PB0)
- net Current_W: now also U4.27 (ADC12_IN9/TIM1_CH3N/TIM8_CH3N/TIM3_CH4/PB1)
- net EN: now also D5.1 (K)
- net GND: now also J10.1 (Pin_1), U19.2 (C), U19.5 (C)
- net LED0: now also U4.9 (PC1/ADC12_IN11)
- net LED1: now also U4.10 (PC2/ADC12_IN12)
- net LED2: now also U4.11 (PC3/ADC12_IN13)
- net OUT_U_Temp: now also U4.20 (ADC12_IN4/PA4)
- net OUT_V_Temp: now also U4.21 (ADC12_IN5/TIM2_CH1_ETR/TIM8_CH1N/PA5)
- net OUT_W_Temp: now also U4.22 (ADC12_IN6/TIM3_CH1/TIM13_CH1/PA6)
- net POWER_ON: now also U4.45 (CAN1_TX/PA12)
- net PWM_U: now also D2.1 (K)
- net PWM_V: now also D3.1 (K)
- net PWM_W: now also D4.1 (K)
- net SW0: now also U4.2 (PC13)
- net SW1: now also U4.3 (PC14/OSC32_IN)
- net TIMx_CH1: now also U4.56 (TIM3_CH1/PB4)
- net TIMx_CH2: now also U4.57 (CAN2_RX/TIM3_CH2/PB5)
- net USARTX_RX: now also U4.43 (USART1_RX/TIM1_CH3/PA10)
- net USARTX_TX: now also U4.42 (USART1_TX/TIM1_CH2/PA9)
- net USARTx_RX: now also U4.17 (USART2_RX/TIM5_CH4/TIM9_CH2/ADC12_IN3/TIM2_CH4/PA3)
- net USARTx_TX: now also U4.16 (USART2_TX/TIM5_CH3/TIM9_CH1/ADC12_IN2/TIM2_CH3/PA2)
- net mode_SW: now also U4.4 (PC15/OSC32_OUT)
- net substrateTemp: now also U4.23 (ADC12_IN7/TIM1_CH1N/TIM8_CH1N/TIM14_CH1/TIM3_CH2/PA7)
- net ADRESS_0: now reaches U4.33 (CAN2_RX/PB12)
- net ADRESS_0: now also U19.3 (1)
- net ADRESS_1: now reaches U4.34 (TIM1_CH1N/CAN2_TX/PB13)
- net ADRESS_1: now also U19.1 (2)
- net ADRESS_2: now reaches U4.35 (TIM1_CH2N/TIM8_CH2N/TIM12_CH1/PB14)
- net ADRESS_2: now also U19.4
- net ADRESS_3: now reaches U4.36 (TIM1_CH3N/TIM8_CH3N/TIM12_CH2/PB15)
- net ADRESS_3: now also U19.6 (8)
- net at U4.37 (PC6/TIM8_CH1/USART6_TX/TIM3_CH1): now also D2.2 (A)
- net at U4.38 (PC7/TIM8_CH2/USART6_RX/TIM3_CH2): now also D3.2 (A)
- net at U4.39 (PC8/TIM8_CH3/TIM3_CH3): now also D4.2 (A)
- net at U4.40 (PC9/TIM8_CH4/TIM3_CH4): now also D5.2 (A)
- net HALL_0: now reaches U4.51 (PC10/UART4_TX/USART3_TX)
- net HALL_0: now also J10.2 (Pin_2), J11.1 (Pin_1), R65.2
- net HALL_1: now reaches U4.52 (PC11/UART4_RX/USART3_RX)
- net HALL_1: now also J10.3 (Pin_3), J12.1 (Pin_1), R64.2
- net HALL_2: now reaches U4.53 (PC12/UART5_TX)
- net HALL_2: now also J10.4 (Pin_4), J13.1 (Pin_1), R63.2
- new net: D12.2 (A), R11.1
- new net: D13.2 (A), R12.1
- new net: D14.2 (A), R13.1
- no-connect marks 16 -> 17
Other:
- moved on the sheet: D12, D13, D14, R21, R22, R23, R24, TH1, TH2, TH3, TH4
