File: Electricity_Manager_40W/Electricity_Manager_40W.sch (KiCad schematic (older format))
At the start: 197 parts, among them IC2 MAIN_SHUTDOWN, IC3 RELAY_STATE, IC4 ADC_RST, J1 SERIAL, P1 SWD, P10 EMERGENCY, P11 EMERGENCY, P12 FRAME_GRAND, P13 BATT_IN, P15 OUT_B, P16 BATT_IN, P17 OUT_A, P2 CAN, P3 CAN, P4 EMERGENCY_SIGNAL, P5 EMERGENCY_SIGNAL, P6 12V_OUT, P7 12V_OUT, P9 MAIN_SW, Q1 FET_N, Q2 NPN, Q3 NPN, Q4 FET_N, Q7 FET_N, SW1 RST, SW2 SW0, SW3 SW1, U1 MAX3051, U10 BD9G101G, U11 OUTA_CHECK, U12 LOGO, U13 LOGO, U14 OUTB_CHECK, U15 BD33FA1, U16 LOGO, U17 LOGO, U18 LOGO, U19 MCP2221A, U2 STM32F405RG, U20 OSRB38C9AA, U21 OSRB38C9AA, U22 HSIN_946, U23 LOGO, U25 LOGO, U3 FULL COLOR, U4 AQM0802_BL, U5 AP3211, U6 SI8900, U7 AZ1086H, U8 ACS70331, U9 LOGO, X1 8MHz

Commit message: だいぶ良いところまで進んだ
Parts:
- C1, C10, C11, C12, C13, C14, C15, C16, C17, C18, C19, C2, C20, C21, C22, C23, C24, C25, C26, C27, C28, C29, C3, C30, C31, C33, C34, C36, C37, C38, C4, C41, C42, C43, C44, C46, C47, C48, C49, C5, C6, C7, C8, C9: symbol Electrocity_Manager_40W-rescue:C-device-Electrocity_Manager-rescue -> Electricity_Manager_40W-rescue:C-device-Electrocity_Manager-rescue-Electrocity_Manager_40W-rescue
- C32, C35: symbol Electrocity_Manager_40W-rescue:CP1-device-Electrocity_Manager-rescue -> Electricity_Manager_40W-rescue:CP1-device-Electrocity_Manager-rescue-Electrocity_Manager_40W-rescue
- D1, D11, D12, D13, D21, D22, D23, D24, D25, D29, D9: symbol Electrocity_Manager_40W-rescue:DIODE-device-Electrocity_Manager-rescue-Electrocity_Manager-rescue -> Electricity_Manager_40W-rescue:DIODE-device-Electrocity_Manager-rescue-Electrocity_Manager-rescue-Electrocity_Manager_4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
- D10: symbol Electrocity_Manager_40W-rescue:SBR_DIODE-Miz-Electrocity_Manager-rescue-Electrocity_Manager-rescue -> Electricity_Manager_40W-rescue:SBR_DIODE-Miz-Electrocity_Manager-rescue-Electrocity_Manager-rescue-Electrocity_Manager_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
- D14, D15, D16, D17, D18, D19, D2, D20, D26, D27, D28, D3, D4, D5, D6, D7, D8: symbol Electrocity_Manager_40W-rescue:LED-device-Electrocity_Manager-rescue -> Electricity_Manager_40W-rescue:LED-device-Electrocity_Manager-rescue-Electrocity_Manager_40W-rescue
- IC2, IC3, IC4: symbol Electrocity_Manager_40W-rescue:TLP291-opto-Electrocity_Manager-rescue -> Electricity_Manager_40W-rescue:TLP291-opto-Electrocity_Manager-rescue-Electrocity_Manager_40W-rescue
- J1: symbol Electrocity_Manager_40W-rescue:USB_B_Micro-Connector-Electrocity_Manager-rescue-Electrocity_Manager-rescue -> Electricity_Manager_40W-rescue:USB_B_Micro-Connector-Electrocity_Manager-rescue-Electrocity_Manager-rescue-Electrocity_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
- JP1, JP2, JP3: symbol Electrocity_Manager_40W-rescue:JUMPER-device-Electrocity_Manager-rescue -> Electricity_Manager_40W-rescue:JUMPER-device-Electrocity_Manager-rescue-Electrocity_Manager_40W-rescue
- L1, L2: symbol Electrocity_Manager_40W-rescue:INDUCTOR_SMALL-device-Electrocity_Manager-rescue -> Electricity_Manager_40W-rescue:INDUCTOR_SMALL-device-Electrocity_Manager-rescue-Electrocity_Manager_40W-rescue
- P1: symbol Electrocity_Manager_40W-rescue:CONN_01X06-conn-Electrocity_Manager-rescue -> Electricity_Manager_40W-rescue:CONN_01X06-conn-Electrocity_Manager-rescue-Electrocity_Manager_40W-rescue
- P10, P11, P13, P15, P16, P17, P6, P7, P9: symbol Electrocity_Manager_40W-rescue:CONN_01X02-conn-Electrocity_Manager-rescue -> Electricity_Manager_40W-rescue:CONN_01X02-conn-Electrocity_Manager-rescue-Electrocity_Manager_40W-rescue
- P12: symbol Electrocity_Manager_40W-rescue:CONN_01X01-conn-Electrocity_Manager-rescue -> Electricity_Manager_40W-rescue:CONN_01X01-conn-Electrocity_Manager-rescue-Electrocity_Manager_40W-rescue
- P2, P3, P4, P5: symbol Electrocity_Manager_40W-rescue:CONN_01X04-conn-Electrocity_Manager-rescue -> Electricity_Manager_40W-rescue:CONN_01X04-conn-Electrocity_Manager-rescue-Electrocity_Manager_40W-rescue
- Q1, Q4, Q7: symbol Electrocity_Manager_40W-rescue:MOSFET_N_123-Hori_lib-Electrocity_Manager-rescue-Electrocity_Manager-rescue -> Electricity_Manager_40W-rescue:MOSFET_N_123-Hori_lib-Electrocity_Manager-rescue-Electrocity_Manager-rescue-Electrocity_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
- Q2, Q3: symbol Electrocity_Manager_40W-rescue:NPN-device-Electrocity_Manager-rescue-Electrocity_Manager-rescue -> Electricity_Manager_40W-rescue:NPN-device-Electrocity_Manager-rescue-Electrocity_Manager-rescue-Electrocity_Manager_40W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
- R1, R10, R11, R12, R13, R14, R15, R16, R17, R18, R19, R2, R20, R21, R22, R23, R24, R25, R26, R27, R28, R29, R3, R30, R31, R32, R33, R34, R35, R36, R37, R38, R39, R4, R40, R41, R42, R43, R44, R45, R46, R47, R48, R49, R5, R50, R51, R52, R53, R54, R58, R59, R6, R7, R8: symbol Electrocity_Manager_40W-rescue:R-device-Electrocity_Manager-rescue -> Electricity_Manager_40W-rescue:R-device-Electrocity_Manager-rescue-Electrocity_Manager_40W-rescue
- SP1: symbol Electrocity_Manager_40W-rescue:SPEAKER-device-Electrocity_Manager-rescue -> Electricity_Manager_40W-rescue:SPEAKER-device-Electrocity_Manager-rescue-Electrocity_Manager_40W-rescue
- SW1, SW2, SW3: symbol Electrocity_Manager_40W-rescue:SW_PUSH-device-Electrocity_Manager-rescue -> Electricity_Manager_40W-rescue:SW_PUSH-device-Electrocity_Manager-rescue-Electrocity_Manager_40W-rescue
- U1: symbol Electrocity_Manager_40W-rescue:MAX3051-myDevice-Electrocity_Manager-rescue-Electrocity_Manager-rescue -> Electricity_Manager_40W-rescue:MAX3051-myDevice-Electrocity_Manager-rescue-Electrocity_Manager-rescue-Electrocity_Manag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
- U10: symbol Electrocity_Manager_40W-rescue:BD9G101G-myDevice-Electrocity_Manager-rescue-Electrocity_Manager-rescue -> Electricity_Manager_40W-rescue:BD9G101G-myDevice-Electrocity_Manager-rescue-Electrocity_Manager-rescue-Electrocity_Mana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
- U12, U16, U17, U18, U23, U25: symbol Electrocity_Manager_40W-rescue:LOGO-myDevice-Electrocity_Manager-rescue-Electrocity_Manager-rescue -> Electricity_Manager_40W-rescue:LOGO-myDevice-Electrocity_Manager-rescue-Electrocity_Manager-rescue-Electrocity_Manager_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
- U15: symbol Electrocity_Manager_40W-rescue:BD33FA1-Miz-Electrocity_Manager-rescue-Electrocity_Manager-rescue -> Electricity_Manager_40W-rescue:BD33FA1-Miz-Electrocity_Manager-rescue-Electrocity_Manager-rescue-Electrocity_Manager_40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
- U19: symbol Electrocity_Manager_40W-rescue:MCP2221-Miz-Electrocity_Manager-rescue-Electrocity_Manager-rescue -> Electricity_Manager_40W-rescue:MCP2221-Miz-Electrocity_Manager-rescue-Electrocity_Manager-rescue-Electrocity_Manager_40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
- U2: symbol Electrocity_Manager_40W-rescue:STM32F405RG_excerpt-stm32f405rg_excerpt-Electrocity_Manager-rescue-Electrocity_Manager-r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 -> Electricity_Manager_40W-rescue:STM32F405RG_excerpt-stm32f405rg_excerpt-Electrocity_Manager-rescue-Electrocity_Manager-r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
- U20, U21: symbol Electrocity_Manager_40W-rescue:OSRB38C9AA-Miz-Electrocity_Manager-rescue-Electrocity_Manager-rescue -> Electricity_Manager_40W-rescue:OSRB38C9AA-Miz-Electrocity_Manager-rescue-Electrocity_Manager-rescue-Electrocity_Manager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
- U22: symbol Electrocity_Manager_40W-rescue:HSIN_946-relays-Electrocity_Manager-rescue -> Electricity_Manager_40W-rescue:HSIN_946-relays-Electrocity_Manager-rescue-Electrocity_Manager_40W-rescue
- U3: symbol Electrocity_Manager_40W-rescue:OSTBABS4C2B-myDevice-Electrocity_Manager-rescue-Electrocity_Manager-rescue -> Electricity_Manager_40W-rescue:OSTBABS4C2B-myDevice-Electrocity_Manager-rescue-Electrocity_Manager-rescue-Electrocity_M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
- U4: symbol Electrocity_Manager_40W-rescue:AQM0802_BL-Hori_lib-Electrocity_Manager-rescue-Electrocity_Manager-rescue -> Electricity_Manager_40W-rescue:AQM0802_BL-Hori_lib-Electrocity_Manager-rescue-Electrocity_Manager-rescue-Electrocity_Ma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
- U5: symbol Electrocity_Manager_40W-rescue:AP3211-Miz-Electrocity_Manager-rescue-Electrocity_Manager-rescue -> Electricity_Manager_40W-rescue:AP3211-Miz-Electrocity_Manager-rescue-Electrocity_Manager-rescue-Electrocity_Manager_40W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
- U6: symbol Electrocity_Manager_40W-rescue:SI8900-Hori_lib-Electrocity_Manager-rescue-Electrocity_Manager-rescue-Electrocity_Manage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 -> Electricity_Manager_40W-rescue:SI8900-Hori_lib-Electrocity_Manager-rescue-Electrocity_Manager-rescue-Electrocity_Manage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
- U7: symbol Electrocity_Manager_40W-rescue:AZ1086H-myDevice-Electrocity_Manager-rescue -> Electricity_Manager_40W-rescue:AZ1086H-myDevice-Electrocity_Manager-rescue-Electrocity_Manager_40W-rescue
- U8: symbol Electrocity_Manager_40W-rescue:ACS70331EESATR-005U3-ACS70331EESATR-005U3 -> Electricity_Manager_40W-rescue:ACS70331EESATR-005U3-ACS70331EESATR-005U3-Electrocity_Manager_40W-rescue
- X1: symbol Electrocity_Manager_40W-rescue:CRYSTAL-device-Electrocity_Manager-rescue -> Electricity_Manager_40W-rescue:CRYSTAL-device-Electrocity_Manager-rescue-Electrocity_Manager_40W-rescue
