File: CAN_BLDCMD_ver.0.0/CAN_BLDCMD.kicad_pcb (KiCad board)
At the start: 2 copper layers, 179 parts, among them J1 SWD, J10 BATT_IN, J11 OUT_U, J12 OUT_V, J13 OUT_W, J2 CAN, J3 CAN, J4 ENC, J5 I/O0, J6 I/O1, J7 SERIAL, J8 FAN, J9 BATT_IN, Q1 MOSFET_N, Q2 MOSFET_N, Q3 MOSFET_N, Q4 MOSFET_N, Q5 MOSFET_N, Q6 MOSFET_N, SW1 SW0, SW2 SW1, U1 MAX3051, U10 SI8900, U11 ADC_~RST, U12 ACS758, U13 ACS758, U14 ACS758, U15 BD9G101G, U16 LTC2644, U17 LTC2644, U18 BD33FA1, U19 LOGO, U2 BD9G101G, U3 STM32F405RG, U4 AZ1086H, U5 SW_ROTARY_16, U6 POWER_ON, U7 SI8274, U8 SI8274, U9 SI8274, Y1 8MHz

Commit message: ぶざーてすときばんは頭悪い
Parts:
- removed C29, C42: 0.1u, Capacitor_SMD:C_0603_1608Metric
- removed C59, C60: 4.7u, Capacitor_SMD:C_0805_2012Metric
- removed R26: 10k, Mizz_lib:1608_WP
- removed R27: 330, Mizz_lib:1608_WP
- removed R28, R32: 4.7k, Mizz_lib:1608_WP
- removed U12, U13, U14: ACS758, Mizz_lib:ACS785xCB
- removed U18: BD33FA1, Package_TO_SOT_SMD:SOT-89-3
- R34: moved to B.Cu
- R39, R40, R41, R42, R43, R44: value 1 -> 10
- U1: value MAX3051 -> ISO1050DUB; footprint Package_SO:SOIC-8_3.9x4.9mm_P1.27mm -> Package_SO:SOP-8_6.62x9.15mm_P2.54mm
- U10: value SI8900 -> ACS758; footprint Package_SO:SOIC-16W_7.5x10.3mm_P1.27mm -> Mizz_lib:ACS785xCB
- U11: value ADC_~RST -> ACS758; footprint Package_SO:SOIC-4_4.55x2.6mm_P1.27mm -> Mizz_lib:ACS785xCB
- U6: value POWER_ON -> ACS758; footprint Package_SO:SOIC-4_4.55x2.6mm_P1.27mm -> Mizz_lib:ACS785xCB
- moved R33 135.5 mm to (205.3, 66.8), turned to 180 degrees
- moved R34 110.0 mm to (198.4, 66.5), turned to 180 degrees
- moved U7 101.7 mm to (179.9, 65.2)
- moved U11 99.6 mm to (150.8, 149.4)
- moved TH1 95.4 mm to (201.0, 60.8), turned to 270 degrees
- moved U10 94.8 mm to (131.8, 149.4)
- moved U6 85.6 mm to (112.8, 149.4)
- moved U1 70.4 mm to (109.7, 156.0)
- moved C36 65.8 mm to (184.8, 62.1), turned to 270 degrees
- moved D9 58.0 mm to (187.1, 68.4), turned to 270 degrees
- moved C37 57.0 mm to (184.8, 68.4), turned to 270 degrees
- moved D8 50.6 mm to (187.1, 62.1), turned to 270 degrees
Connections:
- C10 pad 2: GND -> Earth
- C37 pad 2: GNDPWR -> GND
- C39 pad 2: GNDPWR -> GND
- C41 pad 2: GNDPWR -> GND
- C44 pad 1: GNDPWR -> GND
- C45 pad 1: GNDPWR -> GND
- C46 pad 1: GNDPWR -> GND
- C48 pad 2: GNDPWR -> Net-(C48-Pad2)
- C49 pad 2: GNDPWR -> GND
- C50 pad 2: GNDPWR -> Net-(C48-Pad2)
- C51 pad 2: GNDPWR -> GND
- C52 pad 2: GNDPWR -> GND
- C53 pad 2: GNDPWR -> GND
- C54 pad 2: GNDPWR -> GND
- C55 pad 2: GNDPWR -> GND
- C56 pad 2: GNDPWR -> Net-(C48-Pad2)
- C57 pad 2: GNDPWR -> GND
- C58 pad 1: Net-(C58-Pad1) -> +12P
- C58 pad 2: GNDPWR -> Net-(C48-Pad2)
- C9 pad 2: GND -> Earth
- D14 pad 2: GNDPWR -> GND
- D16 pad 1: Net-(C58-Pad1) -> +12P
- D3 pad 2: +12V -> +12P
- J10 pad 1: GNDPWR -> GND
- J2 pad 1: GND -> Earth
- J3 pad 1: GND -> Earth
- J8 pad 1: GNDPWR -> GND
- J9 pad 1: GNDPWR -> GND
- R46 pad 2: GNDPWR -> GND
- R49 pad 2: GNDPWR -> GND
- R51 pad 2: GNDPWR -> GND
- R53 pad 2: GNDPWR -> GND
- U1 pad 1: /CAN1_TX -> +3V3
- U1 pad 2: GND -> /CAN1_RX
- U1 pad 3: +3V3 -> /CAN1_TX
- U1 pad 4: /CAN1_RX -> GND
- U1 pad 5: GND -> Earth
- U1 pad 8: GND -> Net-(U1-Pad8)
- U10 pad 1: +3.3VP -> +3V3
- U10 pad 2: +3.3VP -> GND
- U10 pad 3: /OUT_U_Analog -> Net-(R30-Pad1)
- U10 pad 4: /OUT_V_Analog -> Net-(Q4-PadS)
- U10 pad 5: /OUT_W_Analog -> GND
- U11 pad 1: /ADC_~RST~_Pin -> +3V3
- U11 pad 2: Net-(R27-Pad1) -> GND
- U11 pad 3: GNDPWR -> Net-(R31-Pad1)
- U11 pad 4: Net-(R28-Pad2) -> Net-(Q6-PadS)
- U15 pad 2: GNDPWR -> GND
- U16 pad 11: GNDPWR -> GND
- U16 pad 12: GNDPWR -> GND
- U16 pad 6: GNDPWR -> GND
- U17 pad 11: GNDPWR -> GND
- U17 pad 12: GNDPWR -> GND
- U17 pad 6: GNDPWR -> GND
- U6 pad 1: Net-(R32-Pad2) -> +3V3
- U6 pad 2: GNDPWR -> GND
- U6 pad 3: /PWR_ON_Pin -> Net-(R29-Pad1)
- U6 pad 4: +3V3 -> Net-(Q2-PadS)
- U7 pad 9: GNDPWR -> GND
- U8 pad 9: GNDPWR -> GND
- U9 pad 9: GNDPWR -> GND
