File: CAN_BLDCMD_ver.0.0/CAN_BLDCMD.sch (KiCad schematic (older format))
At the start: 179 parts, among them J1 SWD, J10 BATT_IN, J11 OUT_U, J12 OUT_V, J13 OUT_W, J2 CAN, J3 CAN, J4 ENC, J5 I/O0, J6 I/O1, J7 SERIAL, J8 FAN, J9 BATT_IN, Q1 MOSFET_N, Q2 MOSFET_N, Q3 MOSFET_N, Q4 MOSFET_N, Q5 MOSFET_N, Q6 MOSFET_N, SW1 SW0, SW2 SW1, U1 MAX3051, U10 SI8900, U11 ADC_~RST, U12 ACS758, U13 ACS758, U14 ACS758, U15 BD9G101G, U16 LTC2644, U17 LTC2644, U18 BD33FA1, U19 LOGO, U2 BD9G101G, U3 STM32F405RG, U4 AZ1086H, U5 SW_ROTARY_16, U6 POWER_ON, U7 SI8274, U8 SI8274, U9 SI8274, Y1 8MHz

Commit message: CAN BLDC やる気が出たバージョンの設計開始
Parts:
- removed C29, C42: 0.1u, Capacitor_SMD:C_0603_1608Metric, symbol Device:C
- removed C59, C60: 4.7u, Capacitor_SMD:C_0805_2012Metric, symbol Device:C
- removed R26: 10k, Mizz_lib:1608_WP, symbol Device:R
- removed R27: 330, Mizz_lib:1608_WP, symbol Device:R
- removed R28, R32: 4.7k, Mizz_lib:1608_WP, symbol Device:R
- removed U1: MAX3051, Package_SO:SOIC-8_3.9x4.9mm_P1.27mm, symbol Interface_UART:MAX3051
- removed U10: SI8900, Package_SO:SOIC-16W_7.5x10.3mm_P1.27mm, symbol Miz:SI8900
- removed U11: ADC_~RST, Package_SO:SOIC-4_4.55x2.6mm_P1.27mm, symbol Isolator:TLP291
- removed U12, U13, U14: ACS758, Mizz_lib:ACS785xCB, symbol Miz:ACS758
- removed U18: BD33FA1, Package_TO_SOT_SMD:SOT-89-3, symbol Miz:BD33FA1
- removed U6: POWER_ON, Package_SO:SOIC-4_4.55x2.6mm_P1.27mm, symbol Isolator:TLP291
- added R?: R, symbol Device:R
- added U?: ISO1050DUB, Package_SO:SOP-8_6.62x9.15mm_P2.54mm, symbol Interface_CAN_LIN:ISO1050DUB
Connections:
- net +12P: now also C58.1, D16.1 (K), D3.2 (A)
- net +12V: no longer D3.2 (A)
- net +3V3: now also U?.1 (VCC1)
- net CAN1_RX: now also U?.2 (RXD)
- net CAN1_TX: now also U?.3 (TXD)
- net CAN_H: now also U?.7 (CANH)
- net CAN_L: now also U?.6 (CANL)
- net GND: now also C37.2, C39.2, C41.2, C44.1, C45.1, C46.1, C49.2, C51.2, C52.2, C53.2, C54.2, C55.2, C57.2, D14.2 (A), J10.1 (Pin_1), J8.1 (Pin_1), J9.1 (Pin_1), R46.2, R49.2, R51.2, R53.2, U15.2 (GND), U16.11 (REFSEL), U16.12 (GND), U16.6 (GND), U17.11 (REFSEL), U17.12 (GND), U17.6 (GND), U7.9 (GNCB), U8.9 (GNCB), U9.9 (GNCB), U?.4 (GND1); no longer C10.2, C9.2, J2.1 (Pin_1), J3.1 (Pin_1)
- net OUT_U_Current: now also Q2.S
- removed net GNDPWR: C37.2, C39.2, C41.2, C44.1, C45.1, C46.1, C48.2, C49.2, C50.2, C51.2, C52.2, C53.2, C54.2, C55.2, C56.2, C57.2, C58.2, D14.2 (A), J10.1 (Pin_1), J8.1 (Pin_1), J9.1 (Pin_1), R46.2, R49.2, R51.2, R53.2, U15.2 (GND), U16.11 (REFSEL), U16.12 (GND), U16.6 (GND), U17.11 (REFSEL), U17.12 (GND), U17.6 (GND), U7.9 (GNCB), U8.9 (GNCB), U9.9 (GNCB)
- new net: C48.2, C50.2, C56.2, C58.2
- new net Earth: C10.2, C9.2, J2.1 (Pin_1), J3.1 (Pin_1), U?.5 (GND2)
Other:
- moved on the sheet: C1, C10, C11, C12, C13, C14, C15, C16, C17, C18, C19, C2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

Commit message: ぶざーてすときばんは頭悪い
Parts:
- removed R?: R, symbol Device:R
- removed U?: ISO1050DUB, Package_SO:SOP-8_6.62x9.15mm_P2.54mm, symbol Interface_CAN_LIN:ISO1050DUB
- added C? (x2): 1u, symbol Device:C
- added C?: 0.1u, symbol Device:C
- added C? (x2): 4.7u, Capacitor_SMD:C_0805_2012Metric, symbol Device:C
- added D?: BATT, symbol Device:LED
- added D? (x2): MAIN_BATT, symbol Device:LED
- added D?: 12VP, symbol Device:LED
- added D?: 12V, symbol Device:LED
- added D?: 5V, symbol Device:LED
- added D?: 3.3V, symbol Device:LED
- added R? (x2): 10k, Mizz_lib:1608_WP, symbol Device:R
- added R? (x2): 4.7k, Mizz_lib:1608_WP, symbol Device:R
- added R?: 2.2k, Mizz_lib:1608_WP, symbol Device:R
- added R? (x2): 510, Mizz_lib:1608_WP, symbol Device:R
- added R?: 1k, Mizz_lib:1608_WP, symbol Device:R
- added R?: 1.2k, Mizz_lib:1608_WP, symbol Device:R
- added R?: 330, Mizz_lib:1608_WP, symbol Device:R
- added U10, U11, U6: ACS758, Mizz_lib:ACS785xCB, symbol Miz:ACS758
- added U?: MAX3051, symbol Interface_UART:MAX3051
- added U?: AQM0802, symbol Miz:AQM1602
- added U?: SI8900, symbol Miz:SI8900
- added U?: TLP291, Package_SO:SOIC-4_4.55x2.6mm_P1.27mm, symbol Isolator:TLP291
- added U?: BD33FA1, symbol Miz:BD33FA1
- R39, R40, R41, R42, R43, R44: value 1 -> 10
Connections:
- net Earth is gone; now on net GND: C10.2, C9.2, J2.1 (Pin_1), J3.1 (Pin_1)
- net +12P: now also C?.1, R?.2, U?.3 (Vcc); no longer D3.2 (A)
- net +12V: now also D3.2 (A), R?.2
- net +3.3VP: now also C?.1, R?.1, R?.2, U?.1 (Vo)
- net +3V3: now also C?.2, C?.2, R?.2, R?.2, R?.2, U10.1 (VCC), U11.1 (VCC), U6.1 (VCC), U?.5 (VDD), U?.9 (/RST)
- net +5V: now also R?.2
- net +BATT: now also R?.2
- net +Batt: now also R?.2
- net ADRESS_0: now also U3.37 (PC6/TIM8_CH1/USART6_TX/TIM3_CH1); no longer U3.29 (USART3_TX/TIM2_CH3/PB10)
- net ADRESS_1: now also U3.38 (PC7/TIM8_CH2/USART6_RX/TIM3_CH2); no longer U3.30 (USART3_RX/TIM2_CH4/PB11)
- net ADRESS_2: now also U3.39 (PC8/TIM8_CH3/TIM3_CH3); no longer U3.33 (CAN2_RX/PB12)
- net ADRESS_3: now also U3.40 (PC9/TIM8_CH4/TIM3_CH4); no longer U3.34 (TIM1_CH1N/CAN2_TX/PB13)
- net CAN1_RX: now also U?.4 (RXD)
- net CAN1_TX: now also U?.1 (TXD)
- net CAN_H: now also U?.7 (CANH)
- net CAN_L: now also U?.6 (CANL)
- net GND: now also SW1.1, SW2.1, C?.1, D?.1 (K), D?.1 (K), D?.1 (K), U10.2 (GND), U11.2 (GND), U6.2 (GND), U?.6 (VSS); no longer C37.2, C39.2, C41.2, C44.1, C45.1, C46.1, C49.2, C51.2, C52.2, C53.2, C54.2, C55.2, C57.2, D14.2 (A), J10.1 (Pin_1), J8.1 (Pin_1), J9.1 (Pin_1), R46.2, R49.2, R51.2, R53.2, U15.2 (GND), U16.11 (REFSEL), U16.12 (GND), U16.6 (GND), U17.11 (REFSEL), U17.12 (GND), U17.6 (GND), U7.9 (GNCB), U8.9 (GNCB), U9.9 (GNCB)
- net OUT_U_Current: no longer Q2.S
- net at Q4.S: now also U10.4 (IP+)
- net at R30.1: now also U10.3 (VIOUT)
- net GNDPWR: now reaches C48.2, C50.2, C56.2, C58.2
- net GNDPWR: now also C37.2, C39.2, C41.2, C44.1, C45.1, C46.1, C49.2, C51.2, C52.2, C53.2, C54.2, C55.2, C57.2, D14.2 (A), J10.1 (Pin_1), J8.1 (Pin_1), J9.1 (Pin_1), R46.2, R49.2, R51.2, R53.2, U15.2 (GND), U16.11 (REFSEL), U16.12 (GND), U16.6 (GND), U17.11 (REFSEL), U17.12 (GND), U17.6 (GND), U7.9 (GNCB), U8.9 (GNCB), U9.9 (GNCB), C?.2, C?.2, D?.1 (K), D?.1 (K), D?.1 (K), D?.1 (K), U10.5 (IP-), U11.5 (IP-), U6.5 (IP-), U?.2 (GND)
- net at Q6.S: now also U11.4 (IP+)
- net at R31.1: now also U11.3 (VIOUT)
- net at R29.1: now also U6.3 (VIOUT)
- new net: Q2.S, U6.4 (IP+)
- new net: C?.1, U?.2 (VOUT)
- new net: C?.1, U?.3 (CAP1N)
- new net: C?.2, U?.4 (CAP1P)
- new net: D?.2 (A), R?.1 (x7)
- new net I2C2_SCL: R?.1, U3.29 (USART3_TX/TIM2_CH3/PB10), U?.8 (SCL)
- new net I2C2_SDA: R?.1, U3.30 (USART3_RX/TIM2_CH4/PB11), U?.7 (SDA)
- no-connect marks 13 -> 14
Other:
- moved on the sheet: C10, J3
