File: CAN_Current_Control_MD/CAN_Current_Control_MD.sch (KiCad schematic (older format))
At the start: 70 parts

Commit message: 電流制御MDをだいぶ進めた
Parts:
- added C1, C10, C19, C22, C37, C42, C54, C6, C9: 0.1u, Capacitor_SMD:C_0603_1608Metric, symbol Device:C
- added C17: 10u, Capacitor_SMD:C_0603_1608Metric, symbol Device:C
- added C18: 22u, Capacitor_SMD:C_0603_1608Metric, symbol Device:C
- added C2, C25, C47, C5, C52, C53: 4.7u, Capacitor_SMD:C_0805_2012Metric, symbol Device:C
- added C20, C21, C23, C24, C28, C31, C32, C33, C34, C35, C36: 0.1u, Mizz_lib:1608_WP, symbol Device:C
- added C26, C27: 1u, Mizz_lib:1608_WP, symbol Device:C
- added C29, C49: 10u, Capacitor_SMD:C_0805_2012Metric, symbol Device:C
- added C30, C48, C50: 100u, Capacitor_THT:CP_Radial_D5.0mm_P2.50mm, symbol Device:CP1
- added C51: 1500u, Mizz_lib:C_Radial_D13mm_H25.0mm_P5.00mm, symbol Device:CP1
- added D1: 12V, Mizz_lib:1608_WP, symbol Device:LED
- added D10: BUS0, LED_SMD:LED_0603_1608Metric, symbol Device:LED
- added D11, D14, D15, D16, D21, D22, D24, D26: DIODE, Diode_SMD:D_SOD-123, symbol Miz:DIODE_rev
- added D12: EMG1, LED_SMD:LED_0603_1608Metric, symbol Device:LED
- added D13: BUS1, LED_SMD:LED_0603_1608Metric, symbol Device:LED
- added D2: 3V3, Mizz_lib:1608_WP, symbol Device:LED
- added D23: DIODE, Diode_SMD:D_SMA, symbol Miz:PWR_DIODE
- added D25: VALVE0, LED_SMD:LED_0603_1608Metric, symbol Device:LED
- added D27: VALVE1, LED_SMD:LED_0603_1608Metric, symbol Device:LED
- added D4: BATT, LED_SMD:LED_0603_1608Metric, symbol Device:LED
- added D5: MAIN_BATT, LED_SMD:LED_0603_1608Metric, symbol Device:LED
- added D6: 12VP, LED_SMD:LED_0603_1608Metric, symbol Device:LED
- added D7: 5VP, LED_SMD:LED_0603_1608Metric, symbol Device:LED
- added D8: 3V3P, LED_SMD:LED_0603_1608Metric, symbol Device:LED
- added D9: EMG0, LED_SMD:LED_0603_1608Metric, symbol Device:LED
- added F1: Polyfuse, symbol Device:Polyfuse
- added J10: FAN, Mizz_lib:XA_2P, symbol Connector_Generic:Conn_01x02
- added J13: VALVE, Mizz_lib:XA_4L, symbol Connector_Generic:Conn_01x04
- added J3: CAN, Mizz_lib:XA_4L, symbol Connector_Generic:Conn_01x04
- added J4: ENC0, Mizz_lib:XA_4L, symbol Connector_Generic:Conn_01x04
- added J5: ENC1, Mizz_lib:XA_4L, symbol Connector_Generic:Conn_01x04
- added J6: I/O_0, Mizz_lib:XA_3L, symbol Connector_Generic:Conn_01x03
- added J7: I/O_1, Mizz_lib:XA_3L, symbol Connector_Generic:Conn_01x03
- added JP2: CAN_JP, Connector_PinHeader_2.54mm:PinHeader_1x02_P2.54mm_Vertical, symbol Device:Jumper
- added JP3: I/O_Vdd, Connector_PinHeader_2.54mm:PinHeader_1x03_P2.54mm_Vertical, symbol Device:Jumper_NC_Dual
- added L1, L2: 22uH, Mizz_lib:Inductor_Taiyo-Yuden_NR-50xx_HandSoldering, symbol Device:L_Small
- added Q10, Q9: NPN, Package_TO_SOT_SMD:SOT-23, symbol Device:Q_NPN_BEC
- added R1: 2.2k, Mizz_lib:1608_WP, symbol Device:R
- added R10, R8: 10k, Resistor_SMD:R_0603_1608Metric, symbol Device:R
- added R11, R12, R13, R14: 240, Resistor_SMD:R_0603_1608Metric, symbol Device:R
- added R15: 120, Resistor_SMD:R_0603_1608Metric, symbol Device:R
- added R16, R17, R18, R19, R30, R32, R33, R34, R35, R36, R37, R38, R39: 10k, Mizz_lib:1608_WP, symbol Device:R
- added R2: 510, Mizz_lib:1608_WP, symbol Device:R
- added R20, R21, R22, R23: 4.7k, Mizz_lib:1608_WP, symbol Device:R
- added R24, R25, R26, R27: 1k, Mizz_lib:1608_WP, symbol Device:R
- added R28: 3.9k, Resistor_SMD:R_0603_1608Metric, symbol Device:R
- added R29: 680, Resistor_SMD:R_0603_1608Metric, symbol Device:R
- added R3, R4: 4.7k, Resistor_SMD:R_0603_1608Metric, symbol Device:R
- added R48: 7.5k, Resistor_SMD:R_0603_1608Metric, symbol Device:R
- added R49, R6: 510, Resistor_SMD:R_0603_1608Metric, symbol Device:R
- added R5: 2.2k, Resistor_SMD:R_0603_1608Metric, symbol Device:R
- added R62: 47, Mizz_lib:R_2812, symbol Device:R
- added R63, R64: 330, Mizz_lib:1608_WP, symbol Device:R
- added R7: 330, Resistor_SMD:R_0603_1608Metric, symbol Device:R
- added SW1: SW0, Button_Switch_SMD:SW_SPST_CK_RS282G05A3, symbol Switch:SW_Push
- added SW2: SW1, Button_Switch_SMD:SW_SPST_CK_RS282G05A3, symbol Switch:SW_Push
- added SW3: RST, Button_Switch_SMD:SW_SPST_CK_RS282G05A3, symbol Switch:SW_Push
- added TH1, TH2, TH3, TH4, TH5: Thermistor, Mizz_lib:1608_WP, symbol Device:Thermistor
- added U1: BD33FA1, Package_TO_SOT_SMD:SOT-89-3, symbol Miz:BD33FA1
- added U12, U6: BD9G101G, Package_SO:TSOP-6_1.65x3.05mm_P0.95mm, symbol Miz:BD9G101G
- added U4: ADRESS, Mizz_lib:rotary_0F, symbol Miz:SW_ROTARY_16
- added U5: AZ1086H, Package_TO_SOT_SMD:SOT-223-3_TabPin2, symbol Miz:AZ1086H
- added U7: AQM0802, Mizz_lib:AQM0802_original, symbol Miz:AQM1602
- C11, C12, C13, C14, C15, C16, C3, C4, C7, C8: renamed from C?; footprint (none) -> Capacitor_SMD:C_0603_1608Metric
- C38, C39, C40, C41: renamed from C?; footprint (none) -> Mizz_lib:1608_WP
- C43, C44, C45, C46: renamed from C?; footprint (none) -> Capacitor_SMD:C_0805_2012Metric
- D17, D18, D19, D20, D3: renamed from D?; footprint (none) -> Diode_SMD:D_SOD-123
- J1: renamed from J?; footprint (none) -> Mizz_lib:ZH_6P
- J11, J12, J8: renamed from J?; footprint (none) -> Mizz_lib:XT60_F
- J2: renamed from J?; footprint (none) -> Mizz_lib:XA_4L
- J9: renamed from J?; footprint (none) -> Mizz_lib:XT60_M
- JP1: renamed from JP?; footprint (none) -> Jumper:SolderJumper-2_P1.3mm_Open_TrianglePad1.0x1.5mm
- Q1, Q2, Q3, Q4, Q5, Q6, Q7, Q8: renamed from Q?; footprint (none) -> Mizz_lib:D2-PAK_compact
- R31, R50, R51, R52, R53, R54, R55, R56, R57, R9: renamed from R?; footprint (none) -> Resistor_SMD:R_0603_1608Metric
- R40, R41, R42, R43, R44, R45, R46, R47: renamed from R?; footprint (none) -> Mizz_lib:1608_WP
- R58, R59, R60, R61: renamed from R?; value 200uOhm -> 2m; footprint (none) -> Mizz_lib:R_2010_5025Metric
- U10, U11, U8, U9: renamed from U?; footprint (none) -> Package_SO:SOIC-8_3.9x4.9mm_P1.27mm
- U15: renamed from U?; footprint (none) -> Mizz_lib:Mini_Monster
- U3: renamed from U?; footprint LQFP64 -> Package_QFP:LQFP-64_10x10mm_P0.5mm
- Y1: renamed from Y?; footprint (none) -> Mizz_lib:Crystal_SMD_5032_2Pads
- gave numbers to parts that had none: 3
Connections:
- net +12P: now also C25.1, C50.1, D22.1 (K), J13.2 (Pin_2), J13.4 (Pin_4), R5.2, U6.4 (EN), U6.5 (VCC)
- net +3.3VP: now also R31.1, C26.2, C28.2, C6.1, D14.1 (K), JP3.1, R30.2, R32.2, R7.2, TH1.1, TH2.1, TH3.1, TH4.1, TH5.1, U7.5 (VDD), U7.9 (/RST)
- net +3V3: now also C1.1, C5.1, R2.2, U1.1 (Vo)
- net +BATT: now also C51.1, C52.1, C53.1, D23.2 (A), R3.2
- net CAN1_RX: now also U3.61 (TIM4_CH3/TIM10_CH1/CAN1_RX/PB8)
- net CAN1_TX: now also U3.62 (TIM4_CH4/TIM11_CH1/CAN1_TX/PB9)
- net Current0_Analog: now also U3.11 (PC3/ADC12_IN13)
- net Current1_Analog: now also U3.10 (PC2/ADC12_IN12)
- net GND: now also J2.1 (Pin_1), C1.2, C10.1, C2.2, C5.2, C9.1, D1.1 (K), D2.1 (K), J3.1 (Pin_1), U1.2 (GND)
- net GNDPWR: now also C17.2, C18.2, C19.2, C20.1, C21.1, C23.1, C24.1, C25.2, C28.1, C29.2, C30.2, C31.2, C32.2, C33.2, C34.2, C35.2, C36.2, C37.2, C47.2, C48.2, C49.2, C50.2, C51.2, C52.2, C53.2, C54.2, C6.2, D10.1 (K), D12.1 (K), D13.1 (K), D15.2 (A), D21.2 (A), D24.2 (A), D25.1 (K), D26.2 (A), D27.1 (K), D4.1 (K), D5.1 (K), D6.1 (K), D7.1 (K), D8.1 (K), D9.1 (K), J10.1 (Pin_1), J4.1 (Pin_1), J5.1 (Pin_1), J6.1 (Pin_1), J7.1 (Pin_1), Q10.2 (E), Q9.2 (E), R16.1, R17.1, R18.1, R19.1, R29.2, R33.2, R34.2, R35.2, R37.2, R38.2, R39.2, R49.2, SW1.1, SW2.1, SW3.1, U12.2 (GND), U4.2 (C), U4.5 (C), U5.1 (GND), U6.2 (GND), U7.6 (VSS)
- net PWM0L: now also U3.38 (PC7/TIM8_CH2/USART6_RX/TIM3_CH2); no longer U9.2 (IN)
- net PWM1L: now also U3.36 (TIM1_CH3N/TIM8_CH3N/TIM12_CH2/PB15); no longer U11.2 (IN)
- net SWCLK: now also U3.49 (SWCLK/PA14)
- net SWDIO: now also U3.46 (SWDIO/PA13)
- net ~RST: now also C54.1, SW3.2
- net BATTERY_VOLTAGE: now reaches U3.15 (UART4_RX/ADC12_IN1/TIM5_CH2/TIM2_CH2/PA1)
- net BATTERY_VOLTAGE: now also C34.1, R36.2, R37.1
- net IO_0: now reaches U3.2 (PC13)
- net IO_0: now also J6.3 (Pin_3)
- net Substrate_Temp: now reaches U3.20 (ADC12_IN4/PA4)
- net Substrate_Temp: now also C31.1, R33.1, TH1.2
- net ADRESS_4: now reaches U3.21 (ADC12_IN5/TIM2_CH1_ETR/TIM8_CH1N/PA5)
- net ADRESS_4: now also U4.4
- net ADRESS_8: now reaches U3.22 (ADC12_IN6/TIM3_CH1/TIM13_CH1/PA6)
- net ADRESS_8: now also U4.6 (8)
- net ADRESS_1: now reaches U3.23 (ADC12_IN7/TIM1_CH1N/TIM8_CH1N/TIM14_CH1/TIM3_CH2/PA7)
- net ADRESS_1: now also U4.3 (1)
- net MD1R_Temp: now reaches U3.25 (PC5/ADC12_IN15)
- net MD1R_Temp: now also C36.1, R39.1, TH5.2
- net MD1L_Temp: now reaches U3.26 (ADC12_IN8/TIM1_CH2N/TIM8_CH2N/TIM3_CH3/PB0)
- net MD1L_Temp: now also C33.1, R35.1, TH3.2
- net ADRESS_2: now reaches U3.27 (ADC12_IN9/TIM1_CH3N/TIM8_CH3N/TIM3_CH4/PB1)
- net ADRESS_2: now also U4.1 (2)
- net at U3.28 (BOOT1/PB2): now also R31.2
- net I2C2_SCL: now reaches U3.29 (USART3_TX/TIM2_CH3/PB10)
- net I2C2_SCL: now also R30.1, U7.8 (SCL)
- net IO_1: now reaches U3.3 (PC14/OSC32_IN)
- net IO_1: now also J7.3 (Pin_3)
- net I2C2_SDA: now reaches U3.30 (USART3_RX/TIM2_CH4/PB11)
- net I2C2_SDA: now also R32.1, U7.7 (SDA)
- net EN1: now reaches U3.34 (TIM1_CH1N/CAN2_TX/PB13)
- net EN1: now also R45.1, R47.1, U10.3 (~SD), U11.3 (~SD)
- net PWM1R: now reaches U3.35 (TIM1_CH2N/TIM8_CH2N/TIM12_CH1/PB14)
- net PWM1R: now also U11.2 (IN)
- net EN0: now reaches U3.37 (PC6/TIM8_CH1/USART6_TX/TIM3_CH1)
- net EN0: now also R41.1, R43.1, U8.3 (~SD), U9.3 (~SD)
- net PWM0R: now reaches U3.39 (PC8/TIM8_CH3/TIM3_CH3)
- net PWM0R: now also U9.2 (IN)
- net SW1: now reaches U3.40 (PC9/TIM8_CH4/TIM3_CH4)
- net SW1: now also R10.2, SW2.2
- net SW0: now reaches U3.41 (TIM1_CH1/PA8)
- net SW0: now also R8.2, SW1.2
- net USART1_TX: now reaches U3.42 (USART1_TX/TIM1_CH2/PA9)
- net USART1_RX: now reaches U3.43 (USART1_RX/TIM1_CH3/PA10)
- net LED0: now reaches U3.52 (PC11/UART4_RX/USART3_RX)
- net LED0: now also R11.1
- net LED1: now reaches U3.53 (PC12/UART5_TX)
- net LED1: now also R12.1
- net LED2: now reaches U3.54 (PD2/UART5_RX)
- net LED2: now also R13.1
- net LED3: now reaches U3.55 (TIM2_CH2/PB3)
- net LED3: now also R14.1
- net TIM3_CH1: now reaches U3.56 (TIM3_CH1/PB4)
- net TIM3_CH1: now also R16.2, R20.2
- net TIM3_CH2: now reaches U3.57 (CAN2_RX/TIM3_CH2/PB5)
- net TIM3_CH2: now also R18.2, R22.2
- net TIM4_CH1: now reaches U3.58 (TIM4_CH1/CAN2_TX/USART1_TX/PB6)
- net TIM4_CH1: now also R17.2, R21.2
- net TIM4_CH2: now reaches U3.59 (USART1_RX/TIM4_CH2/PB7)
- net TIM4_CH2: now also R19.2, R23.2
- net MD0R_Temp: now reaches U3.8 (PC0/ADC12_IN10)
- net MD0R_Temp: now also C35.1, R38.1, TH4.2
- net MD0L_Temp: now reaches U3.9 (PC1/ADC12_IN11)
- net MD0L_Temp: now also C32.1, R34.1, TH2.2
- net CAN_L: now reaches U2.6 (CANL)
- net CAN_L: now also J2.4 (Pin_4), J3.4 (Pin_4), R15.1
- net CAN_H: now reaches U2.7 (CANH)
- net CAN_H: now also J2.3 (Pin_3), J3.3 (Pin_3), JP2.1
- net at J2.2 (Pin_2): now also C10.2, C9.2, D11.2 (A), J3.2 (Pin_2)
- new net: D16.1 (K), F1.2
- new net: C22.2, U6.1 (BST)
- new net: C19.1, R28.2, R29.1, U6.3 (FB)
- new net: C22.1, D15.1 (K), L1.1, U6.6 (Lx)
- new net: C42.2, U12.1 (BST)
- new net: C37.1, R48.2, R49.1, U12.3 (FB)
- new net: C42.1, D21.1 (K), L2.1, U12.6 (Lx)
- new net: J10.2 (Pin_2), R62.1
- new net: C18.1, D14.2 (A), U5.2 (V_OUT)
- new net: C26.1, U7.2 (VOUT)
- new net: C27.1, U7.3 (CAP1N)
- new net: C27.2, U7.4 (CAP1P)
- new net: J4.3 (Pin_3), R22.1, R26.1
- new net: J4.4 (Pin_4), R20.1, R24.1
- new net: D9.2 (A), R11.2
- new net: D10.2 (A), R12.2
- new net: D12.2 (A), R13.2
- new net: D13.2 (A), R14.2
- new net: JP2.2, R15.2
- new net: C23.2, C24.2, J6.2 (Pin_2), J7.2 (Pin_2), JP3.2
- new net: J5.3 (Pin_3), R23.1, R27.1
- new net: J5.4 (Pin_4), R21.1, R25.1
- new net: D4.2 (A), R3.1
- new net: D5.2 (A), R4.1
- new net: D6.2 (A), R5.1
- new net: D7.2 (A), R6.1
- new net: D8.2 (A), R7.1
- new net: D1.2 (A), R1.1
- new net: D2.2 (A), R2.1
- new net: D24.1 (K), J13.1 (Pin_1), Q9.3 (C)
- new net: D26.1 (K), J13.3 (Pin_3), Q10.3 (C)
- new net: D25.2 (A), R63.2
- new net: D27.2 (A), R64.2
- new net +12V: C2.1, D11.1 (K), R1.2, U1.3 (Vcc)
- new net +5VP: C17.1, C20.2, C21.2, F1.1, J4.2 (Pin_2), J5.2 (Pin_2), JP3.3, R10.1, R24.2, R25.2, R26.2, R27.2, R6.2, R8.1, U5.3 (V_IN)
- new net Batt: C47.1, C48.1, D23.1 (K), R36.1, R4.2, R62.2, U12.4 (EN), U12.5 (VCC)
- new net FB_12V: C49.1, D22.2 (A), L2.2, R48.1
- new net FB_5V: C29.1, C30.1, D16.2 (A), L1.2, R28.1
- new net VALVE0: Q9.1 (B), R63.1
- new net VALVE1: Q10.1 (B), R64.1
- no-connect marks 1 -> 2
Other:
- note added: "PolyFuse : http://akizukidenshi.com/catalog/g/gP-13955/"
- moved on the sheet: C38, C39, C40, C41, C43, C44, C45, C46, D17, D18, D19, D20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

Commit message: ぶざーてすときばんは頭悪い
Parts:
- R37: value 10k -> 1k
Connections:
- net +12P: now also D6.2 (A); no longer R5.2
- net GNDPWR: now also R5.1; no longer D6.1 (K)
- new net: D6.1 (K), R5.2
Other:
- moved on the sheet: D6, R5
Changed lines of the file:
@@
 P 8975 2625
 F 0 "R37" H 9045 2671 50  0000 L CNN
-F 1 "10k" H 9045 2580 50  0000 L CNN
+F 1 "1k" H 9045 2580 50  0000 L CNN
 F 2 "Mizz_lib:1608_WP" V 8905 2625 50  0001 C CNN
 F 3 "~" H 8975 2625 50  0001 C CNN
@@
 L Device:R R5
 U 1 1 5F1F4ACD
-P 1275 1400
-F 0 "R5" V 1068 1400 50  0000 C CNN
-F 1 "2.2k" V 1159 1400 50  0000 C CNN
-F 2 "Resistor_SMD:R_0603_1608Metric" V 1205 1400 50  0001 C CNN
-F 3 "~" H 1275 1400 50  0001 C CNN
-	1    1275 1400
+P 1575 1400
+F 0 "R5" V 1368 1400 50  0000 C CNN
+F 1 "2.2k" V 1459 1400 50  0000 C CNN
+F 2 "Resistor_SMD:R_0603_1608Metric" V 1505 1400 50  0001 C CNN
+F 3 "~" H 1575 1400 50  0001 C CNN
+	1    1575 1400
 	0    1    1    0
 $EndComp
@@
 L Device:LED D6
 U 1 1 5F20B9AE
-P 1575 1400
-F 0 "D6" H 1568 1145 50  0000 C CNN
-F 1 "12VP" H 1568 1236 50  0000 C CNN
-F 2 "LED_SMD:LED_0603_1608Metric" H 1575 1400 50  0001 C CNN
-F 3 "~" H 1575 1400 50  0001 C CNN
-	1    1575 1400
+P 1275 1400
+F 0 "D6" H 1268 1145 50  0000 C CNN
+F 1 "12VP" H 1268 1236 50  0000 C CNN
+F 2 "LED_SMD:LED_0603_1608Metric" H 1275 1400 50  0001 C CNN
+F 3 "~" H 1275 1400 50  0001 C CNN
+	1    1275 1400
 	-1   0    0    1
 $EndComp

Commit message: 配置しただけで分かるやばいやつ
Parts:
- added C55, C56: 0.1u, Mizz_lib:1608_WP, symbol Device:C
- C1, C11, C12, C13, C14, C15, C16, C17, C18, C19, C22, C3, C4, C42, C8: footprint Capacitor_SMD:C_0603_1608Metric -> Mizz_lib:1608_WP
- F1: footprint (none) -> Fuse:Fuse_1812_4532Metric_Pad1.30x3.40mm_HandSolder
Connections:
- net +3.3VP: now also C55.1, C56.1
- net GNDPWR: now also C55.2, C56.2
Other:
- note added: "PolyFuse : http://akizukidenshi.com/catalog/g/gP-10074/"
- note removed: "PolyFuse : http://akizukidenshi.com/catalog/g/gP-13955/"
Changed lines of the file:
@@
 F 0 "C16" H 4640 6771 50  0000 L CNN
 F 1 "2.2u" H 4640 6680 50  0000 L CNN
-F 2 "Capacitor_SMD:C_0603_1608Metric" H 4563 6575 50  0001 C CNN
+F 2 "Mizz_lib:1608_WP" H 4563 6575 50  0001 C CNN
 F 3 "~" H 4525 6725 50  0001 C CNN
 	1    4525 6725
@@
 F 0 "C14" H 4490 6771 50  0000 L CNN
 F 1 "2.2u" H 4490 6680 50  0000 L CNN
-F 2 "Capacitor_SMD:C_0603_1608Metric" H 4413 6575 50  0001 C CNN
+F 2 "Mizz_lib:1608_WP" H 4413 6575 50  0001 C CNN
 F 3 "~" H 4375 6725 50  0001 C CNN
 	1    4375 6725
@@
 F 0 "C8" H 3090 2071 50  0000 L CNN
 F 1 "0.1u" H 3090 1980 50  0000 L CNN
-F 2 "Capacitor_SMD:C_0603_1608Metric" H 3013 1875 50  0001 C CNN
+F 2 "Mizz_lib:1608_WP" H 3013 1875 50  0001 C CNN
 F 3 "~" H 2975 2025 50  0001 C CNN
 	1    2975 2025
@@
 F 0 "C11" H 3465 2071 50  0000 L CNN
 F 1 "0.1u" H 3465 1980 50  0000 L CNN
-F 2 "Capacitor_SMD:C_0603_1608Metric" H 3388 1875 50  0001 C CNN
+F 2 "Mizz_lib:1608_WP" H 3388 1875 50  0001 C CNN
 F 3 "~" H 3350 2025 50  0001 C CNN
 	1    3350 2025
@@
 F 0 "C12" H 3840 2071 50  0000 L CNN
 F 1 "0.1u" H 3840 1980 50  0000 L CNN
-F 2 "Capacitor_SMD:C_0603_1608Metric" H 3763 1875 50  0001 C CNN
+F 2 "Mizz_lib:1608_WP" H 3763 1875 50  0001 C CNN
 F 3 "~" H 3725 2025 50  0001 C CNN
 	1    3725 2025
@@
 F 0 "C13" H 4215 2071 50  0000 L CNN
 F 1 "1u" H 4215 1980 50  0000 L CNN
-F 2 "Capacitor_SMD:C_0603_1608Metric" H 4138 1875 50  0001 C CNN
+F 2 "Mizz_lib:1608_WP" H 4138 1875 50  0001 C CNN
 F 3 "~" H 4100 2025 50  0001 C CNN
 	1    4100 2025
@@
 F 0 "C15" H 4590 2071 50  0000 L CNN
 F 1 "4.7u" H 4590 1980 50  0000 L CNN
-F 2 "Capacitor_SMD:C_0603_1608Metric" H 4513 1875 50  0001 C CNN
+F 2 "Mizz_lib:1608_WP" H 4513 1875 50  0001 C CNN
 F 3 "~" H 4475 2025 50  0001 C CNN
 	1    4475 2025
@@
 F 0 "C3" H 1065 2996 50  0000 L CNN
 F 1 "22p" H 1065 2905 50  0000 L CNN
-F 2 "Capacitor_SMD:C_0603_1608Metric" H 988 2800 50  0001 C CNN
+F 2 "Mizz_lib:1608_WP" H 988 2800 50  0001 C CNN
 F 3 "~" H 950 2950 50  0001 C CNN
 	1    950  2950
@@
 F 0 "C4" H 1415 2996 50  0000 L CNN
 F 1 "22p" H 1415 2905 50  0000 L CNN
-F 2 "Capacitor_SMD:C_0603_1608Metric" H 1338 2800 50  0001 C CNN
+F 2 "Mizz_lib:1608_WP" H 1338 2800 50  0001 C CNN
 F 3 "~" H 1300 2950 50  0001 C CNN
 	1    1300 2950
@@
 F 0 "C42" V 10873 900 50  0000 C CNN
 F 1 "0.1u" V 10964 900 50  0000 C CNN
-F 2 "Capacitor_SMD:C_0603_1608Metric" H 11163 750 50  0001 C CNN
+F 2 "Mizz_lib:1608_WP" H 11163 750 50  0001 C CNN
 F 3 "~" H 11125 900 50  0001 C CNN
 	1    11125 900
@@
 F 0 "C22" V 6848 875 50  0000 C CNN
 F 1 "0.1u" V 6939 875 50  0000 C CNN
-F 2 "Capacitor_SMD:C_0603_1608Metric" H 7138 725 50  0001 C CNN
+F 2 "Mizz_lib:1608_WP" H 7138 725 50  0001 C CNN
 F 3 "~" H 7100 875 50  0001 C CNN
 	1    7100 875
@@
 F 0 "C19" H 6265 1696 50  0000 L CNN
 F 1 "0.1u" H 6265 1605 50  0000 L CNN
-F 2 "Capacitor_SMD:C_0603_1608Metric" H 6188 1500 50  0001 C CNN
+F 2 "Mizz_lib:1608_WP" H 6188 1500 50  0001 C CNN
 F 3 "~" H 6150 1650 50  0001 C CNN
 	1    6150 1650
@@
 F 0 "F1" V 8650 1300 50  0000 C CNN
 F 1 "Polyfuse" V 8741 1300 50  0000 C CNN
-F 2 "" H 8925 1100 50  0001 L CNN
+F 2 "Fuse:Fuse_1812_4532Metric_Pad1.30x3.40mm_HandSolder" H 8925 1100 50  0001 L CNN
 F 3 "~" H 8875 1300 50  0001 C CNN
 	1    8875 1300
@@
 	7825 1400 7625 1400
 Text Notes 8275 1000 0    50   ~ 0
-PolyFuse : http://akizukidenshi.com/catalog/g/gP-13955/
+PolyFuse : http://akizukidenshi.com/catalog/g/gP-10074/
 $Comp
 L Miz:AZ1086H U5
@@
 F 0 "C17" H 4840 1296 50  0000 L CNN
 F 1 "10u" H 4840 1205 50  0000 L CNN
-F 2 "Capacitor_SMD:C_0603_1608Metric" H 4763 1100 50  0001 C CNN
+F 2 "Mizz_lib:1608_WP" H 4763 1100 50  0001 C CNN
 F 3 "~" H 4725 1250 50  0001 C CNN
 	1    4725 1250
@@
 F 0 "C18" H 5740 1296 50  0000 L CNN
 F 1 "22u" H 5740 1205 50  0000 L CNN
-F 2 "Capacitor_SMD:C_0603_1608Metric" H 5663 1100 50  0001 C CNN
+F 2 "Mizz_lib:1608_WP" H 5663 1100 50  0001 C CNN
 F 3 "~" H 5625 1250 50  0001 C CNN
 	1    5625 1250
@@
 F 0 "C1" H 940 7646 50  0000 L CNN
 F 1 "0.1u" H 940 7555 50  0000 L CNN
-F 2 "Capacitor_SMD:C_0603_1608Metric" H 863 7450 50  0001 C CNN
+F 2 "Mizz_lib:1608_WP" H 863 7450 50  0001 C CNN
 F 3 "~" H 825 7600 50  0001 C CNN
 	1    825  7600
@@
 $EndComp
 Connection ~ 6825 10425
+$Comp
+L power:+3.3VP #PWR0214
+U 1 1 5E6A2DA9
+P 14100 4800
+F 0 "#PWR0214" H 14250 4750 50  0001 C CNN
+F 1 "+3.3VP" H 14120 4943 50  0000 C CNN
+F 2 "" H 14100 4800 50  0001 C CNN
+F 3 "" H 14100 4800 50  0001 C CNN
+	1    14100 4800
+	1    0    0    -1
+$EndComp
+$Comp
+L power:GNDPWR #PWR0215
+U 1 1 5E6A31A1
+P 14100 5100
+F 0 "#PWR0215" H 14100 4900 50  0001 C CNN
+F 1 "GNDPWR" H 14104 4946 50  0000 C CNN
+F 2 "" H 14100 5050 50  0001 C CNN
+F 3 "" H 14100 5050 50  0001 C CNN
+	1    14100 5100
+	1    0    0    -1
+$EndComp
+$Comp
+L power:+3.3VP #PWR0216
+U 1 1 5E6A4880
+P 14100 8275
+F 0 "#PWR0216" H 14250 8225 50  0001 C CNN
+F 1 "+3.3VP" H 14120 8418 50  0000 C CNN
+F 2 "" H 14100 8275 50  0001 C CNN
+F 3 "" H 14100 8275 50  0001 C CNN
+	1    14100 8275
+	1    0    0    -1
+$EndComp
+$Comp
+L power:GNDPWR #PWR0217
+U 1 1 5E6A488A
+P 14100 8575
+F 0 "#PWR0217" H 14100 8375 50  0001 C CNN
+F 1 "GNDPWR" H 14104 8421 50  0000 C CNN
+F 2 "" H 14100 8525 50  0001 C CNN
+F 3 "" H 14100 8525 50  0001 C CNN
+	1    14100 8575
+	1    0    0    -1
+$EndComp
+$Comp
+L Device:C C56
+U 1 1 5E6E5792
+P 14100 8425
+F 0 "C56" H 14215 8471 50  0000 L CNN
+F 1 "0.1u" H 14215 8380 50  0000 L CNN
+F 2 "Mizz_lib:1608_WP" H 14138 8275 50  0001 C CNN
+F 3 "~" H 14100 8425 50  0001 C CNN
+	1    14100 8425
+	1    0    0    -1
+$EndComp
+$Comp
+L Device:C C55
+U 1 1 5E6E8E7D
+P 14100 4950
+F 0 "C55" H 14215 4996 50  0000 L CNN
+F 1 "0.1u" H 14215 4905 50  0000 L CNN
+F 2 "Mizz_lib:1608_WP" H 14138 4800 50  0001 C CNN
+F 3 "~" H 14100 4950 50  0001 C CNN
+	1    14100 4950
+	1    0    0    -1
+$EndComp
 $EndSCHEMATC
