File: CAN_Current_Control_MD/CAN_Current_Control_MD.sch (KiCad schematic (older format))
At the start: 200 parts, among them J1 SWD, J10 FAN, J11 OUT_0, J12 OUT_1, J13 VALVE, J2 CAN, J3 CAN, J4 ENC0, J5 ENC1, J6 I/O_0, J7 I/O_1, J8 BATT_IN, J9 BATT_IN, Q1 MOSFET_N, Q10 NPN, Q2 MOSFET_N, Q3 MOSFET_N, Q4 MOSFET_N, Q5 MOSFET_N, Q6 MOSFET_N, Q7 MOSFET_N, Q8 MOSFET_N, Q9 NPN, SW1 SW0, SW2 SW1, SW3 RST, U1 BD33FA1, U10 NCP5104, U11 NCP5104, U12 BD9G101G, U13 INA181A1, U14 INA181A1, U15 LOGO, U2 ISO1050DUB, U3 STM32F405RG, U4 ADRESS, U5 AZ1086H, U6 BD9G101G, U7 AQM0802, U8 NCP5104, U9 NCP5104, Y1 8MHz

Commit message: もうちょいで電流制御MDの配線が終わる
Parts:
- D10, D12, D13, D9: footprint LED_SMD:LED_0603_1608Metric -> Mizz_lib:1608_WP
- R6, R7: footprint Resistor_SMD:R_0603_1608Metric -> Mizz_lib:1608_WP
Connections:
- net +3.3VP: now also R11.1, R12.1, R13.1, R14.1
- net Current0_Analog: now also U3.10 (PC2/ADC12_IN12); no longer U3.11 (PC3/ADC12_IN13)
- net Current1_Analog: now also U3.11 (PC3/ADC12_IN13); no longer U3.10 (PC2/ADC12_IN12)
- net GNDPWR: no longer D10.1 (K), D12.1 (K), D13.1 (K), D9.1 (K)
- net LED0: now also D9.1 (K); no longer R11.1
- net LED1: now also D10.1 (K); no longer R12.1
- net LED2: now also D12.1 (K); no longer R13.1
- net LED3: now also D13.1 (K); no longer R14.1
- net PWM0L: now also U3.39 (PC8/TIM8_CH3/TIM3_CH3); no longer U3.38 (PC7/TIM8_CH2/USART6_RX/TIM3_CH2)
- net PWM0R: now also U3.38 (PC7/TIM8_CH2/USART6_RX/TIM3_CH2); no longer U3.39 (PC8/TIM8_CH3/TIM3_CH3)
- net SW0: now also U3.40 (PC9/TIM8_CH4/TIM3_CH4); no longer U3.41 (TIM1_CH1/PA8)
- net SW1: now also U3.41 (TIM1_CH1/PA8); no longer U3.40 (PC9/TIM8_CH4/TIM3_CH4)
- net TIM3_CH1: now also R17.2, R21.2; no longer R16.2, R20.2
- net TIM3_CH2: now also R19.2, R23.2; no longer R18.2, R22.2
- net TIM4_CH1: now also R16.2, R20.2; no longer R17.2, R21.2
- net TIM4_CH2: now also R18.2, R22.2; no longer R19.2, R23.2
Other:
- moved on the sheet: D10, D12, D13, D9, R11, R12, R13, R14
Changed lines of the file:
@@
 L Device:LED D9
 U 1 1 5EA6BE27
-P 2225 10325
-F 0 "D9" V 2264 10208 50  0000 R CNN
-F 1 "EMG0" V 2173 10208 50  0000 R CNN
-F 2 "LED_SMD:LED_0603_1608Metric" H 2225 10325 50  0001 C CNN
-F 3 "~" H 2225 10325 50  0001 C CNN
-	1    2225 10325
+P 2300 10325
+F 0 "D9" V 2339 10208 50  0000 R CNN
+F 1 "EMG0" V 2248 10208 50  0000 R CNN
+F 2 "Mizz_lib:1608_WP" H 2300 10325 50  0001 C CNN
+F 3 "~" H 2300 10325 50  0001 C CNN
+	1    2300 10325
 	0    -1   -1   0
 $EndComp
@@
 L Device:LED D10
 U 1 1 5EA6C9E4
-P 2600 10325
-F 0 "D10" V 2639 10208 50  0000 R CNN
-F 1 "BUS0" V 2548 10208 50  0000 R CNN
-F 2 "LED_SMD:LED_0603_1608Metric" H 2600 10325 50  0001 C CNN
-F 3 "~" H 2600 10325 50  0001 C CNN
-	1    2600 10325
+P 2675 10325
+F 0 "D10" V 2714 10208 50  0000 R CNN
+F 1 "BUS0" V 2623 10208 50  0000 R CNN
+F 2 "Mizz_lib:1608_WP" H 2675 10325 50  0001 C CNN
+F 3 "~" H 2675 10325 50  0001 C CNN
+	1    2675 10325
 	0    -1   -1   0
 $EndComp
@@
 L Device:LED D12
 U 1 1 5EA6D533
-P 2975 10325
-F 0 "D12" V 3014 10208 50  0000 R CNN
-F 1 "EMG1" V 2923 10208 50  0000 R CNN
-F 2 "LED_SMD:LED_0603_1608Metric" H 2975 10325 50  0001 C CNN
-F 3 "~" H 2975 10325 50  0001 C CNN
-	1    2975 10325
+P 3050 10325
+F 0 "D12" V 3089 10208 50  0000 R CNN
+F 1 "EMG1" V 2998 10208 50  0000 R CNN
+F 2 "Mizz_lib:1608_WP" H 3050 10325 50  0001 C CNN
+F 3 "~" H 3050 10325 50  0001 C CNN
+	1    3050 10325
 	0    -1   -1   0
 $EndComp
@@
 L Device:LED D13
 U 1 1 5EA6D53D
-P 3350 10325
-F 0 "D13" V 3389 10208 50  0000 R CNN
-F 1 "BUS1" V 3298 10208 50  0000 R CNN
-F 2 "LED_SMD:LED_0603_1608Metric" H 3350 10325 50  0001 C CNN
-F 3 "~" H 3350 10325 50  0001 C CNN
-	1    3350 10325
+P 3425 10325
+F 0 "D13" V 3464 10208 50  0000 R CNN
+F 1 "BUS1" V 3373 10208 50  0000 R CNN
+F 2 "Mizz_lib:1608_WP" H 3425 10325 50  0001 C CNN
+F 3 "~" H 3425 10325 50  0001 C CNN
+	1    3425 10325
 	0    -1   -1   0
-$EndComp
-$Comp
-L Device:R R11
-U 1 1 5EA7ECE1
-P 2225 10025
-F 0 "R11" H 2295 10071 50  0000 L CNN
-F 1 "240" H 2295 9980 50  0000 L CNN
-F 2 "Resistor_SMD:R_0603_1608Metric" V 2155 10025 50  0001 C CNN
-F 3 "~" H 2225 10025 50  0001 C CNN
-	1    2225 10025
-	1    0    0    -1
-$EndComp
-$Comp
-L Device:R R12
-U 1 1 5EA7F1D4
-P 2600 10025
-F 0 "R12" H 2670 10071 50  0000 L CNN
-F 1 "240" H 2670 9980 50  0000 L CNN
-F 2 "Resistor_SMD:R_0603_1608Metric" V 2530 10025 50  0001 C CNN
-F 3 "~" H 2600 10025 50  0001 C CNN
-	1    2600 10025
-	1    0    0    -1
-$EndComp
-$Comp
-L Device:R R13
-U 1 1 5EA7F48F
-P 2975 10025
-F 0 "R13" H 3045 10071 50  0000 L CNN
-F 1 "240" H 3045 9980 50  0000 L CNN
-F 2 "Resistor_SMD:R_0603_1608Metric" V 2905 10025 50  0001 C CNN
-F 3 "~" H 2975 10025 50  0001 C CNN
-	1    2975 10025
-	1    0    0    -1
-$EndComp
-$Comp
-L Device:R R14
-U 1 1 5EA7F9E8
-P 3350 10025
-F 0 "R14" H 3420 10071 50  0000 L CNN
-F 1 "240" H 3420 9980 50  0000 L CNN
-F 2 "Resistor_SMD:R_0603_1608Metric" V 3280 10025 50  0001 C CNN
-F 3 "~" H 3350 10025 50  0001 C CNN
-	1    3350 10025
-	1    0    0    -1
-$EndComp
-$Comp
-L power:GNDPWR #PWR0166
-U 1 1 5EA7FFF4
-P 3350 10475
-F 0 "#PWR0166" H 3350 10275 50  0001 C CNN
-F 1 "GNDPWR" H 3354 10321 50  0000 C CNN
-F 2 "" H 3350 10425 50  0001 C CNN
-F 3 "" H 3350 10425 50  0001 C CNN
-	1    3350 10475
-	1    0    0    -1
-$EndComp
-$Comp
-L power:GNDPWR #PWR0167
-U 1 1 5EA8063C
-P 2975 10475
-F 0 "#PWR0167" H 2975 10275 50  0001 C CNN
-F 1 "GNDPWR" H 2979 10321 50  0000 C CNN
-F 2 "" H 2975 10425 50  0001 C CNN
-F 3 "" H 2975 10425 50  0001 C CNN
-	1    2975 10475
-	1    0    0    -1
-$EndComp
-$Comp
-L power:GNDPWR #PWR0168
-U 1 1 5EA80A12
-P 2600 10475
-F 0 "#PWR0168" H 2600 10275 50  0001 C CNN
-F 1 "GNDPWR" H 2604 10321 50  0000 C CNN
-F 2 "" H 2600 10425 50  0001 C CNN
-F 3 "" H 2600 10425 50  0001 C CNN
-	1    2600 10475
-	1    0    0    -1
-$EndComp
-$Comp
-L power:GNDPWR #PWR0169
-U 1 1 5EA80D9B
-P 2225 10475
-F 0 "#PWR0169" H 2225 10275 50  0001 C CNN
-F 1 "GNDPWR" H 2229 10321 50  0000 C CNN
-F 2 "" H 2225 10425 50  0001 C CNN
-F 3 "" H 2225 10425 50  0001 C CNN
-	1    2225 10475
-	1    0    0    -1
 $EndComp
 $Comp
@@
 Text Label 2375 6075 2    50   ~ 0
 IO_1
+Text Label 4850 8900 2    50   ~ 0
+TIM3_CH2
+Text Label 4850 9000 2    50   ~ 0
+TIM3_CH1
 Text Label 4850 7775 2    50   ~ 0
-TIM3_CH2
+TIM4_CH2
 Text Label 4850 7875 2    50   ~ 0
-TIM3_CH1
-Text Label 4850 8900 2    50   ~ 0
-TIM4_CH2
-Text Label 4850 9000 2    50   ~ 0
 TIM4_CH1
 Wire Wire Line
@@
 	1550 10150 1550 10175
 Connection ~ 1550 10150
-Text Label 2225 9875 2    50   ~ 0
+Text Label 2300 10475 2    50   ~ 0
 LED0
-Text Label 2600 9875 2    50   ~ 0
+Text Label 2675 10475 2    50   ~ 0
 LED1
-Text Label 2975 9875 2    50   ~ 0
+Text Label 3050 10475 2    50   ~ 0
 LED2
-Text Label 3350 9875 2    50   ~ 0
+Text Label 3425 10475 2    50   ~ 0
 LED3
 Text Label 2375 5775 2    50   ~ 0
@@
 LED3
 Text Label 2375 5575 2    50   ~ 0
+SW0
+Text Label 6775 3775 0    50   ~ 0
 SW1
-Text Label 6775 3775 0    50   ~ 0
-SW0
 Text Label 2375 4975 2    50   ~ 0
+Current1_Analog
+Text Label 2375 4875 2    50   ~ 0
 Current0_Analog
-Text Label 2375 4875 2    50   ~ 0
-Current1_Analog
 Text Label 6775 5175 0    50   ~ 0
 TIM3_CH2
@@
 EN0
 Text Label 2375 5375 2    50   ~ 0
+PWM0R
+Text Label 2375 5475 2    50   ~ 0
 PWM0L
-Text Label 2375 5475 2    50   ~ 0
-PWM0R
 Text Label 2375 4675 2    50   ~ 0
 MD0R_Temp
@@
 F 0 "R6" V 1068 1700 50  0000 C CNN
 F 1 "510" V 1159 1700 50  0000 C CNN
-F 2 "Resistor_SMD:R_0603_1608Metric" V 1205 1700 50  0001 C CNN
+F 2 "Mizz_lib:1608_WP" V 1205 1700 50  0001 C CNN
 F 3 "~" H 1275 1700 50  0001 C CNN
 	1    1275 1700
@@
 F 0 "R7" V 1068 2000 50  0000 C CNN
 F 1 "330" V 1159 2000 50  0000 C CNN
-F 2 "Resistor_SMD:R_0603_1608Metric" V 1205 2000 50  0001 C CNN
+F 2 "Mizz_lib:1608_WP" V 1205 2000 50  0001 C CNN
 F 3 "~" H 1275 2000 50  0001 C CNN
 	1    1275 2000
@@
 	1    0    0    -1
 $EndComp
+$Comp
+L Device:R R14
+U 1 1 5EA7F9E8
+P 3425 10025
+F 0 "R14" H 3495 10071 50  0000 L CNN
+F 1 "240" H 3495 9980 50  0000 L CNN
+F 2 "Resistor_SMD:R_0603_1608Metric" V 3355 10025 50  0001 C CNN
+F 3 "~" H 3425 10025 50  0001 C CNN
+	1    3425 10025
+	1    0    0    -1
+$EndComp
+$Comp
+L Device:R R13
+U 1 1 5EA7F48F
+P 3050 10025
+F 0 "R13" H 3120 10071 50  0000 L CNN
+F 1 "240" H 3120 9980 50  0000 L CNN
+F 2 "Resistor_SMD:R_0603_1608Metric" V 2980 10025 50  0001 C CNN
+F 3 "~" H 3050 10025 50  0001 C CNN
+	1    3050 10025
+	1    0    0    -1
+$EndComp
+$Comp
+L Device:R R12
+U 1 1 5EA7F1D4
+P 2675 10025
+F 0 "R12" H 2745 10071 50  0000 L CNN
+F 1 "240" H 2745 9980 50  0000 L CNN
+F 2 "Resistor_SMD:R_0603_1608Metric" V 2605 10025 50  0001 C CNN
+F 3 "~" H 2675 10025 50  0001 C CNN
+	1    2675 10025
+	1    0    0    -1
+$EndComp
+$Comp
+L Device:R R11
+U 1 1 5EA7ECE1
+P 2300 10025
+F 0 "R11" H 2370 10071 50  0000 L CNN
+F 1 "240" H 2370 9980 50  0000 L CNN
+F 2 "Resistor_SMD:R_0603_1608Metric" V 2230 10025 50  0001 C CNN
+F 3 "~" H 2300 10025 50  0001 C CNN
+	1    2300 10025
+	1    0    0    -1
+$EndComp
+$Comp
+L power:+3.3VP #PWR0166
+U 1 1 5E71DD61
+P 2300 9875
+F 0 "#PWR0166" H 2450 9825 50  0001 C CNN
+F 1 "+3.3VP" H 2320 10018 50  0000 C CNN
+F 2 "" H 2300 9875 50  0001 C CNN
+F 3 "" H 2300 9875 50  0001 C CNN
+	1    2300 9875
+	1    0    0    -1
+$EndComp
+$Comp
+L power:+3.3VP #PWR0167
+U 1 1 5E71E7CC
+P 2675 9875
+F 0 "#PWR0167" H 2825 9825 50  0001 C CNN
+F 1 "+3.3VP" H 2695 10018 50  0000 C CNN
+F 2 "" H 2675 9875 50  0001 C CNN
+F 3 "" H 2675 9875 50  0001 C CNN
+	1    2675 9875
+	1    0    0    -1
+$EndComp
+$Comp
+L power:+3.3VP #PWR0168
+U 1 1 5E71EAFD
+P 3050 9875
+F 0 "#PWR0168" H 3200 9825 50  0001 C CNN
+F 1 "+3.3VP" H 3070 10018 50  0000 C CNN
+F 2 "" H 3050 9875 50  0001 C CNN
+F 3 "" H 3050 9875 50  0001 C CNN
+	1    3050 9875
+	1    0    0    -1
+$EndComp
+$Comp
+L power:+3.3VP #PWR0169
+U 1 1 5E71F1B5
+P 3425 9875
+F 0 "#PWR0169" H 3575 9825 50  0001 C CNN
+F 1 "+3.3VP" H 3445 10018 50  0000 C CNN
+F 2 "" H 3425 9875 50  0001 C CNN
+F 3 "" H 3425 9875 50  0001 C CNN
+	1    3425 9875
+	1    0    0    -1
+$EndComp
