File: CAN_Current_Control_MD_ver0/CAN_Current_Control_MD.sch (KiCad schematic (older format))
At the start: 200 parts, among them J1 SWD, J10 FAN, J11 OUT_0, J12 OUT_1, J13 VALVE, J2 CAN, J3 CAN, J4 ENC0, J5 ENC1, J6 I/O_0, J7 I/O_1, J8 BATT_IN, J9 BATT_IN, Q1 MOSFET_N, Q10 NPN, Q2 MOSFET_N, Q3 MOSFET_N, Q4 MOSFET_N, Q5 MOSFET_N, Q6 MOSFET_N, Q7 MOSFET_N, Q8 MOSFET_N, Q9 NPN, SW1 SW0, SW2 SW1, SW3 RST, U1 BD33FA1, U10 NCP5104, U11 NCP5104, U12 BD9G101G, U13 INA181A1, U14 INA181A1, U15 LOGO, U2 ISO1050DUB, U3 STM32F405RG, U4 ADRESS, U5 AZ1086H, U6 BD9G101G, U7 AQM0802, U8 NCP5104, U9 NCP5104, Y1 8MHz

Commit message: 電流制御MD(仮)配線(仮)完成(仮)
Connections:
- net ADRESS_1: now also U3.20 (ADC12_IN4/PA4); no longer U3.23 (ADC12_IN7/TIM1_CH1N/TIM8_CH1N/TIM14_CH1/TIM3_CH2/PA7)
- net ADRESS_4: now also U3.23 (ADC12_IN7/TIM1_CH1N/TIM8_CH1N/TIM14_CH1/TIM3_CH2/PA7); no longer U3.21 (ADC12_IN5/TIM2_CH1_ETR/TIM8_CH1N/PA5)
- net Substrate_Temp: now also U3.21 (ADC12_IN5/TIM2_CH1_ETR/TIM8_CH1N/PA5); no longer U3.20 (ADC12_IN4/PA4)
Changed lines of the file:
@@
 Wire Wire Line
 	8975 4700 8975 4725
-Text Label 6775 3375 0    50   ~ 0
+Text Label 6775 3475 0    50   ~ 0
 Substrate_Temp
 Text Label 6775 3875 0    50   ~ 0
@@
 Text Label 6775 3075 0    50   ~ 0
 BATTERY_VOLTAGE
-Text Label 6775 3475 0    50   ~ 0
-ADRESS_4
+Text Label 6775 3375 0    50   ~ 0
+ADRESS_1
 Text Label 6775 3575 0    50   ~ 0
 ADRESS_8
 Text Label 6775 3675 0    50   ~ 0
-ADRESS_1
+ADRESS_4
 Text Label 6775 5575 0    50   ~ 0
 CAN1_TX

Commit message: 電流制御MDシリアル通信ポート忘れていたので，追加した
Parts:
- added C57: 0.1u, Mizz_lib:1608_WP, symbol Device:C
- added J14: SERIAL, Connector_PinSocket_2.54mm:PinSocket_1x04_P2.54mm_Vertical, symbol Connector_Generic:Conn_01x04
- SW1, SW2: footprint Button_Switch_SMD:SW_SPST_CK_RS282G05A3 -> Button_Switch_SMD:SW_SPST_PTS810
Connections:
- net +5VP: now also C57.2, J14.1 (Pin_1)
- net GNDPWR: now also C57.1, J14.2 (Pin_2)
- net USART1_RX: now also J14.3 (Pin_3)
- net USART1_TX: now also J14.4 (Pin_4)
Changed lines of the file:
@@
 F 0 "SW1" V 1596 10327 50  0000 R CNN
 F 1 "SW0" V 1505 10327 50  0000 R CNN
-F 2 "Button_Switch_SMD:SW_SPST_CK_RS282G05A3" H 1550 10575 50  0001 C CNN
+F 2 "Button_Switch_SMD:SW_SPST_PTS810" H 1550 10575 50  0001 C CNN
 F 3 "~" H 1550 10575 50  0001 C CNN
 	1    1550 10375
@@
 F 0 "SW2" V 1946 10327 50  0000 R CNN
 F 1 "SW1" V 1855 10327 50  0000 R CNN
-F 2 "Button_Switch_SMD:SW_SPST_CK_RS282G05A3" H 1900 10575 50  0001 C CNN
+F 2 "Button_Switch_SMD:SW_SPST_PTS810" H 1900 10575 50  0001 C CNN
 F 3 "~" H 1900 10575 50  0001 C CNN
 	1    1900 10375
@@
 	1    0    0    -1
 $EndComp
+$Comp
+L Connector_Generic:Conn_01x04 J14
+U 1 1 5E5EE089
+P 9000 7675
+F 0 "J14" H 9080 7667 50  0000 L CNN
+F 1 "SERIAL" H 9080 7576 50  0000 L CNN
+F 2 "Connector_PinSocket_2.54mm:PinSocket_1x04_P2.54mm_Vertical" H 9000 7675 50  0001 C CNN
+F 3 "~" H 9000 7675 50  0001 C CNN
+	1    9000 7675
+	1    0    0    -1
+$EndComp
+$Comp
+L Device:C C57
+U 1 1 5E5F14E2
+P 8650 7675
+F 0 "C57" V 8398 7675 50  0000 C CNN
+F 1 "0.1u" V 8489 7675 50  0000 C CNN
+F 2 "Mizz_lib:1608_WP" H 8688 7525 50  0001 C CNN
+F 3 "~" H 8650 7675 50  0001 C CNN
+	1    8650 7675
+	0    1    1    0
+$EndComp
+$Comp
+L power:GNDPWR #PWR0218
+U 1 1 5E5F1C14
+P 8800 7675
+F 0 "#PWR0218" H 8800 7475 50  0001 C CNN
+F 1 "GNDPWR" H 8804 7521 50  0000 C CNN
+F 2 "" H 8800 7625 50  0001 C CNN
+F 3 "" H 8800 7625 50  0001 C CNN
+	1    8800 7675
+	1    0    0    -1
+$EndComp
+Connection ~ 8800 7675
+$Comp
+L power:+5VP #PWR0219
+U 1 1 5E5F8890
+P 8500 7575
+F 0 "#PWR0219" H 8500 7425 50  0001 C CNN
+F 1 "+5VP" H 8515 7748 50  0000 C CNN
+F 2 "" H 8500 7575 50  0001 C CNN
+F 3 "" H 8500 7575 50  0001 C CNN
+	1    8500 7575
+	1    0    0    -1
+$EndComp
+Wire Wire Line
+	8500 7575 8800 7575
+Wire Wire Line
+	8500 7675 8500 7575
+Connection ~ 8500 7575
+Wire Wire Line
+	8500 7875 8800 7875
+Wire Wire Line
+	8800 7775 8500 7775
+Text Label 8500 7875 2    50   ~ 0
+USART1_TX
+Text Label 8500 7775 2    50   ~ 0
+USART1_RX
 $EndSCHEMATC

Commit message: いろいろ修正しました
Parts:
- R50, R51, R52, R53, R54, R55, R56, R57: value 3 -> FILTER
Other:
- note added: "FILTER : 3Ohm"
Changed lines of the file:
@@
 P 11875 3650
 F 0 "R51" V 11668 3650 50  0000 C CNN
-F 1 "3" V 11759 3650 50  0000 C CNN
+F 1 "FILTER" V 11759 3650 50  0000 C CNN
 F 2 "Resistor_SMD:R_0603_1608Metric" V 11805 3650 50  0001 C CNN
 F 3 "~" H 11875 3650 50  0001 C CNN
@@
 P 11875 3250
 F 0 "R50" V 11668 3250 50  0000 C CNN
-F 1 "3" V 11759 3250 50  0000 C CNN
+F 1 "FILTER" V 11759 3250 50  0000 C CNN
 F 2 "Resistor_SMD:R_0603_1608Metric" V 11805 3250 50  0001 C CNN
 F 3 "~" H 11875 3250 50  0001 C CNN
@@
 P 11875 5200
 F 0 "R53" V 11668 5200 50  0000 C CNN
-F 1 "3" V 11759 5200 50  0000 C CNN
+F 1 "FILTER" V 11759 5200 50  0000 C CNN
 F 2 "Resistor_SMD:R_0603_1608Metric" V 11805 5200 50  0001 C CNN
 F 3 "~" H 11875 5200 50  0001 C CNN
@@
 P 11875 4800
 F 0 "R52" V 11668 4800 50  0000 C CNN
-F 1 "3" V 11759 4800 50  0000 C CNN
+F 1 "FILTER" V 11759 4800 50  0000 C CNN
 F 2 "Resistor_SMD:R_0603_1608Metric" V 11805 4800 50  0001 C CNN
 F 3 "~" H 11875 4800 50  0001 C CNN
@@
 P 11875 7075
 F 0 "R55" V 11668 7075 50  0000 C CNN
-F 1 "3" V 11759 7075 50  0000 C CNN
+F 1 "FILTER" V 11759 7075 50  0000 C CNN
 F 2 "Resistor_SMD:R_0603_1608Metric" V 11805 7075 50  0001 C CNN
 F 3 "~" H 11875 7075 50  0001 C CNN
@@
 P 11875 6675
 F 0 "R54" V 11668 6675 50  0000 C CNN
-F 1 "3" V 11759 6675 50  0000 C CNN
+F 1 "FILTER" V 11759 6675 50  0000 C CNN
 F 2 "Resistor_SMD:R_0603_1608Metric" V 11805 6675 50  0001 C CNN
 F 3 "~" H 11875 6675 50  0001 C CNN
@@
 P 11875 8625
 F 0 "R57" V 11668 8625 50  0000 C CNN
-F 1 "3" V 11759 8625 50  0000 C CNN
+F 1 "FILTER" V 11759 8625 50  0000 C CNN
 F 2 "Resistor_SMD:R_0603_1608Metric" V 11805 8625 50  0001 C CNN
 F 3 "~" H 11875 8625 50  0001 C CNN
@@
 P 11875 8225
 F 0 "R56" V 11668 8225 50  0000 C CNN
-F 1 "3" V 11759 8225 50  0000 C CNN
+F 1 "FILTER" V 11759 8225 50  0000 C CNN
 F 2 "Resistor_SMD:R_0603_1608Metric" V 11805 8225 50  0001 C CNN
 F 3 "~" H 11875 8225 50  0001 C CNN
@@
 Text Label 8500 7775 2    50   ~ 0
 USART1_RX
+Text Notes 11650 2825 0    50   ~ 0
+FILTER : 3Ohm
 $EndSCHEMATC
