File: stm32f4_Centaurus_ver.2.1.1/stm32f4_Centaurus_ver.2.1.1/stm32f4_Centaurus.sch (KiCad schematic (older format))
At the start: 219 parts, among them IC1 PIC24FJ64GB004, J1 SERIAL1, J2 EXTERNAL_~RST, P1 PICKit3, P10 XA2_12V, P11 CAN0, P12 CAN1, P13 CAN0, P14 CAN1, P15 SERIAL2, P16 SERIAL0, P17 XA2_5V, P18 SWD, P2 SERIAL5_SBDBT, P23 A/D, P24 PWM, P25 A/D_batt, P26 PWM_batt, P27 EMERGENCY_CHECK, P28 I/O_5V, P29 I/O_Variable, P3 ENC0, P30 I/O_5V_batt, P31 I/O_Variable, P4 ENC2, P6 ENC3, P7 ENC1, P8 SERIAL4, P9 SERIAL3, Q1 FET_P, Q2 FET_P, Q3 FET_P, Q4 NPN, Q5 NPN, Q6 FET_P, Q7 FET_N, Q8 FET_N, SW1 Main_POWER, SW2 SW1, SW3 SW0, SW4 SW2, SW5 SW3, U1 STM32F407VG, U10 LOGO, U12 25LC010A, U13 LOGO, U2 AZ1086H, U3 MCP2221A, U4 BD9G101G, U5 MAX3051, U6 MAX3051, U7 AQM1602_BL, U8 OSTBABS4C2B, U9 LOGO, X1 8MHz

Commit message: MAIN基板，大体の構成完了．あとは配線を少し修正するのみ
Parts:
- removed C41: 0.1u, Mizz_lib:C_0603, symbol stm32f4_Centaurus-rescue:C-device
- removed R64: 10, Mizz_lib:R_0603, symbol stm32f4_Centaurus-rescue:R-device
- removed U12: 25LC010A, Mizz_lib:DIP-8_W7.62mm, symbol stm32f4_Centaurus-rescue:25LC010A-Miz
- added C32: 0.1u, Mizz_lib:C_0603, symbol stm32f4_Centaurus-rescue:C-device
- added D33, D34: LED, Mizz_lib:LED_0603, symbol stm32f4_Centaurus-rescue:LED-device
- added JP6: RST_JP, Connector_PinHeader_2.54mm:PinHeader_1x02_P2.54mm_Vertical, symbol Device:Jumper
- added P5: SPI0, Mizz_lib:XA_6T, symbol stm32f4_Centaurus-rescue:Conn_01x06
- R46, R47, R48: footprint Mizz_lib:R_0603 -> Mizz_lib:1608_WP
- R62, R63: value 10 -> 330
Connections:
- net +5V: now also C32.2, P5.2 (Pin_2)
- net GND: now also R62.2, R63.2, C32.1, P5.1 (Pin_1)
- net PE10: now also P5.6 (Pin_6)
- net PE7: now also D33.1 (A)
- net PE8: now also D34.1 (A)
- net SPI2_MISO: now also P5.4 (Pin_4); no longer R62.2
- net SPI2_MOSI: now also P5.3 (Pin_3)
- net SPI2_SCK: now also P5.5 (Pin_5); no longer R63.1
- net ~RST: now also JP6.2; no longer Q8.2 (S), R77.2
- net at R62.1: now also D33.2 (K)
- new net: JP6.1, Q8.2 (S), R77.2
- new net: D34.2 (K), R63.1
Other:
- note added: "I/O,ADC,PWM,SPI"
- note removed: "I/O,ADC,PWM"
- moved on the sheet: D19, D21, D22, D23, D24, D25, J2, Q8, R45, R49, R54, R55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
