File: stm32f4_Centaurus_ver.3.0/stm32f4_Centaurus_ver.3.0/stm32f4_Centaurus.sch (KiCad schematic (older format))
At the start: 221 parts, among them IC1 PIC24FJ64GB004, J1 SERIAL1, J2 EXTERNAL_~RST, P1 PICKit3, P10 XA2_12V, P11 CAN0, P12 CAN1, P13 CAN0, P14 CAN1, P15 SERIAL2, P16 SERIAL0, P17 XA2_5V, P18 SWD, P2 SERIAL5_SBDBT, P23 A/D, P24 PWM, P25 A/D_batt, P26 PWM_batt, P27 EMERGENCY_CHECK, P28 I/O_5V, P29 I/O_Variable, P3 ENC0, P30 I/O_5V_batt, P31 I/O_Variable, P4 ENC2, P5 SPI0, P6 ENC3, P7 ENC1, P8 SERIAL4, P9 SERIAL3, Q1 FET_P, Q2 FET_P, Q3 FET_P, Q4 NPN, Q5 NPN, Q6 FET_P, Q7 FET_N, SW1 Main_POWER, SW2 SW1, SW3 SW0, SW4 SW2, SW5 SW3, U1 STM32F407VG, U10 LOGO, U11 TLP4227G-2, U13 LOGO, U2 AZ1086H, U3 MCP2221A, U4 BD9G101G, U5 MAX3051, U6 MAX3051, U7 AQM1602_BL, U8 OSTBABS4C2B, U9 LOGO, X1 8MHz

Commit message: 電源基板とかの回路図変更していなかった気がする
Parts:
- U11: symbol Miz:TLP4227G-2 -> stm32f4_Centaurus-rescue:TLP4227G-2-Miz
Changed lines of the file:
@@
 EESchema Schematic File Version 4
+LIBS:stm32f4_Centaurus-cache
 EELAYER 30 0
 EELAYER END
@@
 ST-LINK_Vdd
 $Comp
-L Miz:TLP4227G-2 U11
+L stm32f4_Centaurus-rescue:TLP4227G-2-Miz U11
 U 1 1 5EFA93F3
 P 16775 900
