File: CAN_BLDCMD_type0/CAN_BLDCMD.sch (KiCad schematic (older format))
At the start: 179 parts, among them J1 SWD, J10 BATT_IN, J11 OUT_U, J12 OUT_V, J13 OUT_W, J2 CAN, J3 CAN, J4 ENC, J5 I/O0, J6 I/O1, J7 SERIAL, J8 FAN, J9 BATT_IN, Q1 MOSFET_N, Q2 MOSFET_N, Q3 MOSFET_N, Q4 MOSFET_N, Q5 MOSFET_N, Q6 MOSFET_N, SW1 SW0, SW2 SW1, U1 MAX3051, U10 SI8900, U11 ADC_~RST, U12 ACS758, U13 ACS758, U14 ACS758, U15 BD9G101G, U16 LTC2644, U17 LTC2644, U18 BD33FA1, U19 LOGO, U2 BD9G101G, U3 STM32F405RG, U4 AZ1086H, U5 SW_ROTARY_16, U6 POWER_ON, U7 SI8274, U8 SI8274, U9 SI8274, Y1 8MHz

Commit message: BLDCMD本格的に設計開始
Parts:
- added J14: VALVE, Mizz_lib:XA_4L, symbol Connector_Generic:Conn_01x04
- added U?: AQM0802, symbol Miz:AQM1602
- C49: value 1500u -> 2200u
- JP2: value Jumper -> CAN_JP
- R39, R40, R41, R42, R43, R44: value 1 -> 10
- U5: value SW_ROTARY_16 -> ADRESS
Changed lines of the file:
@@
 P 16675 6825
 F 0 "R41" V 16468 6825 50  0000 C CNN
-F 1 "1" V 16559 6825 50  0000 C CNN
+F 1 "10" V 16559 6825 50  0000 C CNN
 F 2 "Mizz_lib:1608_WP" V 16605 6825 50  0001 C CNN
 F 3 "~" H 16675 6825 50  0001 C CNN
@@
 P 16675 7575
 F 0 "R42" V 16468 7575 50  0000 C CNN
-F 1 "1" V 16559 7575 50  0000 C CNN
+F 1 "10" V 16559 7575 50  0000 C CNN
 F 2 "Mizz_lib:1608_WP" V 16605 7575 50  0001 C CNN
 F 3 "~" H 16675 7575 50  0001 C CNN
@@
 	3575 10425 3550 10425
 $Comp
-L Device:Jumper JP2
-U 1 1 5E536B67
-P 3800 9275
-F 0 "JP2" H 3800 9539 50  0000 C CNN
-F 1 "Jumper" H 3800 9448 50  0000 C CNN
-F 2 "Connector_PinHeader_2.54mm:PinHeader_1x02_P2.54mm_Vertical" H 3800 9275 50  0001 C CNN
-F 3 "~" H 3800 9275 50  0001 C CNN
-	1    3800 9275
-	1    0    0    -1
-$EndComp
-$Comp
 L Device:R R4
 U 1 1 5E53789E
@@
 P 19175 1100
 F 0 "C49" H 19290 1146 50  0000 L CNN
-F 1 "1500u" H 19290 1055 50  0000 L CNN
+F 1 "2200u" H 19290 1055 50  0000 L CNN
 F 2 "Mizz_lib:C_Radial_D13mm_H25.0mm_P5.00mm" H 19175 1100 50  0001 C CNN
 F 3 "~" H 19175 1100 50  0001 C CNN
@@
 P 16675 9050
 F 0 "R43" V 16468 9050 50  0000 C CNN
-F 1 "1" V 16559 9050 50  0000 C CNN
+F 1 "10" V 16559 9050 50  0000 C CNN
 F 2 "Mizz_lib:1608_WP" V 16605 9050 50  0001 C CNN
 F 3 "~" H 16675 9050 50  0001 C CNN
@@
 P 16675 9800
 F 0 "R44" V 16468 9800 50  0000 C CNN
-F 1 "1" V 16559 9800 50  0000 C CNN
+F 1 "10" V 16559 9800 50  0000 C CNN
 F 2 "Mizz_lib:1608_WP" V 16605 9800 50  0001 C CNN
 F 3 "~" H 16675 9800 50  0001 C CNN
@@
 P 16675 4600
 F 0 "R39" V 16468 4600 50  0000 C CNN
-F 1 "1" V 16559 4600 50  0000 C CNN
+F 1 "10" V 16559 4600 50  0000 C CNN
 F 2 "Mizz_lib:1608_WP" V 16605 4600 50  0001 C CNN
 F 3 "~" H 16675 4600 50  0001 C CNN
@@
 P 16675 5350
 F 0 "R40" V 16468 5350 50  0000 C CNN
-F 1 "1" V 16559 5350 50  0000 C CNN
+F 1 "10" V 16559 5350 50  0000 C CNN
 F 2 "Mizz_lib:1608_WP" V 16605 5350 50  0001 C CNN
 F 3 "~" H 16675 5350 50  0001 C CNN
@@
 P 7275 11350
 F 0 "U5" H 7275 11787 60  0000 C CNN
-F 1 "SW_ROTARY_16" H 7275 11681 60  0000 C CNN
+F 1 "ADRESS" H 7275 11681 60  0000 C CNN
 F 2 "Mizz_lib:rotary_0F" H 7275 11350 60  0001 C CNN
 F 3 "" H 7275 11350 60  0001 C CNN
@@
 	1    0    0    -1
 $EndComp
+$Comp
+L Device:Jumper JP2
+U 1 1 5E536B67
+P 3800 9275
+F 0 "JP2" H 3800 9539 50  0000 C CNN
+F 1 "CAN_JP" H 3800 9448 50  0000 C CNN
+F 2 "Connector_PinHeader_2.54mm:PinHeader_1x02_P2.54mm_Vertical" H 3800 9275 50  0001 C CNN
+F 3 "~" H 3800 9275 50  0001 C CNN
+	1    3800 9275
+	1    0    0    -1
+$EndComp
+$Comp
+L Connector_Generic:Conn_01x04 J14
+U 1 1 5E67B09F
+P 6100 10225
+F 0 "J14" H 6180 10217 50  0000 L CNN
+F 1 "VALVE" H 6180 10126 50  0000 L CNN
+F 2 "Mizz_lib:XA_4L" H 6100 10225 50  0001 C CNN
+F 3 "~" H 6100 10225 50  0001 C CNN
+	1    6100 10225
+	1    0    0    -1
+$EndComp
+$Comp
+L Miz:AQM1602 U?
+U 1 1 5E68D963
+P 10675 10875
+F 0 "U?" H 10953 10871 50  0000 L CNN
+F 1 "AQM0802" H 10953 10780 50  0000 L CNN
+F 2 "" H 10475 11025 50  0001 C CNN
+F 3 "" H 10475 11025 50  0001 C CNN
+	1    10675 10875
+	1    0    0    -1
+$EndComp

Commit message: BLDC(仮)が形になってきた
Parts:
- added C61, C62: 1u, Mizz_lib:1608_WP, symbol Device:C
- added C63, C64: 0.1u, Mizz_lib:1608_WP, symbol Device:C
- added D17, D18: DIODE, Diode_SMD:D_SOD-123, symbol Miz:DIODE_rev
- added D19: VALVE0, LED_SMD:LED_0603_1608Metric, symbol Device:LED
- added D20: VALVE1, LED_SMD:LED_0603_1608Metric, symbol Device:LED
- added D21: 12V, LED_SMD:LED_0603_1608Metric, symbol Device:LED
- added D22: 5V, LED_SMD:LED_0603_1608Metric, symbol Device:LED
- added D23: 3V3, LED_SMD:LED_0603_1608Metric, symbol Device:LED
- added D24: BATT, LED_SMD:LED_0603_1608Metric, symbol Device:LED
- added D25: MAIN_BATT, LED_SMD:LED_0603_1608Metric, symbol Device:LED
- added D26: 12VP, LED_SMD:LED_0603_1608Metric, symbol Device:LED
- added D27: 3V3P, LED_SMD:LED_0603_1608Metric, symbol Device:LED
- added Q7, Q8: NPN, Package_TO_SOT_SMD:SOT-23, symbol Device:Q_NPN_BEC
- added R54, R55: 10k, Mizz_lib:1608_WP, symbol Device:R
- added R56, R57, R60: 330, Mizz_lib:1608_WP, symbol Device:R
- added R58: 1.2k, Mizz_lib:1608_WP, symbol Device:R
- added R59, R64: 510, Mizz_lib:1608_WP, symbol Device:R
- added R61, R62: 4.7k, Mizz_lib:1608_WP, symbol Device:R
- added R63: 2.2k, Mizz_lib:1608_WP, symbol Device:R
- added SW3: RST, Button_Switch_SMD:SW_SPST_CK_RS282G05A3, symbol Switch:SW_Push
- R13, R14: value R -> 330
- U20: renamed from U?; footprint (none) -> Mizz_lib:AQM0802_original
Connections:
- net +12P: now also C58.1, C59.1, D16.1 (K), U18.3 (Vcc), R63.2
- net +12V: now also J14.2 (Pin_2), J14.4 (Pin_4), R58.2
- net +3.3VP: now also R64.2
- net +3V3: now also U20.5 (VDD), U20.9 (/RST), C61.2, C63.2, R54.1, R55.1, R60.2
- net +5V: now also R59.2
- net +BATT: now also R61.2
- net +Batt: now also R62.2
- net GND: now also SW1.1, SW2.1, U20.6 (VSS), C63.1, C64.1, D17.2 (A), D18.2 (A), D19.1 (K), D20.1 (K), D21.1 (K), D22.1 (K), D23.1 (K), Q7.2 (E), Q8.2 (E), SW3.1
- net GNDPWR: now also D24.1 (K), D25.1 (K), D26.1 (K), D27.1 (K)
- net ~RST: now also C64.2, SW3.2
- net at J14.1 (Pin_1): now also D17.1 (K), Q7.3 (C)
- net at J14.3 (Pin_3): now also D18.1 (K), Q8.3 (C)
- net at U20.2 (VOUT): now also C61.1
- net at U20.3 (CAP1N): now also C62.1
- net at U20.4 (CAP1P): now also C62.2
- net I2Cx_SDA: now reaches U20.7 (SDA)
- net I2Cx_SDA: now also R55.2
- net I2Cx_SCL: now reaches U20.8 (SCL)
- net I2Cx_SCL: now also R54.2
- new net: D19.2 (A), R56.2
- new net: D20.2 (A), R57.2
- new net: D24.2 (A), R61.1
- new net: D25.2 (A), R62.1
- new net: D26.2 (A), R63.1
- new net: D27.2 (A), R64.1
- new net: D21.2 (A), R58.1
- new net: D22.2 (A), R59.1
- new net: D23.2 (A), R60.1
- new net VALVE_0: Q7.1 (B), R56.1
- new net VALVE_1: Q8.1 (B), R57.1
- no-connect marks 13 -> 14
Other:
- moved on the sheet: C10, C3, C9, D5, D6, J14, J2, J3, JP2, R11, R13, R14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

Commit message: いろいろ修正しました
Parts:
- added J15: HALL_IN, Mizz_lib:ZH_6P, symbol Connector_Generic:Conn_01x06
- added R65: 10k, Mizz_lib:1608_WP, symbol Device:R
- added SW4: MODE, Mizz_lib:SW_Micro_SPST, symbol Switch:SW_SPDT
- D14, D16: value DIODE] -> DIODE
- D15: footprint Diode_SMD:D_SMA -> Diode_SMD:D_2010_5025Metric_Pad1.52x2.65mm_HandSolder
- R47: footprint Mizz_lib:R_2812 -> Resistor_SMD:R_2512_6332Metric
- SW1, SW2: footprint Button_Switch_SMD:SW_SPST_CK_RS282G05A3 -> Button_Switch_SMD:SW_SPST_PTS810
Connections:
- net +3V3: now also D1.1 (K), R65.1; no longer JP1.2
- net +5V: now also J15.6 (Pin_6)
- net GND: now also J15.1 (Pin_1), SW4.3 (C)
- net SW_MODE: now reaches U3.37 (PC6/TIM8_CH1/USART6_TX/TIM3_CH1)
- net SW_MODE: now also R65.2, SW4.2 (B)
- net HALL_0: now reaches U3.51 (PC10/UART4_TX/USART3_TX)
- net HALL_0: now also J15.2 (Pin_2)
- net HALL_1: now reaches U3.52 (PC11/UART4_RX/USART3_RX)
- net HALL_1: now also J15.3 (Pin_3)
- net HALL_2: now reaches U3.53 (PC12/UART5_TX)
- net HALL_2: now also J15.4 (Pin_4)
- net at J1.2 (Pin_2): now also JP1.1; no longer D1.2 (A)
- new net: D1.2 (A), JP1.2
- no-connect marks 14 -> 16
Other:
- moved on the sheet: D1, JP1
Changed lines of the file:
@@
 L Miz:DIODE_rev D1
 U 1 1 5E4321DC
-P 975 3525
-F 0 "D1" H 975 3717 40  0000 C CNN
-F 1 "DIODE" H 975 3641 40  0000 C CNN
-F 2 "Diode_SMD:D_SOD-123" H 975 3525 60  0001 C CNN
-F 3 "" H 975 3525 60  0000 C CNN
-	1    975  3525
+P 1575 3525
+F 0 "D1" H 1575 3717 40  0000 C CNN
+F 1 "DIODE" H 1575 3641 40  0000 C CNN
+F 2 "Diode_SMD:D_SOD-123" H 1575 3525 60  0001 C CNN
+F 3 "" H 1575 3525 60  0000 C CNN
+	1    1575 3525
 	1    0    0    -1
 $EndComp
@@
 L Device:Jumper JP1
 U 1 1 5E433921
-P 1475 3525
-F 0 "JP1" H 1475 3789 50  0000 C CNN
-F 1 "SWD_JP" H 1475 3698 50  0000 C CNN
-F 2 "Jumper:SolderJumper-2_P1.3mm_Open_TrianglePad1.0x1.5mm" H 1475 3525 50  0001 C CNN
-F 3 "~" H 1475 3525 50  0001 C CNN
-	1    1475 3525
+P 1075 3525
+F 0 "JP1" H 1075 3789 50  0000 C CNN
+F 1 "SWD_JP" H 1075 3698 50  0000 C CNN
+F 2 "Jumper:SolderJumper-2_P1.3mm_Open_TrianglePad1.0x1.5mm" H 1075 3525 50  0001 C CNN
+F 3 "~" H 1075 3525 50  0001 C CNN
+	1    1075 3525
 	1    0    0    -1
 $EndComp
@@
 F 0 "D15" H 19475 1890 50  0000 C CNN
 F 1 "DIODE" H 19475 1799 50  0000 C CNN
-F 2 "Diode_SMD:D_SMA" H 19475 1625 50  0001 C CNN
+F 2 "Diode_SMD:D_2010_5025Metric_Pad1.52x2.65mm_HandSolder" H 19475 1625 50  0001 C CNN
 F 3 "~" H 19475 1625 50  0001 C CNN
 	1    19475 1625
@@
 P 18950 1975
 F 0 "D14" H 18950 1783 40  0000 C CNN
-F 1 "DIODE]" H 18950 1859 40  0000 C CNN
+F 1 "DIODE" H 18950 1859 40  0000 C CNN
 F 2 "Diode_SMD:D_SOD-123" H 18950 1975 60  0001 C CNN
 F 3 "" H 18950 1975 60  0000 C CNN
@@
 P 19875 2400
 F 0 "D16" H 19875 2592 40  0000 C CNN
-F 1 "DIODE]" H 19875 2516 40  0000 C CNN
+F 1 "DIODE" H 19875 2516 40  0000 C CNN
 F 2 "Diode_SMD:D_SOD-123" H 19875 2400 60  0001 C CNN
 F 3 "" H 19875 2400 60  0000 C CNN
@@
 F 0 "R47" V 17743 1350 50  0000 C CNN
 F 1 "47" V 17834 1350 50  0000 C CNN
-F 2 "Mizz_lib:R_2812" V 17880 1350 50  0001 C CNN
+F 2 "Resistor_SMD:R_2512_6332Metric" V 17880 1350 50  0001 C CNN
 F 3 "~" H 17950 1350 50  0001 C CNN
 	1    17950 1350
@@
 F 0 "SW2" V 2471 12202 50  0000 R CNN
 F 1 "SW1" V 2380 12202 50  0000 R CNN
-F 2 "Button_Switch_SMD:SW_SPST_CK_RS282G05A3" H 2425 12450 50  0001 C CNN
+F 2 "Button_Switch_SMD:SW_SPST_PTS810" H 2425 12450 50  0001 C CNN
 F 3 "~" H 2425 12450 50  0001 C CNN
 	1    2425 12250
@@
 F 0 "SW1" V 2121 12202 50  0000 R CNN
 F 1 "SW0" V 2030 12202 50  0000 R CNN
-F 2 "Button_Switch_SMD:SW_SPST_CK_RS282G05A3" H 2075 12450 50  0001 C CNN
+F 2 "Button_Switch_SMD:SW_SPST_PTS810" H 2075 12450 50  0001 C CNN
 F 3 "~" H 2075 12450 50  0001 C CNN
 	1    2075 12250
@@
 Wire Wire Line
 	8450 1825 8450 1475
+$Comp
+L Connector_Generic:Conn_01x06 J15
+U 1 1 5E62F58F
+P 1450 13475
+F 0 "J15" H 1368 13892 50  0000 C CNN
+F 1 "HALL_IN" H 1368 13801 50  0000 C CNN
+F 2 "Mizz_lib:ZH_6P" H 1450 13475 50  0001 C CNN
+F 3 "~" H 1450 13475 50  0001 C CNN
+	1    1450 13475
+	-1   0    0    -1
+$EndComp
+$Comp
+L Switch:SW_SPDT SW4
+U 1 1 5E6375D3
+P 2000 14475
+F 0 "SW4" H 2000 14760 50  0000 C CNN
+F 1 "MODE" H 2000 14669 50  0000 C CNN
+F 2 "Mizz_lib:SW_Micro_SPST" H 2000 14475 50  0001 C CNN
+F 3 "~" H 2000 14475 50  0001 C CNN
+	1    2000 14475
+	1    0    0    -1
+$EndComp
+$Comp
+L power:GND #PWR0246
+U 1 1 5E63F088
+P 1675 13275
+F 0 "#PWR0246" H 1675 13025 50  0001 C CNN
+F 1 "GND" H 1680 13102 50  0000 C CNN
+F 2 "" H 1675 13275 50  0001 C CNN
+F 3 "" H 1675 13275 50  0001 C CNN
+	1    1675 13275
+	1    0    0    -1
+$EndComp
+Text Label 1725 13375 0    50   ~ 0
+HALL_0
+Wire Wire Line
+	1725 13375 1650 13375
+Wire Wire Line
+	1675 13275 1650 13275
+Text Label 1725 13475 0    50   ~ 0
+HALL_1
+Text Label 1725 13575 0    50   ~ 0
+HALL_2
+Wire Wire Line
+	1725 13575 1650 13575
+Wire Wire Line
+	1725 13475 1650 13475
+NoConn ~ 1650 13675
+$Comp
+L power:+5V #PWR0247
+U 1 1 5E719BD9
+P 1725 13775
+F 0 "#PWR0247" H 1725 13625 50  0001 C CNN
+F 1 "+5V" H 1740 13948 50  0000 C CNN
+F 2 "" H 1725 13775 50  0001 C CNN
+F 3 "" H 1725 13775 50  0001 C CNN
+	1    1725 13775
+	1    0    0    -1
+$EndComp
+Wire Wire Line
+	1725 13775 1650 13775
+Text Label 2225 6775 2    50   ~ 0
+HALL_0
+Text Label 2225 6875 2    50   ~ 0
+HALL_1
+Text Label 2225 6975 2    50   ~ 0
+HALL_2
+Text Label 2225 6375 2    50   ~ 0
+SW_MODE
+Text Label 1700 14475 2    50   ~ 0
+SW_MODE
+$Comp
+L Device:R R65
+U 1 1 5E786CAC
+P 1750 14325
+F 0 "R65" H 1820 14371 50  0000 L CNN
+F 1 "10k" H 1820 14280 50  0000 L CNN
+F 2 "Mizz_lib:1608_WP" V 1680 14325 50  0001 C CNN
+F 3 "~" H 1750 14325 50  0001 C CNN
+	1    1750 14325
+	1    0    0    -1
+$EndComp
+Wire Wire Line
+	1700 14475 1750 14475
+Connection ~ 1750 14475
+Wire Wire Line
+	1750 14475 1800 14475
+$Comp
+L power:+3.3V #PWR0248
+U 1 1 5E7E3663
+P 1750 14175
+F 0 "#PWR0248" H 1750 14025 50  0001 C CNN
+F 1 "+3.3V" H 1765 14348 50  0000 C CNN
+F 2 "" H 1750 14175 50  0001 C CNN
+F 3 "" H 1750 14175 50  0001 C CNN
+	1    1750 14175
+	1    0    0    -1
+$EndComp
+NoConn ~ 2200 14375
+$Comp
+L power:GND #PWR0249
+U 1 1 5E8114EB
+P 2250 14575
+F 0 "#PWR0249" H 2250 14325 50  0001 C CNN
+F 1 "GND" H 2255 14402 50  0000 C CNN
+F 2 "" H 2250 14575 50  0001 C CNN
+F 3 "" H 2250 14575 50  0001 C CNN
+	1    2250 14575
+	1    0    0    -1
+$EndComp
+Wire Wire Line
+	2250 14575 2200 14575
 $EndSCHEMATC

Commit message: BLDC 途中
Parts:
- added D28: MODE, LED_SMD:LED_0603_1608Metric, symbol Device:LED
- added R66: 330, Mizz_lib:1608_WP, symbol Device:R
- D15: footprint Diode_SMD:D_2010_5025Metric_Pad1.52x2.65mm_HandSolder -> Diode_SMD:D_SOD-123
- D5: value LED -> BUS
- D6: value LED -> EMG
- R32: value 4.7k -> 20k
Connections:
- net ADC_~RST~_Pin: now also U3.53 (PC12/UART5_TX); no longer U3.15 (UART4_RX/ADC12_IN1/TIM5_CH2/TIM2_CH2/PA1)
- net Drive_U_Temp: now also U3.14 (UART4_TX/TIM2_CH1_ETR/ADC12_IN0/TIM5_CH1/PA0); no longer U3.20 (ADC12_IN4/PA4)
- net Drive_V_Temp: now also U3.10 (PC2/ADC12_IN12); no longer U3.21 (ADC12_IN5/TIM2_CH1_ETR/TIM8_CH1N/PA5)
- net Drive_W_Temp: now also U3.8 (PC0/ADC12_IN10); no longer U3.22 (ADC12_IN6/TIM3_CH1/TIM13_CH1/PA6)
- net GND: now also D28.1 (K)
- net HALL_0: now also U3.38 (PC7/TIM8_CH2/USART6_RX/TIM3_CH2); no longer U3.51 (PC10/UART4_TX/USART3_TX)
- net HALL_1: now also U3.39 (PC8/TIM8_CH3/TIM3_CH3); no longer U3.52 (PC11/UART4_RX/USART3_RX)
- net HALL_2: now also U3.40 (PC9/TIM8_CH4/TIM3_CH4); no longer U3.53 (PC12/UART5_TX)
- net LED0: now also U3.50 (TIM2_CH1_ETR/PA15); no longer U3.9 (PC1/ADC12_IN11)
- net LED1: now also U3.58 (TIM4_CH1/CAN2_TX/USART1_TX/PB6); no longer U3.10 (PC2/ADC12_IN12)
- net OUT_U_Current: now also U3.15 (UART4_RX/ADC12_IN1/TIM5_CH2/TIM2_CH2/PA1); no longer U3.25 (PC5/ADC12_IN15)
- net OUT_V_Current: now also U3.11 (PC3/ADC12_IN13); no longer U3.26 (ADC12_IN8/TIM1_CH2N/TIM8_CH2N/TIM3_CH3/PB0)
- net OUT_W_Current: now also U3.9 (PC1/ADC12_IN11); no longer U3.27 (ADC12_IN9/TIM1_CH3N/TIM8_CH3N/TIM3_CH4/PB1)
- net PWR_ON_Pin: now also U3.55 (TIM2_CH2/PB3); no longer U3.14 (UART4_TX/TIM2_CH1_ETR/ADC12_IN0/TIM5_CH1/PA0)
- net Subscribe_Temp: now also U3.17 (USART2_RX/TIM5_CH4/TIM9_CH2/ADC12_IN3/TIM2_CH4/PA3); no longer U3.23 (ADC12_IN7/TIM1_CH1N/TIM8_CH1N/TIM14_CH1/TIM3_CH2/PA7)
- net USARTx_RX: now also U3.52 (PC11/UART4_RX/USART3_RX); no longer U3.17 (USART2_RX/TIM5_CH4/TIM9_CH2/ADC12_IN3/TIM2_CH4/PA3)
- net USARTx_TX: now also U3.51 (PC10/UART4_TX/USART3_TX); no longer U3.16 (USART2_TX/TIM5_CH3/TIM9_CH1/ADC12_IN2/TIM2_CH3/PA2)
- net LED2: now reaches U3.59 (USART1_RX/TIM4_CH2/PB7)
- net LED2: now also R66.1
- new net: D28.2 (A), R66.2
Changed lines of the file:
@@
 EESchema Schematic File Version 4
-LIBS:CAN_BLDCMD-cache
 EELAYER 30 0
 EELAYER END
@@
 F 0 "D15" H 19475 1890 50  0000 C CNN
 F 1 "DIODE" H 19475 1799 50  0000 C CNN
-F 2 "Diode_SMD:D_2010_5025Metric_Pad1.52x2.65mm_HandSolder" H 19475 1625 50  0001 C CNN
+F 2 "Diode_SMD:D_SOD-123" H 19475 1625 50  0001 C CNN
 F 3 "~" H 19475 1625 50  0001 C CNN
 	1    19475 1625
@@
 P 15850 3625
 F 0 "R32" V 15643 3625 50  0000 C CNN
-F 1 "4.7k" V 15734 3625 50  0000 C CNN
+F 1 "20k" V 15734 3625 50  0000 C CNN
 F 2 "Mizz_lib:1608_WP" V 15780 3625 50  0001 C CNN
 F 3 "~" H 15850 3625 50  0001 C CNN
@@
 P 2875 12050
 F 0 "D5" V 2914 11933 50  0000 R CNN
-F 1 "LED" V 2823 11933 50  0000 R CNN
+F 1 "BUS" V 2823 11933 50  0000 R CNN
 F 2 "LED_SMD:LED_0603_1608Metric" H 2875 12050 50  0001 C CNN
 F 3 "~" H 2875 12050 50  0001 C CNN
@@
 P 3200 12050
 F 0 "D6" V 3239 11933 50  0000 R CNN
-F 1 "LED" V 3148 11933 50  0000 R CNN
+F 1 "EMG" V 3148 11933 50  0000 R CNN
 F 2 "LED_SMD:LED_0603_1608Metric" H 3200 12050 50  0001 C CNN
 F 3 "~" H 3200 12050 50  0001 C CNN
@@
 	1    0    0    -1
 $EndComp
-Text Label 6625 4275 0    50   ~ 0
+Text Label 2225 6775 2    50   ~ 0
 USARTx_TX
-Text Label 6625 4375 0    50   ~ 0
+Text Label 2225 6875 2    50   ~ 0
 USARTx_RX
-Text Label 6625 4475 0    50   ~ 0
-Drive_U_Temp
-Text Label 6625 4575 0    50   ~ 0
+Text Label 2225 5975 2    50   ~ 0
 Drive_V_Temp
-Text Label 6625 4675 0    50   ~ 0
+Text Label 2225 5775 2    50   ~ 0
 Drive_W_Temp
-Text Label 6625 4775 0    50   ~ 0
+Text Label 6625 4375 0    50   ~ 0
 Subscribe_Temp
 $Comp
@@
 Text Label 6625 5075 0    50   ~ 0
 USARTX_RX
-Text Label 6625 4175 0    50   ~ 0
+Text Label 2225 6975 2    50   ~ 0
 ADC_~RST~_Pin
-Text Label 6625 4075 0    50   ~ 0
+Text Label 6625 6075 0    50   ~ 0
 PWR_ON_Pin
-Text Label 2225 6275 2    50   ~ 0
-OUT_U_Current
-Text Label 6625 5775 0    50   ~ 0
+Text Label 2225 6075 2    50   ~ 0
 OUT_V_Current
-Text Label 6625 5875 0    50   ~ 0
+Text Label 2225 5875 2    50   ~ 0
 OUT_W_Current
 Wire Wire Line
 	6625 5975 7300 5975
-Text Label 2225 5875 2    50   ~ 0
+Text Label 6625 5575 0    50   ~ 0
 LED0
-Text Label 2225 5975 2    50   ~ 0
+Text Label 6625 6375 0    50   ~ 0
 LED1
 Text Label 6625 6275 0    50   ~ 0
@@
 Text Label 2225 7075 2    50   ~ 0
 SW0
-Text Label 6625 6775 0    50   ~ 0
-ADRESS_0
-Text Label 6625 6875 0    50   ~ 0
-ADRESS_1
 Text Label 6625 6975 0    50   ~ 0
 ADRESS_2
@@
 Wire Wire Line
 	1725 13775 1650 13775
-Text Label 2225 6775 2    50   ~ 0
+Text Label 2225 6475 2    50   ~ 0
 HALL_0
-Text Label 2225 6875 2    50   ~ 0
+Text Label 2225 6575 2    50   ~ 0
 HALL_1
-Text Label 2225 6975 2    50   ~ 0
+Text Label 2225 6675 2    50   ~ 0
 HALL_2
 Text Label 2225 6375 2    50   ~ 0
@@
 Wire Wire Line
 	2250 14575 2200 14575
+Text Label 6625 4075 0    50   ~ 0
+Drive_U_Temp
+Text Label 6625 4175 0    50   ~ 0
+OUT_U_Current
+Text Label 6625 6875 0    50   ~ 0
+ADRESS_1
+Text Label 6625 6775 0    50   ~ 0
+ADRESS_0
+Text Label 6625 6475 0    50   ~ 0
+LED2
+$Comp
+L Device:LED D28
+U 1 1 5E9EDAB1
+P 3525 12050
+F 0 "D28" V 3564 11933 50  0000 R CNN
+F 1 "MODE" V 3473 11933 50  0000 R CNN
+F 2 "LED_SMD:LED_0603_1608Metric" H 3525 12050 50  0001 C CNN
+F 3 "~" H 3525 12050 50  0001 C CNN
+	1    3525 12050
+	0    -1   -1   0
+$EndComp
+$Comp
+L Device:R R66
+U 1 1 5E9EDABB
+P 3525 11750
+F 0 "R66" H 3595 11796 50  0000 L CNN
+F 1 "330" H 3595 11705 50  0000 L CNN
+F 2 "Mizz_lib:1608_WP" V 3455 11750 50  0001 C CNN
+F 3 "~" H 3525 11750 50  0001 C CNN
+	1    3525 11750
+	1    0    0    -1
+$EndComp
+$Comp
+L power:GND #PWR0250
+U 1 1 5E9EDAC5
+P 3525 12200
+F 0 "#PWR0250" H 3525 11950 50  0001 C CNN
+F 1 "GND" H 3530 12027 50  0000 C CNN
+F 2 "" H 3525 12200 50  0001 C CNN
+F 3 "" H 3525 12200 50  0001 C CNN
+	1    3525 12200
+	1    0    0    -1
+$EndComp
+Text Label 3525 11600 2    50   ~ 0
+LED2
 $EndSCHEMATC
