File: CAN_BLDCMD_type0/CAN_BLDCMD.kicad_pcb (KiCad board)
At the start: 2 copper layers, 179 parts, among them J1 SWD, J10 BATT_IN, J11 OUT_U, J12 OUT_V, J13 OUT_W, J2 CAN, J3 CAN, J4 ENC, J5 I/O0, J6 I/O1, J7 SERIAL, J8 FAN, J9 BATT_IN, Q1 MOSFET_N, Q2 MOSFET_N, Q3 MOSFET_N, Q4 MOSFET_N, Q5 MOSFET_N, Q6 MOSFET_N, SW1 SW0, SW2 SW1, U1 MAX3051, U10 SI8900, U11 ADC_~RST, U12 ACS758, U13 ACS758, U14 ACS758, U15 BD9G101G, U16 LTC2644, U17 LTC2644, U18 BD33FA1, U19 LOGO, U2 BD9G101G, U3 STM32F405RG, U4 AZ1086H, U5 SW_ROTARY_16, U6 POWER_ON, U7 SI8274, U8 SI8274, U9 SI8274, Y1 8MHz

Commit message: BLDCMD本格的に設計開始
Parts:
- added J14: VALVE, Mizz_lib:XA_4L, F.Cu at (186.5, 151.8)
- C49: value 1500u -> 2200u
- C55, C57, R34, R4, U1: moved to B.Cu
- JP2: value Jumper -> CAN_JP
- R39, R40, R41, R42, R43, R44: value 1 -> 10
- U5: value SW_ROTARY_16 -> ADRESS
- moved J7 200.6 mm to (228.5, 127.8), turned to 270 degrees
- moved J10 199.3 mm to (235.6, 75.5), turned to 180 degrees
- moved U3 171.7 mm to (215.0, 121.0), turned to 315 degrees
- moved J9 168.8 mm to (235.6, 83.8), turned to 180 degrees
- moved C49 166.7 mm to (232.6, 64.8)
- moved C55 161.4 mm to (235.6, 87.2)
- moved J6 161.1 mm to (198.7, 134.8)
- moved J4 150.5 mm to (208.7, 134.8)
- moved U10 149.5 mm to (236.8, 103.8), turned to 90 degrees
- moved C50 145.7 mm to (239.4, 93.1)
- moved J5 144.3 mm to (188.7, 134.8)
- moved U5 138.1 mm to (234.5, 119.8)
- moved J2 135.0 mm to (182.8, 115.2), turned to 270 degrees
- moved J3 130.6 mm to (182.8, 127.7), turned to 270 degrees
- moved U9 129.1 mm to (223.1, 103.8), turned to 90 degrees
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Routing:
- net /OUT_U: track 0.00 -> 25.8 mm, vias 0 -> 1
- net Net-(R33-Pad2): track 0.00 -> 22.7 mm
- net Net-(R34-Pad2): track 0.00 -> 17.8 mm, vias 0 -> 1
- net GNDPWR: track 0.00 -> 11.9 mm
- net Net-(Q1-PadG): track 0.00 -> 7.80 mm, vias 0 -> 1
- net Net-(C36-Pad1): track 0.00 -> 4.74 mm
- net Net-(D8-Pad2): track 0.00 -> 2.06 mm
- net (no net): vias 0 -> 4
- added copper zone on B.Cu, net +BATT
- added copper zone on B.Cu, net /OUT_U
- added copper zone on F.Cu, net /OUT_U
- added copper zone on B.Cu, net /OUT_V
- added copper zone on F.Cu, net /OUT_V
- added copper zone on B.Cu, net /OUT_W
- added copper zone on F.Cu, net /OUT_W
Other:
- board outline added: 70 x 90 mm

Commit message: BLDC(仮)が形になってきた
Parts:
- added C61: 1u, Mizz_lib:1608_WP, F.Cu at (146.9, 109.8)
- added C62: 1u, Mizz_lib:1608_WP, F.Cu at (146.9, 111.8)
- added C63: 0.1u, Mizz_lib:1608_WP, F.Cu at (145.6, 116.5)
- added C64: 0.1u, Mizz_lib:1608_WP, F.Cu at (149.6, 129.7)
- added D17: DIODE, Diode_SMD:D_SOD-123, B.Cu at (191.5, 137.5)
- added D18: DIODE, Diode_SMD:D_SOD-123, B.Cu at (196.5, 137.5)
- added D19: VALVE0, LED_SMD:LED_0603_1608Metric, F.Cu at (190.8, 132.5)
- added D20: VALVE1, LED_SMD:LED_0603_1608Metric, F.Cu at (195.9, 132.5)
- added D21: 12V, LED_SMD:LED_0603_1608Metric, F.Cu at (185.4, 128.0)
- added D22: 5V, LED_SMD:LED_0603_1608Metric, F.Cu at (266.0, 43.1)
- added D23: 3V3, LED_SMD:LED_0603_1608Metric, F.Cu at (270.1, 40.5)
- added D24: BATT, LED_SMD:LED_0603_1608Metric, F.Cu at (235.8, 57.0)
- added D25: MAIN_BATT, LED_SMD:LED_0603_1608Metric, F.Cu at (270.1, 43.1)
- added D26: 12VP, LED_SMD:LED_0603_1608Metric, F.Cu at (180.1, 99.2)
- added D27: 3V3P, LED_SMD:LED_0603_1608Metric, F.Cu at (270.1, 45.7)
- added Q7: NPN, Package_TO_SOT_SMD:SOT-23, B.Cu at (189.8, 131.0)
- added Q8: NPN, Package_TO_SOT_SMD:SOT-23, B.Cu at (194.8, 131.0)
- added R54: 10k, Mizz_lib:1608_WP, F.Cu at (146.9, 113.8)
- added R55: 10k, Mizz_lib:1608_WP, F.Cu at (141.2, 125.5)
- added R56: 330, Mizz_lib:1608_WP, B.Cu at (187.4, 130.9)
- added R57: 330, Mizz_lib:1608_WP, B.Cu at (192.4, 130.9)
- added R58: 1.2k, Mizz_lib:1608_WP, F.Cu at (185.4, 130.1)
- added R59: 510, Mizz_lib:1608_WP, F.Cu at (277.9, 40.2)
- added R60: 330, Mizz_lib:1608_WP, F.Cu at (273.9, 44.8)
- added R61: 4.7k, Mizz_lib:1608_WP, F.Cu at (232.5, 57.0)
- added R62: 4.7k, Mizz_lib:1608_WP, F.Cu at (273.9, 46.8)
- added R63: 2.2k, Mizz_lib:1608_WP, F.Cu at (180.1, 96.0)
- added R64: 510, Mizz_lib:1608_WP, F.Cu at (277.5, 46.8)
- added SW3: RST, Button_Switch_SMD:SW_SPST_CK_RS282G05A3, F.Cu at (238.5, 135.8)
- added U20: AQM0802, Mizz_lib:AQM0802_original, F.Cu at (194.3, 110.5)
- C47, C48, D3, U11, U15, U18, U6: moved to B.Cu
- R13, R14: value R -> 330
- moved J1 167.2 mm to (234.5, 130.8)
- moved D5 165.2 mm to (185.2, 153.3)
- moved D13 154.5 mm to (226.2, 96.8)
- moved SW1 152.7 mm to (238.8, 116.2), turned to 180 degrees
- moved U18 152.6 mm to (263.8, 113.5), turned to 90 degrees
- moved SW2 143.9 mm to (238.8, 112.2), turned to 180 degrees
- moved R47 143.4 mm to (257.5, 103.8), turned to 180 degrees
- moved C48 139.3 mm to (253.6, 90.8)
- moved U6 135.4 mm to (233.8, 103.8), turned to 270 degrees
- moved L1 134.1 mm to (204.3, 156.7)
- moved U11 132.0 mm to (238.5, 103.8), turned to 90 degrees
- moved C47 126.0 mm to (258.1, 97.0), turned to 270 degrees
- moved U15 122.1 mm to (255.8, 97.0), turned to 90 degrees
- moved R44 121.6 mm to (226.2, 95.0)
- moved J8 121.0 mm to (239.6, 93.5), turned to 90 degrees
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Connections:
- C58 pad 1: Net-(C58-Pad1) -> +12P
- C59 pad 1: Net-(C58-Pad1) -> +12P
- D16 pad 1: Net-(C58-Pad1) -> +12P
- J14 pad 2: Net-(J14-Pad2) -> +12V
- J14 pad 4: Net-(J14-Pad4) -> +12V
- SW1 pad 1: Net-(SW1-Pad1) -> GND
- SW2 pad 1: Net-(SW2-Pad1) -> GND
- U18 pad 3: Net-(C58-Pad1) -> +12P
Routing:
- net +12V: track 0.00 -> 26.2 mm
- net /Drive_U_Temp: track 0.00 -> 21.1 mm, vias 0 -> 3
- net +BATT: track 0.00 -> 8.91 mm, vias 0 -> 102
- net GNDPWR: track 11.9 -> 20.2 mm, vias 0 -> 16
- net /OUT_U: track 25.8 -> 19.7 mm, vias 1 -> 40
- net Net-(D18-Pad1): track 0.00 -> 5.62 mm
- net Net-(D17-Pad1): track 0.00 -> 5.62 mm
- net Net-(D20-Pad2): track 0.00 -> 2.95 mm, vias 0 -> 1
- net Net-(D19-Pad2): track 0.00 -> 2.95 mm, vias 0 -> 1
- net Net-(D24-Pad2): track 0.00 -> 1.56 mm
- net /VALVE_1: track 0.00 -> 1.35 mm
- net /VALVE_0: track 0.00 -> 1.35 mm
- net Net-(C12-Pad1): track 0.00 -> 1.25 mm
- net Net-(R34-Pad2): track 17.8 -> 17.0 mm
- net Net-(Q6-PadS): vias 0 -> 10
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- added copper zone on F.Cu, net +BATT
- added copper zone on B.Cu, net GND
- added copper zone on F.Cu, net GND
- added copper zone on B.Cu, net GNDPWR
- added copper zone on F.Cu, net GNDPWR
- added copper zone on B.Cu, net Net-(Q2-PadS)
- added copper zone on F.Cu, net Net-(Q2-PadS)
- added copper zone on B.Cu, net Net-(Q4-PadS)
- added copper zone on F.Cu, net Net-(Q4-PadS)
- added copper zone on B.Cu, net Net-(Q6-PadS)
- added copper zone on F.Cu, net Net-(Q6-PadS)
Other:
- outline, holes or cut-outs redrawn
- board text added: "+"
- board text added: "Brushless DC-Motor Driver Type-0 ver.0.0 Virgo Spica."
- board text removed: "Virgo Spica"

Commit message: いろいろ修正しました
Parts:
- added J15: HALL_IN, Mizz_lib:ZH_6P, F.Cu at (234.9, 112.3)
- added R65: 10k, Mizz_lib:1608_WP, F.Cu at (140.3, 86.5)
- added SW4: MODE, Mizz_lib:SW_Micro_SPST, F.Cu at (234.2, 139.8)
- D14, D16: value DIODE] -> DIODE
- D15: footprint Diode_SMD:D_SMA -> Diode_SMD:D_2010_5025Metric_Pad1.52x2.65mm_HandSolder
- R47: footprint Mizz_lib:R_2812 -> Resistor_SMD:R_2512_6332Metric
- SW1, SW2: footprint Button_Switch_SMD:SW_SPST_CK_RS282G05A3 -> Button_Switch_SMD:SW_SPST_PTS810
- moved U16 97.1 mm to (209.5, 57.2), turned to 180 degrees
- moved U17 87.2 mm to (226.8, 57.2), turned to 180 degrees
- moved R49 83.4 mm to (196.5, 48.2), turned to 270 degrees
- moved R48 54.0 mm to (195.0, 48.2), turned to 90 degrees
- moved R47 12.5 mm to (250.8, 114.2)
- moved SW3 2.01 mm to (238.7, 133.8)
- moved SW2 1.96 mm to (240.7, 112.8)
- moved SW1 1.90 mm to (240.7, 116.2)
- moved J7 1.35 mm to (227.9, 126.0)
- moved J1 1.20 mm to (234.6, 129.6)
- moved U5 0.60 mm to (238.6, 123.2)
- moved D15 0.25 mm to (234.0, 91.2)
Connections:
- D1 pad 1: Net-(D1-Pad1) -> +3V3
- J1 pad 2: Net-(D1-Pad2) -> Net-(J1-Pad2)
- JP1 pad 1: Net-(D1-Pad1) -> Net-(J1-Pad2)
- JP1 pad 2: +3V3 -> Net-(D1-Pad2)
- U3 pad 37: Net-(U3-Pad37) -> /SW_MODE
- U3 pad 51: Net-(U3-Pad51) -> /HALL_0
- U3 pad 52: Net-(U3-Pad52) -> /HALL_1
- U3 pad 53: Net-(U3-Pad53) -> /HALL_2
Routing:
- net +BATT: track 8.91 -> 10.7 mm

Commit message: BLDC 途中
Parts:
- added D28: MODE, LED_SMD:LED_0603_1608Metric, F.Cu at (232.8, 117.3)
- added R66: 330, Mizz_lib:1608_WP, F.Cu at (154.1, 140.4)
- C24, C61, C62, C63, R45, R54, R55: moved to B.Cu
- D15: footprint Diode_SMD:D_2010_5025Metric_Pad1.52x2.65mm_HandSolder -> Diode_SMD:D_SOD-123
- D5: value LED -> BUS
- D6: value LED -> EMG
- moved D6 199.7 mm to (232.8, 115.9), turned to 180 degrees
- moved R32 177.1 mm to (230.1, 92.7), turned to 180 degrees
- moved C24 112.1 mm to (230.2, 120.2), turned to 270 degrees
- moved U19 107.2 mm to (210.8, 120.2)
- moved R45 93.9 mm to (229.6, 98.0), turned to 90 degrees
- moved R55 71.4 mm to (212.3, 131.9), turned to 90 degrees
- moved R54 69.3 mm to (213.8, 131.9), turned to 90 degrees
- moved C63 65.5 mm to (209.3, 131.9), turned to 90 degrees
- moved C62 63.3 mm to (207.1, 131.4)
- moved C61 62.0 mm to (204.8, 131.9), turned to 270 degrees
- moved D5 61.4 mm to (232.8, 114.5), turned to 180 degrees
- moved C50 23.8 mm to (234.7, 95.3), turned to 180 degrees
- moved U15 23.7 mm to (232.0, 98.1), turned to 0 degrees
- moved C48 19.1 mm to (235.6, 97.1)
- moved U8 3.85 mm to (200.9, 103.6)
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Connections:
- U3 pad 10: /LED1 -> /Drive_V_Temp
- U3 pad 11: Net-(U3-Pad11) -> /OUT_V_Current
- U3 pad 14: /PWR_ON_Pin -> /Drive_U_Temp
- U3 pad 15: /ADC_~RST~_Pin -> /OUT_U_Current
- U3 pad 16: /USARTx_TX -> Net-(U3-Pad16)
- U3 pad 17: /USARTx_RX -> /Subscribe_Temp
- U3 pad 20: /Drive_U_Temp -> Net-(U3-Pad20)
- U3 pad 21: /Drive_V_Temp -> Net-(U3-Pad21)
- U3 pad 22: /Drive_W_Temp -> Net-(U3-Pad22)
- U3 pad 23: /Subscribe_Temp -> Net-(U3-Pad23)
- U3 pad 25: /OUT_U_Current -> Net-(U3-Pad25)
- U3 pad 26: /OUT_V_Current -> Net-(U3-Pad26)
- U3 pad 27: /OUT_W_Current -> Net-(U3-Pad27)
- U3 pad 38: Net-(U3-Pad38) -> /HALL_0
- U3 pad 39: Net-(U3-Pad39) -> /HALL_1
- U3 pad 40: Net-(U3-Pad40) -> /HALL_2
- U3 pad 50: Net-(U3-Pad50) -> /LED0
- U3 pad 51: /HALL_0 -> /USARTx_TX
- U3 pad 52: /HALL_1 -> /USARTx_RX
- U3 pad 53: /HALL_2 -> /ADC_~RST~_Pin
- U3 pad 55: Net-(U3-Pad55) -> /PWR_ON_Pin
- U3 pad 58: Net-(U3-Pad58) -> /LED1
- U3 pad 59: Net-(U3-Pad59) -> /LED2
- U3 pad 8: Net-(U3-Pad8) -> /Drive_W_Temp
- U3 pad 9: /LED0 -> /OUT_W_Current
Routing:
- net +3V3: track 0.00 -> 17.8 mm
- net Net-(R32-Pad2): track 0.00 -> 11.7 mm, vias 0 -> 1
- net +BATT: track 10.7 -> 16.5 mm
- net +5V: track 0.00 -> 2.22 mm
- net Net-(C62-Pad1): track 0.00 -> 1.41 mm
- net Net-(C62-Pad2): track 0.00 -> 1.41 mm
- net Net-(C61-Pad1): track 0.00 -> 0.95 mm
- net /I2Cx_SDA: track 0.00 -> 0.95 mm
- net /I2Cx_SCL: track 0.00 -> 0.95 mm
Other:
- board text added: "0"
- board text added: "1"
- board text added: "SW"

Commit message: BLDCMD type0
Parts:
- C48, R45, U15: moved to F.Cu
- moved L2 151.5 mm to (251.5, 103.0)
- moved R45 24.2 mm to (253.8, 98.2)
- moved U15 19.3 mm to (251.3, 98.2), turned to 180 degrees
- moved C48 13.1 mm to (248.7, 98.2), turned to 270 degrees
- moved C40 7.50 mm to (212.4, 99.0)
- moved C41 7.50 mm to (218.8, 99.0)
- moved D12 7.50 mm to (212.4, 96.8)
- moved D13 7.50 mm to (218.8, 96.8)
- moved R43 7.50 mm to (212.4, 95.0)
- moved R44 7.50 mm to (218.8, 95.0)
- moved U9 7.50 mm to (215.6, 103.8)
- moved U10 5.75 mm to (230.5, 103.7)
- moved J8 0.35 mm to (239.6, 93.2)
- moved C38 0.20 mm to (197.8, 99.0)
- moved C39 0.20 mm to (204.2, 99.0)
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Routing:
- net Net-(R32-Pad2): track 11.7 -> 0.00 mm, vias 1 -> 0

Commit message: 電流制御用のMDのコンデンサの配置ミスがあったため，直した
Parts:
- moved L2 12.5 mm to (239.5, 99.4), turned to 180 degrees
Changed lines of the file:
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@@
   )
   (setup
-    (last_trace_width 0.5)
+    (last_trace_width 0.25)
     (user_trace_width 0.2)
     (user_trace_width 0.3)
@@
   )
   (module Mizz_lib:Inductor_Taiyo-Yuden_NR-50xx_HandSoldering (layer F.Cu)
-    (at 251.5 102.975)
+    (at 239.5 99.4 180)
     (descr "Inductor, Taiyo Yuden, NR series, Taiyo-Yuden_NR-50xx, 4.9mmx4.9mm")
     (tags "inductor taiyo-yuden nr smd")
@@
     (fp_line (start -2.45 -1.65) (end -1.65 -2.45) (layer F.Fab) (width 0.15))
     (fp_line (start -2.45 0) (end -2.45 -1.65) (layer F.Fab) (width 0.15))
-    (pad 2 smd rect (at 2.25 0) (size 2.4 4.2) (layers F.Cu F.Paste F.Mask)
+    (pad 2 smd rect (at 2.25 0 180) (size 2.4 4.2) (layers F.Cu F.Paste F.Mask)
       (net 34 /FB_12P))
-    (pad 1 smd rect (at -2.25 0) (size 2.4 4.2) (layers F.Cu F.Paste F.Mask)
+    (pad 1 smd rect (at -2.25 0 180) (size 2.4 4.2) (layers F.Cu F.Paste F.Mask)
       (net 39 "Net-(C47-Pad1)"))
     (model Inductors.3dshapes/Inductor_Taiyo-Yuden_NR-50xx.wrl
