File: PowerMD_ver1-0_another/SteerMD.sch (KiCad schematic (older format))
At the start: 218 parts, among them P1 SWD, P10 OUT_1, P11 ENC_0, P13 ENC_1, P14 I/O_1, P15 OUT_0, P2 MOTOR_COOLING, P3 CAN, P4 CAN, P5 SERIAL, P6 I/O_0, P7 FAN, P8 BATT_IN, P9 BATT_IN, Q1 MOSFET_N, Q2 MOSFET_N, Q3 MOSFET_N, Q4 MOSFET_N, Q5 MOSFET_N, Q6 MOSFET_N, Q7 MOSFET_N, Q8 MOSFET_N, SW1 RST, SW3 SW0, SW4 SW1, U1 MAX3051, U10 ACS758, U11 POWER_ON, U12 SI8274, U13 ACS758, U14 SI8274, U15 AZ1086H, U16 LOGO, U17 AQM0802, U19 ADRESS, U2 BD9G101, U2 MCP16331, U3 STM32F405RG, U4 SI8274, U5 SI8900, U6 ADC_~RST, U8 SI8274, U9 BD33FA1, Y1 8MHz

Commit message: Add project Power-MD ver.1.0 another-0
Parts:
- removed D10, D6: DIODE, Diode_SMD:D_SOD-123, symbol Miz:DIODE_rev
- removed U2: MCP16331, Package_SO:TSOP-6_1.65x3.05mm_P0.95mm, symbol SteerMD-rescue:MCP16331-Miz
- added C27, C51, C65, C66, C67: 0.1u, Mizz_lib:1608_WP, symbol SteerMD-rescue:C-Device-MD_Enbarr_x2-rescue-F4_CAN_DCMD-rescue
- added D10, D12, D17, D25, D28, D6: DIODE, Diode_SMD:D_SOD-123, symbol SteerMD-rescue:DIODE-device-MD_Enbarr_x2-rescue-F4_CAN_DCMD-rescue
- added R75, R77: 10k, Mizz_lib:1608_WP, symbol SteerMD-rescue:R-Device-MD_Enbarr_x2-rescue-F4_CAN_DCMD-rescue
- added R76, R78: 1k, Mizz_lib:1608_WP, symbol SteerMD-rescue:R-Device-MD_Enbarr_x2-rescue-F4_CAN_DCMD-rescue
- added U18: LTC2644, Package_SO:MSOP-12_3x4mm_P0.65mm, symbol Miz:LTC2644
- added U7: MCP16331, Package_SO:TSOP-6_1.65x3.05mm_P0.95mm, symbol Miz:MCP16331
Connections:
- net labels added: MOTOR0_OUT, MOTOR1_OUT
- wire segments 337 -> 363
