File: PowerMD_ver1-1_another/SteerMD.sch (KiCad schematic (older format))
At the start: 218 parts, among them P1 SWD, P10 OUT_1, P11 ENC_0, P13 ENC_1, P14 I/O_1, P15 OUT_0, P2 MOTOR_COOLING, P3 CAN, P4 CAN, P5 SERIAL, P6 I/O_0, P7 FAN, P8 BATT_IN, P9 BATT_IN, Q1 MOSFET_N, Q2 MOSFET_N, Q3 MOSFET_N, Q4 MOSFET_N, Q5 MOSFET_N, Q6 MOSFET_N, Q7 MOSFET_N, Q8 MOSFET_N, SW1 RST, SW3 SW0, SW4 SW1, U1 MAX3051, U10 ACS758, U11 POWER_ON, U12 SI8274, U13 ACS758, U14 SI8274, U15 AZ1086H, U16 LOGO, U17 AQM0802, U19 ADRESS, U2 BD9G101, U2 MCP16331, U3 STM32F405RG, U4 SI8274, U5 SI8900, U6 ADC_~RST, U8 SI8274, U9 BD33FA1, Y1 8MHz

Commit message: Add project Power-MD ver.1.0 another-0
Parts:
- U2: symbol Miz:MCP16331 -> SteerMD-rescue:MCP16331-Miz
Changed lines of the file:
@@
 EESchema Schematic File Version 4
-LIBS:SteerMD-cache
 EELAYER 30 0
 EELAYER END
@@
 	11125 1850 11125 2275
 Wire Wire Line
-	11125 2375 11125 2475
-Wire Wire Line
 	11225 2375 11425 2375
 Connection ~ 11225 2375
@@
 	13600 2725 13750 2725
 $Comp
-L Miz:MCP16331 U2
-U 1 1 5E871719
-P 10725 2475
-F 0 "U2" H 10725 2940 50  0000 C CNN
-F 1 "MCP16331" H 10725 2849 50  0000 C CNN
-F 2 "Package_SO:TSOP-6_1.65x3.05mm_P0.95mm" H 10725 2475 50  0001 C CNN
-F 3 "" H 10725 2475 50  0001 C CNN
-	1    10725 2475
-	1    0    0    -1
-$EndComp
-Connection ~ 11125 2275
-Wire Wire Line
-	11125 2475 11125 2675
-Connection ~ 11125 2475
-$Comp
 L Miz:DIODE_rev D6
 U 1 1 5E8AD331
@@
 Wire Wire Line
 	13750 2725 13900 2725
+Connection ~ 11125 2475
+Connection ~ 11125 2275
+Wire Wire Line
+	11125 2475 11125 2675
+Wire Wire Line
+	11125 2375 11125 2475
+$Comp
+L SteerMD-rescue:MCP16331-Miz U2
+U 1 1 5E871719
+P 10725 2475
+F 0 "U2" H 10725 2940 50  0000 C CNN
+F 1 "MCP16331" H 10725 2849 50  0000 C CNN
+F 2 "Package_SO:TSOP-6_1.65x3.05mm_P0.95mm" H 10725 2475 50  0001 C CNN
+F 3 "" H 10725 2475 50  0001 C CNN
+	1    10725 2475
+	1    0    0    -1
+$EndComp
 $EndSCHEMATC
