File: PowerMD_ver1-another/SteerMD.kicad_pcb (KiCad board)
At the start: 2 copper layers, 75 x 88 mm, 232 parts, among them P1 SWD, P10 OUT_1, P11 ENC_0, P13 ENC_1, P14 I/O_1, P15 OUT_0, P2 MOTOR_COOLING, P3 CAN, P4 CAN, P5 SERIAL, P6 I/O_0, P7 FAN, P8 BATT_IN, P9 BATT_IN, Q1 MOSFET_N, Q2 MOSFET_N, Q3 MOSFET_N, Q4 MOSFET_N, Q5 MOSFET_N, Q6 MOSFET_N, Q7 MOSFET_N, Q8 MOSFET_N, SW1 RST, SW3 SW0, SW4 SW1, U1 MAX3051, U10 ACS758, U11 POWER_ON, U12 SI8274, U13 ACS758, U14 SI8274, U15 AZ1086H, U16 LOGO, U17 AQM0802, U18 LTC2644, U19 ADRESS, U2 BD9G101, U3 STM32F405RG, U4 SI8274, U5 SI8900, U6 ADC_~RST, U7 MCP16331, U8 SI8274, U9 BD33FA1, Y1 8MHz

Commit message: ビアの開け方(この前ちらっとネット上で観測した開け方参考)により，放熱性能が上がるかチェックするMD作成
Parts:
- removed C27, C51, C65, C66, C67: 0.1u, Mizz_lib:1608_WP
- removed D12, D17, D25, D28: DIODE, Diode_SMD:D_SOD-123
- removed R75, R77: 10k, Mizz_lib:1608_WP
- removed R76, R78: 1k, Mizz_lib:1608_WP
- removed U18: LTC2644, Package_SO:MSOP-12_3x4mm_P0.65mm
- removed U7: MCP16331, Package_SO:TSOP-6_1.65x3.05mm_P0.95mm
- U2: value BD9G101 -> MCP16331
- moved U2 63.5 mm to (135.2, 69.0), turned to 90 degrees
- moved D10 32.1 mm to (144.8, 71.8), turned to 90 degrees
- moved D6 28.8 mm to (144.8, 67.0), turned to 270 degrees
Connections:
- D10 pad 1: Net-(D10-Pad1) -> /FB_PWR_OUT
- D10 pad 2: /OUT1_R -> Net-(D10-Pad2)
- D6 pad 1: Net-(D10-Pad1) -> Net-(C23-Pad1)
- D6 pad 2: /OUT1_L -> Net-(D10-Pad2)
- U2 pad 1: Net-(C39-Pad2) -> Net-(C23-Pad2)
- U2 pad 2: GND -> GNDPWR
- U2 pad 3: /FB -> /FB_PWR
- U2 pad 4: +12V -> /batt
- U2 pad 5: +12V -> /batt
- U2 pad 6: Net-(C39-Pad1) -> Net-(C23-Pad1)
Routing:
- net GNDPWR: track 152.5 -> 87.3 mm, vias 38 -> 35
- net /MOTOR0_VOLTAGE_DAC: track 63.7 -> 0.00 mm, vias 2 -> 0
- net /MOTOR1_VOLTAGE_DAC: track 62.4 -> 0.00 mm, vias 2 -> 0
- net +3.3VP: track 93.2 -> 48.3 mm, vias 5 -> 3
- net /OUT1_R: track 43.1 -> 26.8 mm, vias 30 -> 29
- net /OUT0_L: track 49.8 -> 34.5 mm, vias 36 -> 35
- net /OUT0_R: track 36.6 -> 23.9 mm, vias 33 -> 32
- net /OUT1_L: track 36.1 -> 24.0 mm, vias 24 -> 23
- net /MOTOR0_OUT: track 11.1 -> 0.00 mm
- net /MOTOR1_OUT: track 10.8 -> 0.00 mm
- net Net-(D10-Pad1): track 6.73 -> 0.00 mm
- net Net-(D12-Pad1): track 6.65 -> 0.00 mm
- net /FB_PWR_OUT: track 11.3 -> 16.1 mm, vias 2 -> 3
- net Net-(C23-Pad1): track 8.85 -> 12.7 mm, vias 0 -> 1
- net Net-(D10-Pad2): track 0.00 -> 1.45 mm
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Other:
- board text added: "CAN DC-MotroDriver Aqualius Sadalmeric ver.1.0-another edition."
- board text removed: "CAN DC-MotroDriver Aqualius Sadalmeric ver.1.0-0 another"
