File: CAN_DCMD_Normal_ver0/NormalMD.kicad_pcb (KiCad board)
At the start: 2 copper layers, 75 x 88 mm, 224 parts, among them P1 SWD, P10 OUT_1, P11 ENC_0, P13 ENC_1, P14 I/O_1, P15 OUT_0, P2 VALVE, P3 CAN, P4 CAN, P5 SERIAL, P6 I/O_0, P7 FAN, P8 BATT_IN, P9 BATT_IN, Q1 MOSFET_N, Q10 NPN, Q2 MOSFET_N, Q3 MOSFET_N, Q4 MOSFET_N, Q5 MOSFET_N, Q6 MOSFET_N, Q7 MOSFET_N, Q8 MOSFET_N, Q9 NPN, SW1 RST, SW3 SW0, SW4 SW1, U1 MAX3051, U11 POWER_ON, U12 SI8274, U14 SI8274, U15 AZ1086H, U16 LOGO, U17 AQM0802, U19 ADRESS, U2 BD9G101, U3 STM32F405RG, U4 SI8274, U5 SI8900, U6 ADC_~RST, U7 BD9G101G, U8 SI8274, U9 BD33FA1, Y1 8MHz

Commit message: 配置しただけで分かるやばいやつ
Connections:
- U3 pad 50: Net-(U3-Pad50) -> /VALVE0
- U3 pad 51: Net-(U3-Pad51) -> /VALVE1
Routing:
- net /VALVE0: track 6.79 -> 49.6 mm, vias 0 -> 1
- net /VALVE1: track 6.36 -> 46.0 mm, vias 0 -> 1
- net +BATT: track 127.9 -> 126.5 mm
Other:
- board text added: "CAN DC-MotroDriver Leo Regulus ver.0.1"
- board text added: "Vdd"
- board text removed: "CAN DC-MotroDriver Leo Regulus ver.0.0"

Commit message: 電流制御MD(仮)配線(仮)完成(仮)
Parts:
- R37: value 50k -> 3.9k
- R38: value 10k -> 680
- R57, R60, R75, R76: value 2m -> 1m
Changed lines of the file:
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@@
   )
   (setup
-    (last_trace_width 0.8)
+    (last_trace_width 0.25)
     (user_trace_width 0.2)
     (user_trace_width 0.3)
@@
       (effects (font (size 1 1) (thickness 0.15)) (justify mirror))
     )
-    (fp_text value 50k (at -2.45 0 90) (layer B.SilkS)
+    (fp_text value 3.9k (at -2.45 0 90) (layer B.SilkS)
       (effects (font (size 0.8 0.8) (thickness 0.15)) (justify mirror))
     )
@@
       (effects (font (size 1 1) (thickness 0.15)) (justify mirror))
     )
-    (fp_text value 10k (at 2.5 0) (layer B.SilkS)
+    (fp_text value 680 (at 2.5 0) (layer B.SilkS)
       (effects (font (size 0.8 0.8) (thickness 0.15)) (justify mirror))
     )
@@
       (effects (font (size 1 1) (thickness 0.15)) (justify mirror))
     )
-    (fp_text value 2m (at 0 -0.05 90) (layer B.SilkS)
+    (fp_text value 1m (at 0 -0.05 90) (layer B.SilkS)
       (effects (font (size 1 1) (thickness 0.15)) (justify mirror))
     )
@@
       (effects (font (size 1 1) (thickness 0.15)) (justify mirror))
     )
-    (fp_text value 2m (at 0 0 90) (layer B.SilkS)
+    (fp_text value 1m (at 0 0 90) (layer B.SilkS)
       (effects (font (size 1 1) (thickness 0.15)) (justify mirror))
     )
@@
       (effects (font (size 1 1) (thickness 0.15)) (justify mirror))
     )
-    (fp_text value 2m (at 0 0 270) (layer B.SilkS)
+    (fp_text value 1m (at 0 0 270) (layer B.SilkS)
       (effects (font (size 1 1) (thickness 0.15)) (justify mirror))
     )
@@
       (effects (font (size 1 1) (thickness 0.15)) (justify mirror))
     )
-    (fp_text value 2m (at 0 0 270) (layer B.SilkS)
+    (fp_text value 1m (at 0 0 270) (layer B.SilkS)
       (effects (font (size 1 1) (thickness 0.15)) (justify mirror))
     )

Commit message: いろいろ修正しました
Changed lines of the file:
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@@
       (effects (font (size 1 1) (thickness 0.15)))
     )
-    (fp_text value SI8274 (at 0 5.9 90) (layer F.Fab)
+    (fp_text value SI8274 (at 0 5.9 90) (layer F.SilkS)
       (effects (font (size 1 1) (thickness 0.15)))
     )
@@
       (effects (font (size 1 1) (thickness 0.15)))
     )
-    (fp_text value SI8274 (at 0 5.9 90) (layer F.Fab)
+    (fp_text value SI8274 (at 0 5.9 90) (layer F.SilkS)
       (effects (font (size 1 1) (thickness 0.15)))
     )
@@
       (effects (font (size 1 1) (thickness 0.15)))
     )
-    (fp_text value SI8274 (at 0 5.9 90) (layer F.Fab)
+    (fp_text value SI8274 (at 0 5.9 90) (layer F.SilkS)
       (effects (font (size 1 1) (thickness 0.15)))
     )
@@
       (effects (font (size 1 1) (thickness 0.15)))
     )
-    (fp_text value SI8274 (at 0 5.9 90) (layer F.Fab)
-      (effects (font (size 1 1) (thickness 0.15)))
-    )
+    (fp_text value SI8274 (at 0 5.9 90) (layer F.SilkS)
+      (effects (font (size 1 1) (thickness 0.15)))
+    )

Commit message: 抵抗値を実装されているものに変更した
Parts:
- R40: value 4.7k -> 20k
Changed lines of the file:
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@@
-(kicad_pcb (version 20171130) (host pcbnew "(5.1.4)-1")
+(kicad_pcb (version 20171130) (host pcbnew "(5.1.5)-3")
   (general
     (thickness 1.6)
@@
       (drillshape 0)
       (scaleselection 1)
-      (outputdirectory "C:/Users/3Zuta/OneDrive/デスクトップ/NHK_RC20_PCBs/CAN_DCMD_Normal_ver0/加工/"))
+      (outputdirectory "C:/Users/3Zuta/Documents/NHK_RC20_PCBs/CAN_DCMD_Normal_ver0/加工/"))
   )
   (net 0 "")
@@
       (effects (font (size 1 1) (thickness 0.15)) (justify mirror))
     )
-    (fp_text value 4.7k (at 0 1.25 90) (layer B.SilkS)
+    (fp_text value 20k (at 0 1.25 90) (layer B.SilkS)
       (effects (font (size 0.8 0.8) (thickness 0.15)) (justify mirror))
     )
