File: PowerMD_ver1.2/SteerMD.kicad_pcb (KiCad board)
At the start: 2 copper layers, 75 x 88 mm, 217 parts, among them P1 SWD, P10 OUT_1, P11 ENC_0, P13 ENC_1, P14 I/O_1, P15 OUT_0, P2 MOTOR_COOLING, P3 CAN, P4 CAN, P5 SERIAL, P6 I/O_0, P7 FAN, P8 BATT_IN, P9 BATT_IN, Q1 MOSFET_N, Q2 MOSFET_N, Q3 MOSFET_N, Q4 MOSFET_N, Q5 MOSFET_N, Q6 MOSFET_N, Q7 MOSFET_N, Q8 MOSFET_N, SW1 RST, SW3 SW0, SW4 SW1, U1 MAX3051, U10 ACS758, U11 POWER_ON, U12 SI8274, U13 ACS758, U14 SI8274, U15 AZ1086H, U16 LOGO, U17 AQM0802, U19 ADRESS, U2 MCP16331, U3 STM32F405RG, U4 SI8274, U5 SI8900, U6 ADC_~RST, U8 SI8274, U9 BD33FA1, Y1 8MHz

Commit message: can dc-md ver.1.2
Other:
- board text added: "CAN DC-MotroDriver Aqualius Sadalmeric ver.1.2"
- board text added: "Designed by A.Mizuta in 2020/04/01."
- board text removed: "CAN DC-MotroDriver Aqualius Sadalmeric ver.1.0-1 another edition."
- board text removed: "Designed by A.Mizuta in 2020/02/22."
Changed lines of the file:
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@@
-(kicad_pcb (version 20171130) (host pcbnew "(5.1.4)-1")
+(kicad_pcb (version 20171130) (host pcbnew "(5.1.5)-3")
   (general
     (thickness 1.6)
@@
   )
   (setup
-    (last_trace_width 0.5)
+    (last_trace_width 0.25)
     (user_trace_width 0.2)
     (user_trace_width 0.3)
@@
     (effects (font (size 0.8 0.8) (thickness 0.15)) (justify mirror))
   )
-  (gr_text "CAN DC-MotroDriver\nAqualius Sadalmeric ver.1.0-1 another edition." (at 146 91.75 90) (layer F.SilkS)
+  (gr_text "CAN DC-MotroDriver\nAqualius Sadalmeric ver.1.2" (at 146 91.75 90) (layer F.SilkS)
     (effects (font (size 0.8 0.8) (thickness 0.2) italic) (justify left))
   )
@@
     (effects (font (size 2 2) (thickness 0.5)))
   )
-  (gr_text "Designed by A.Mizuta in 2020/02/22." (at 146.65 102.3 90) (layer B.SilkS)
+  (gr_text "Designed by A.Mizuta in 2020/04/01." (at 146.65 102.3 90) (layer B.SilkS)
     (effects (font (size 0.8 0.8) (thickness 0.2) italic) (justify left mirror))
   )

Commit message: MD,12V出力回路変更
Parts:
- removed D10, D6: DIODE, Diode_SMD:D_SOD-123
- added U7: BD9G101, Package_SO:TSOP-6_1.65x3.05mm_P0.95mm, B.Cu at (135.2, 69.0)
- L1: value 56uH -> 22uH
- U2: value MCP16331 -> BD9G101
- moved U2 63.6 mm to (93.1, 116.6), turned to 180 degrees
Connections:
- U2 pad 1: Net-(C23-Pad2) -> Net-(C39-Pad2)
- U2 pad 2: GNDPWR -> GND
- U2 pad 3: /FB_PWR -> /FB
- U2 pad 4: /batt -> +12V
- U2 pad 5: /batt -> +12V
- U2 pad 6: Net-(C23-Pad1) -> Net-(C39-Pad1)
Routing:
- net Net-(C23-Pad1): track 12.7 -> 8.85 mm, vias 1 -> 0
- net Net-(D10-Pad2): track 1.45 -> 0.00 mm
