File: Electricity_Manager_ver.3.0/Electricity_Manager.sch (KiCad schematic (older format))
At the start: 196 parts, among them IC2 MAIN_SHUTDOWN, IC3 RELAY_STATE, IC4 ADC_RST, J1 SERIAL, P1 SWD, P10 EMERGENCY, P11 EMERGENCY, P12 FRAME_GRAND, P13 BATT_IN, P15 OUT_B, P16 BATT_IN, P17 OUT_A, P2 CAN, P3 CAN, P4 EMERGENCY_SIGNAL, P5 EMERGENCY_SIGNAL, P6 12V_OUT, P7 12V_OUT, P8 MAIN_~RST, P9 MAIN_SW, Q1 FET_N, Q2 NPN, Q3 NPN, Q4 FET_N, Q7 FET_N, SW1 RST, SW2 SW0, SW3 SW1, U1 MAX3051, U10 BD9G101G, U11 OUTA_CHECK, U12 V23134J1052D642, U13 ACS70331, U14 OUTB_CHECK, U15 BD33FA1, U16 LOGO, U17 LOGO, U18 LOGO, U19 MCP2221A, U2 STM32F405RG, U20 OSRB38C9AA, U21 OSRB38C9AA, U22 HSIN_946, U23 LOGO, U24 LOGO, U25 LOGO, U3 FULL COLOR, U4 AQM0802_BL, U5 AP3211, U6 SI8900, U7 AZ1086H, U8 V23134J1052D642, U9 RPA60-12FW/N, X1 8MHz

Commit message: 電源基板ver.3.0の3D化&修正
Connections:
- net 24V: now also P9.1 (P1); no longer P9.2 (P2)
- net at D10.3 (Kathode): now also P9.2 (P2); no longer P9.1 (P1)
Changed lines of the file:
@@
 U 1 1 5C902D16
 P 9425 1125
-F 0 "P9" H 9502 1166 50  0000 L CNN
-F 1 "MAIN_SW" H 9502 1075 50  0000 L CNN
+F 0 "P9" H 9500 1075 50  0000 L CNN
+F 1 "MAIN_SW" H 9500 1150 50  0000 L CNN
 F 2 "Mizz_lib:XA_2T" H 9425 1125 50  0001 C CNN
 F 3 "" H 9425 1125 50  0000 C CNN
 	1    9425 1125
-	1    0    0    -1
+	1    0    0    1
 $EndComp
 $Comp
