File: CAN_BLDCMD_type2/ver.0.0/CAN_BLDCMD.sch (KiCad schematic (older format))
At the start: 203 parts, among them J1 SWD, J10 BATT_IN, J11 OUT_U, J12 OUT_V, J13 OUT_W, J14 VALVE, J15 HALL_IN, J2 CAN, J3 CAN, J4 ENC, J5 I/O0, J6 I/O1, J7 SERIAL, J8 FAN, J9 BATT_IN, Q1 MOSFET_N, Q2 MOSFET_N, Q3 MOSFET_N, Q4 MOSFET_N, Q5 MOSFET_N, Q6 MOSFET_N, Q7 NPN, Q8 NPN, SW1 SW0, SW2 SW1, SW3 RST, SW4 MODE, U1 MAX3051, U10 LM339, U11 NJM78L05, U12 ACS758, U15 BD9G101G, U19 LOGO, U2 BD9G101G, U20 AQM0802, U3 STM32F405RG, U4 AZ1086H, U5 ADRESS, U6 POWER_ON, U7 SI8274, U8 SI8274, U9 SI8274, Y1 8MHz

Commit message: 上げ忘れていた工大祭モータドライバ(前身開発基板)とJetsonNanoの電源基板関係
Parts:
- D15: symbol Miz:PWR_DIODE -> CAN_BLDCMD-rescue:PWR_DIODE-Miz
- ISO1: symbol Miz:Si866x -> CAN_BLDCMD-rescue:Si866x-Miz
- U11: symbol Miz:NJM78L00 -> CAN_BLDCMD-rescue:NJM78L00-Miz
- U5: symbol Miz:SW_ROTARY_16 -> CAN_BLDCMD-rescue:SW_ROTARY_16-Miz
Changed lines of the file:
@@
 EESchema Schematic File Version 4
+LIBS:CAN_BLDCMD-cache
 EELAYER 30 0
 EELAYER END
@@
 $EndComp
 $Comp
-L Miz:PWR_DIODE D15
+L CAN_BLDCMD-rescue:PWR_DIODE-Miz D15
 U 1 1 5E571D6A
 P 19475 1625
@@
 Connection ~ 7000 9350
 $Comp
-L Miz:SW_ROTARY_16 U5
+L CAN_BLDCMD-rescue:SW_ROTARY_16-Miz U5
 U 1 1 5EE0DA05
 P 7275 11675
@@
 SIGNAL_W
 $Comp
-L Miz:Si866x ISO1
+L CAN_BLDCMD-rescue:Si866x-Miz ISO1
 U 1 1 5E894867
 P 15425 12425
@@
 	20475 2850 21025 2850
 $Comp
-L Miz:NJM78L00 U11
+L CAN_BLDCMD-rescue:NJM78L00-Miz U11
 U 1 1 5E7609B0
 P 21025 2500
