File: CAN_BLDCMD_type3/CAN_BLDCMD_type3.sch (KiCad schematic (older format))
At the start: 1 part

Commit message: 上げ忘れていた工大祭モータドライバ(前身開発基板)とJetsonNanoの電源基板関係
Parts:
- removed U?: DRV8308, Package_DFN_QFN:Texas_S-PVQFN-N40_EP3.52x2.62mm, symbol Driver_Motor:DRV8308
- added C? (x3): 0.1u, symbol Device:C
- added C?: C, symbol Device:C
- added J?: SWD, symbol Connector_Generic:Conn_01x06
- added J?: HALL_IN, symbol Connector_Generic:Conn_01x06
- added J? (x2): BATT_IN, symbol Connector_Generic:Conn_01x02
- added J?: OUT_U, symbol Connector_Generic:Conn_01x01
- added J?: OUT_V, symbol Connector_Generic:Conn_01x01
- added J?: OUT_W, symbol Connector_Generic:Conn_01x01
- added Q? (x2): MOSFET_N, symbol Miz:MOSFET_N
- added R? (x4): 10k, symbol Device:R
- added R?: 1k, symbol Device:R
- added R?: 330, symbol Device:R
- added R?: R, symbol Device:R
- added TH? (x2): Thermistor, symbol Device:Thermistor
- added U?: DRV8304HRHAT, RHA40_TEX, symbol Miz:DRV8304HRHAT
- added U?: LOGO, symbol Miz:LOGO
- added U?: STM32F405RG, Package_QFP:LQFP-64_10x10mm_P0.5mm, symbol Miz:STM32F405RG
- added U?: SI8900, symbol Miz:SI8900
- added U?: TLP291, Package_SO:SOIC-4_4.55x2.6mm_P1.27mm, symbol Isolator:TLP291
Connections:
- net labels added: +3.3V, +3.3VP, +BATT, BATT_VOLTAGE, DRIVE_TEMP, GND, GNDPWR, IOS_ADC_~RST, OUT_U, REGULATOR_TEMP, SI8900_~RST, USARTx_RX, USARTx_TX
- wire segments 0 -> 33
