File: PowerMD_ver1.1(発熱・電流量がどれくらい変わるか試験)/SteerMD.sch (KiCad schematic (older format))
At the start: 232 parts, among them P1 SWD, P10 OUT_1, P11 ENC_0, P13 ENC_1, P14 I/O_1, P15 OUT_0, P2 MOTOR_COOLING, P3 CAN, P4 CAN, P5 SERIAL, P6 I/O_0, P7 FAN, P8 BATT_IN, P9 BATT_IN, Q1 MOSFET_N, Q2 MOSFET_N, Q3 MOSFET_N, Q4 MOSFET_N, Q5 MOSFET_N, Q6 MOSFET_N, Q7 MOSFET_N, Q8 MOSFET_N, SW1 RST, SW3 SW0, SW4 SW1, U1 MAX3051, U10 ACS758, U11 POWER_ON, U12 SI8274, U13 ACS758, U14 SI8274, U15 AZ1086H, U16 LOGO, U17 AQM0802, U18 LTC2644, U19 ADRESS, U2 BD9G101, U3 STM32F405RG, U4 SI8274, U5 SI8900, U6 ADC_~RST, U7 MCP16331, U8 SI8274, U9 BD33FA1, Y1 8MHz

Commit message: 上げ忘れていた工大祭モータドライバ(前身開発基板)とJetsonNanoの電源基板関係
Parts:
- U18: symbol Miz:LTC2644 -> SteerMD-rescue:LTC2644-Miz
- U7: symbol Miz:MCP16331 -> SteerMD-rescue:MCP16331-Miz
Changed lines of the file:
@@
 EESchema Schematic File Version 4
+LIBS:SteerMD-cache
 EELAYER 30 0
 EELAYER END
@@
 	12450 6225 12450 6125
 $Comp
-L Miz:LTC2644 U18
+L SteerMD-rescue:LTC2644-Miz U18
 U 1 1 5E609A08
 P 11675 3750
@@
 Connection ~ 13975 8900
 $Comp
-L Miz:MCP16331 U7
+L SteerMD-rescue:MCP16331-Miz U7
 U 1 1 5E8009AC
 P 10725 2475
