File: MotorDriver/Brushed-DCMotor-Driver/CAN_Current_Control_MD_ver0/CAN_Current_Control_MD.sch (KiCad schematic (older format))
At the start: 202 parts, among them J1 SWD, J10 FAN, J11 OUT_0, J12 OUT_1, J13 VALVE, J14 SERIAL, J2 CAN, J3 CAN, J4 ENC0, J5 ENC1, J6 I/O_0, J7 I/O_1, J8 BATT_IN, J9 BATT_IN, Q1 MOSFET_N, Q10 NPN, Q2 MOSFET_N, Q3 MOSFET_N, Q4 MOSFET_N, Q5 MOSFET_N, Q6 MOSFET_N, Q7 MOSFET_N, Q8 MOSFET_N, Q9 NPN, SW1 SW0, SW2 SW1, SW3 RST, U1 BD33FA1, U10 NCP5104, U11 NCP5104, U12 BD9G101G, U13 INA181A1, U14 INA181A1, U15 LOGO, U2 ISO1050DUB, U3 STM32F405RG, U4 ADRESS, U5 AZ1086H, U6 BD9G101G, U7 AQM0802, U8 NCP5104, U9 NCP5104, Y1 8MHz

Commit message: test
Parts:
- D23: symbol Miz:PWR_DIODE -> CAN_Current_Control_MD-rescue:PWR_DIODE-Miz
- U10, U11, U8, U9: symbol Miz:NCP5104 -> CAN_Current_Control_MD-rescue:NCP5104-Miz
- U4: symbol Miz:SW_ROTARY_16 -> CAN_Current_Control_MD-rescue:SW_ROTARY_16-Miz-CAN_Current_Control_MD-rescue
Changed lines of the file:
@@
 EESchema Schematic File Version 4
-LIBS:CAN_Current_Control_MD-cache
 EELAYER 30 0
 EELAYER END
@@
 	2375 3175 1875 3175
 $Comp
-L Miz:NCP5104 U8
+L CAN_Current_Control_MD-rescue:NCP5104-Miz U8
 U 1 1 5E530EDC
 P 10925 3350
@@
 $EndComp
 $Comp
-L Miz:NCP5104 U9
+L CAN_Current_Control_MD-rescue:NCP5104-Miz U9
 U 1 1 5E531612
 P 10925 4900
@@
 	13225 5400 13300 5400
 $Comp
-L Miz:NCP5104 U10
+L CAN_Current_Control_MD-rescue:NCP5104-Miz U10
 U 1 1 5E5FCEBA
 P 10925 6775
@@
 $EndComp
 $Comp
-L Miz:NCP5104 U11
+L CAN_Current_Control_MD-rescue:NCP5104-Miz U11
 U 1 1 5E5FCEC4
 P 10925 8325
@@
 $EndComp
 $Comp
-L Miz:PWR_DIODE D23
+L CAN_Current_Control_MD-rescue:PWR_DIODE-Miz D23
 U 1 1 5E561D43
 P 13425 1175
@@
 $EndComp
 $Comp
-L Miz:SW_ROTARY_16 U4
+L CAN_Current_Control_MD-rescue:SW_ROTARY_16-Miz-CAN_Current_Control_MD-rescue U4
 U 1 1 5E781202
 P 4600 10225
