File: other/F407_io_ver2(青基板)/stm32f4_board_test.sch (KiCad schematic (older format))
At the start: 128 parts, among them P1 ENC3, P10 ADC, P11 PWM, P12 I/O, P13 ADC_Vdd, P14 PWM_Vdd, P15 I/O_Vdd, P16 VALVE_Vdd, P17 USART0, P2 ENC0, P3 ENC1, P4 ENC2, P5 USART1, P6 SWD, P7 CAN, P8 CAN, P9 VALVE, SW1 ADDR, SW2 SW0, SW3 SW1, SW6 RESET, U1 STM32F407VG, U2 AP3211, U3 OSTBABS4C2B, U4 AZ1086H, U5 MAX3051, U6 TBD62083A, U7 ADRES, U8 LOGO, U9 LOGO, Y1 Crystal

Commit message: test
Parts:
- U7: symbol Miz:OSL10321-Lx -> stm32f4_board_test-rescue:OSL10321-Lx-Miz-stm32f4_board_test-rescue
Changed lines of the file:
@@
 EESchema Schematic File Version 4
-LIBS:74xgxx
-LIBS:74xx
-LIBS:audio
-LIBS:device
-LIBS:graphic
-LIBS:interface
-LIBS:power
-LIBS:pspice
-LIBS:video
-LIBS:stm32f4_board_test-cache
 EELAYER 30 0
 EELAYER END
@@
 $EndComp
 $Comp
-L Miz:OSL10321-Lx U7
+L stm32f4_board_test-rescue:OSL10321-Lx-Miz-stm32f4_board_test-rescue U7
 U 1 1 5D27C6DC
 P 12575 14600
