File: MotorDriver/Brushed-DCMotor-Driver/CAN_DCMD_Normal_ver0/NormalMD.kicad_pcb (KiCad board)
At the start: 2 copper layers, 75 x 88 mm, 224 parts, among them P1 SWD, P10 OUT_1, P11 ENC_0, P13 ENC_1, P14 I/O_1, P15 OUT_0, P2 VALVE, P3 CAN, P4 CAN, P5 SERIAL, P6 I/O_0, P7 FAN, P8 BATT_IN, P9 BATT_IN, Q1 MOSFET_N, Q10 NPN, Q2 MOSFET_N, Q3 MOSFET_N, Q4 MOSFET_N, Q5 MOSFET_N, Q6 MOSFET_N, Q7 MOSFET_N, Q8 MOSFET_N, Q9 NPN, SW1 RST, SW3 SW0, SW4 SW1, U1 MAX3051, U11 POWER_ON, U12 SI8274, U14 SI8274, U15 AZ1086H, U16 LOGO, U17 AQM0802, U19 ADRESS, U2 BD9G101, U3 STM32F405RG, U4 SI8274, U5 SI8900, U6 ADC_~RST, U7 BD9G101G, U8 SI8274, U9 BD33FA1, Y1 8MHz

Commit message: 今更修正
Other:
- board text added: "CAN DC-MotorDriver Leo Regulus ver.0.1"
- board text removed: "CAN DC-MotroDriver Leo Regulus ver.0.1"
Changed lines of the file:
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@@
     (effects (font (size 0.8 0.8) (thickness 0.15)) (justify mirror))
   )
-  (gr_text "CAN DC-MotroDriver \nLeo Regulus ver.0.1" (at 145.1 91.6 90) (layer F.SilkS)
+  (gr_text "CAN DC-MotorDriver \nLeo Regulus ver.0.1" (at 145.1 91.6 90) (layer F.SilkS)
     (effects (font (size 1.2 1.2) (thickness 0.25) italic) (justify left))
   )
