File: MotorDriver/Brushed-DCMotor-Driver/CAN_DCMD_Normal_ver0/NormalMD.sch (KiCad schematic (older format))
At the start: 224 parts, among them P1 SWD, P10 OUT_1, P11 ENC_0, P13 ENC_1, P14 I/O_1, P15 OUT_0, P2 VALVE, P3 CAN, P4 CAN, P5 SERIAL, P6 I/O_0, P7 FAN, P8 BATT_IN, P9 BATT_IN, Q1 MOSFET_N, Q10 NPN, Q2 MOSFET_N, Q3 MOSFET_N, Q4 MOSFET_N, Q5 MOSFET_N, Q6 MOSFET_N, Q7 MOSFET_N, Q8 MOSFET_N, Q9 NPN, SW1 RST, SW3 SW0, SW4 SW1, U1 MAX3051, U11 POWER_ON, U12 SI8274, U14 SI8274, U15 AZ1086H, U16 LOGO, U17 AQM0802, U19 ADRESS, U2 BD9G101, U3 STM32F405RG, U4 SI8274, U5 SI8900, U6 ADC_~RST, U7 BD9G101G, U8 SI8274, U9 BD33FA1, Y1 8MHz

Commit message: update main circuit:ver.3.1.1
Parts:
- added U?: ACS781, symbol Miz:ACS781
Connections:
- net +3V3: now also U?.1 (VCC)
- net +BATT: now also U?.5 (IP+)
- net GND: now also U?.2 (GND)
- net MOTOR0_BATT: now also U?.6 (IP-)
- new net Current_Value: U?.3 (VOUT)
Changed lines of the file:
@@
 EESchema Schematic File Version 4
-LIBS:NormalMD-cache
 EELAYER 30 0
 EELAYER END
@@
 Text Label 8950 5925 0    50   ~ 0
 VALVE0
+$Comp
+L Miz:ACS781 U?
+U 1 1 6080468A
+P 20425 6250
+F 0 "U?" H 20425 6637 60  0000 C CNN
+F 1 "ACS781" H 20425 6531 60  0000 C CNN
+F 2 "" H 20425 6250 60  0000 C CNN
+F 3 "" H 20425 6250 60  0000 C CNN
+	1    20425 6250
+	1    0    0    -1
+$EndComp
+$Comp
+L NormalMD-rescue:+BATT-power-MD_Enbarr_x2-rescue-F4_CAN_DCMD-rescue-SteerMD-rescue #PWR?
+U 1 1 60804CB5
+P 19975 6150
+F 0 "#PWR?" H 19975 6000 50  0001 C CNN
+F 1 "+BATT" H 19990 6323 50  0000 C CNN
+F 2 "" H 19975 6150 50  0001 C CNN
+F 3 "" H 19975 6150 50  0001 C CNN
+	1    19975 6150
+	1    0    0    -1
+$EndComp
+Text Label 19900 6350 2    50   ~ 0
+MOTOR0_BATT
+Wire Wire Line
+	19900 6350 19975 6350
+Text Label 20975 6150 0    50   ~ 0
+Current_Value
+Wire Wire Line
+	20975 6150 20875 6150
+$Comp
+L power:GND #PWR?
+U 1 1 60878E0B
+P 20975 6500
+F 0 "#PWR?" H 20975 6250 50  0001 C CNN
+F 1 "GND" H 20980 6327 50  0000 C CNN
+F 2 "" H 20975 6500 50  0001 C CNN
+F 3 "" H 20975 6500 50  0001 C CNN
+	1    20975 6500
+	1    0    0    -1
+$EndComp
+Wire Wire Line
+	20975 6500 20975 6250
+Wire Wire Line
+	20975 6250 20875 6250
+$Comp
+L power:+3.3V #PWR?
+U 1 1 608A2689
+P 21075 6350
+F 0 "#PWR?" H 21075 6200 50  0001 C CNN
+F 1 "+3.3V" H 21090 6523 50  0000 C CNN
+F 2 "" H 21075 6350 50  0001 C CNN
+F 3 "" H 21075 6350 50  0001 C CNN
+	1    21075 6350
+	1    0    0    -1
+$EndComp
+Wire Wire Line
+	21075 6350 20875 6350
 $EndSCHEMATC
