File: MotorDriver/Brushed-DCMotor-Driver/PowerMD_ver0/SteerMD.kicad_pcb (KiCad board)
At the start: 2 copper layers, 75 x 88 mm, 216 parts, among them P1 SWD, P10 OUT_1, P11 ENC_0, P13 ENC_1, P14 I/O_1, P15 OUT_0, P2 MOTOR_COOLING, P3 CAN, P4 CAN, P5 SERIAL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

Commit message: 今更修正
Other:
- board text added: "CAN DC-MotorDriver Aqualius Sadalmeric ver.0.0"
- board text removed: "CAN DC-MotroDriver Aqualius Sadalmeric ver.0.0"
