File: Main/stm32f4_Centaurus_ver.3.1/stm32f4_Centaurus.sch (KiCad schematic (older format))
At the start: 230 parts, among them IC1 PIC24FJ64GB004, J1 SERIAL1, J2 EXTERNAL_~RST, P1 PICKit3, P10 XA2_12V, P11 CAN0, P12 CAN1, P13 CAN0, P14 CAN1, P15 SERIAL2, P16 SERIAL0, P17 XA2_5V, P18 SWD, P2 ADVANCED_SBDBT, P23 A/D, P24 PWM, P25 A/D_batt, P26 PWM_batt, P27 EMERGENCY_CHECK, P28 I/O_5V, P29 I/O_Variable, P3 ENC0, P30 I/O_5V_batt, P31 I/O_Variable, P4 ENC2, P5 SPI0, P6 ENC3, P7 ENC1, P8 SERIAL4, P9 SERIAL3, Q1 FET_P, Q2 FET_P, Q3 FET_P, Q4 NPN, Q5 NPN, Q6 FET_P, Q7 FET_N, Q8 FET_P, SW1 Main_POWER, SW2 SW1, SW3 SW0, SW4 SW2, SW5 SW3, U1 STM32F407VG, U10 LOGO, U11 CPC1106N, U12 PS7200K-1A, U13 LOGO, U2 AZ1086H, U3 MCP2221A, U4 BD9G101G, U5 MAX3051, U6 MAX3051, U7 AQM1602_BL, U8 OSTBABS4C2B, U9 LOGO, X1 8MHz

Commit message: 今更修正
Parts:
- added R82, R83: 4.7k, Mizz_lib:R_0603, symbol stm32f4_Centaurus-rescue:R-device
Connections:
- net GND: now also R82.2, R83.2
- net at J1.A5 (CC1): now also R83.1
- net at J1.B5 (CC2): now also R82.1
- no-connect marks 47 -> 45
Changed lines of the file:
@@
 F 3 "" H 4775 3525 60  0000 C CNN
 	1    4775 3525
-	0    1    1    0
+	1    0    0    -1
 $EndComp
 Text Label 4775 3725 2    50   ~ 0
@@
 Wire Wire Line
 	1650 13950 1650 14050
-NoConn ~ 1650 13450
-NoConn ~ 1650 13550
 NoConn ~ 1650 14250
 NoConn ~ 1650 14350
@@
 	19500 2450 19375 2450
 Connection ~ 19375 2450
+Wire Wire Line
+	1650 13550 2000 13550
+Wire Wire Line
+	2100 13450 1650 13450
+Wire Wire Line
+	2100 13450 2100 13800
+Wire Wire Line
+	1050 15850 2000 15850
+Wire Wire Line
+	2100 15850 2100 14100
+Wire Wire Line
+	2000 13850 2000 15850
+Connection ~ 2000 15850
+Wire Wire Line
+	2000 15850 2100 15850
+Connection ~ 1050 15850
+$Comp
+L stm32f4_Centaurus-rescue:R-device R83
+U 1 1 606C3CE8
+P 2100 13950
+F 0 "R83" H 2178 13988 40  0000 L CNN
+F 1 "4.7k" H 2178 13912 40  0000 L CNN
+F 2 "Mizz_lib:R_0603" V 2030 13950 30  0001 C CNN
+F 3 "" H 2100 13950 30  0000 C CNN
+	1    2100 13950
+	1    0    0    -1
+$EndComp
+$Comp
+L stm32f4_Centaurus-rescue:R-device R82
+U 1 1 606C4A2F
+P 2000 13700
+F 0 "R82" H 2078 13738 40  0000 L CNN
+F 1 "4.7k" H 2078 13662 40  0000 L CNN
+F 2 "Mizz_lib:R_0603" V 1930 13700 30  0001 C CNN
+F 3 "" H 2000 13700 30  0000 C CNN
+	1    2000 13700
+	1    0    0    -1
+$EndComp
 $EndSCHEMATC

Commit message: update main circuit:ver.3.1.1
Parts:
- removed R82, R83: 4.7k, Mizz_lib:R_0603, symbol stm32f4_Centaurus-rescue:R-device
Changed lines of the file:
@@
 	19500 2450 19375 2450
 Connection ~ 19375 2450
-Wire Wire Line
-	1650 13550 2000 13550
-Wire Wire Line
-	2100 13450 1650 13450
-Wire Wire Line
-	2100 13450 2100 13800
-Wire Wire Line
-	1050 15850 2000 15850
-Wire Wire Line
-	2100 15850 2100 14100
-Wire Wire Line
-	2000 13850 2000 15850
-Connection ~ 2000 15850
-Wire Wire Line
-	2000 15850 2100 15850
-Connection ~ 1050 15850
-$Comp
-L stm32f4_Centaurus-rescue:R-device R83
-U 1 1 606C3CE8
-P 2100 13950
-F 0 "R83" H 2178 13988 40  0000 L CNN
-F 1 "4.7k" H 2178 13912 40  0000 L CNN
-F 2 "Mizz_lib:R_0603" V 2030 13950 30  0001 C CNN
-F 3 "" H 2100 13950 30  0000 C CNN
-	1    2100 13950
-	1    0    0    -1
-$EndComp
-$Comp
-L stm32f4_Centaurus-rescue:R-device R82
-U 1 1 606C4A2F
-P 2000 13700
-F 0 "R82" H 2078 13738 40  0000 L CNN
-F 1 "4.7k" H 2078 13662 40  0000 L CNN
-F 2 "Mizz_lib:R_0603" V 1930 13700 30  0001 C CNN
-F 3 "" H 2000 13700 30  0000 C CNN
-	1    2000 13700
-	1    0    0    -1
-$EndComp
 $EndSCHEMATC
