File: MotorDriver/Brushless-DCMotor-Driver/CAN_BLDCMD_type0/CAN_BLDCMD.sch (KiCad schematic (older format))
At the start: 215 parts, among them J1 SWD, J10 BATT_IN, J11 OUT_U, J12 OUT_V, J13 OUT_W, J14 VALVE, J15 HALL_IN, J2 CAN, J3 CAN, J4 ENC, J5 I/O0, J6 I/O1, J7 SERIAL, J8 FAN, J9 BATT_IN, Q1 MOSFET_N, Q2 MOSFET_N, Q3 MOSFET_N, Q4 MOSFET_N, Q5 MOSFET_N, Q6 MOSFET_N, Q7 NPN, Q8 NPN, SW1 SW0, SW2 SW1, SW3 RST, SW4 MODE, U1 MAX3051, U10 SI8900, U11 ADC_~RST, U12 ACS758, U13 ACS758, U14 ACS758, U15 BD9G101G, U16 LTC2644, U17 LTC2644, U18 BD33FA1, U19 LOGO, U2 BD9G101G, U20 AQM0802, U3 STM32F405RG, U4 AZ1086H, U5 ADRESS, U6 POWER_ON, U7 SI8274, U8 SI8274, U9 SI8274, Y1 8MHz

Commit message: update main circuit:ver.3.1.1
Parts:
- D15: symbol Miz:PWR_DIODE -> CAN_BLDCMD-rescue:PWR_DIODE-Miz
- U16, U17: symbol Miz:LTC2644 -> CAN_BLDCMD-rescue:LTC2644-Miz
- U7, U8, U9: symbol Miz:SI8274 -> CAN_BLDCMD-rescue:SI8274-Miz
Changed lines of the file:
@@
 Connection ~ 8525 6300
 $Comp
-L Miz:SI8274 U8
+L CAN_BLDCMD-rescue:SI8274-Miz U8
 U 1 1 5E4619A5
 P 15425 7375
@@
 $EndComp
 $Comp
-L Miz:PWR_DIODE D15
+L CAN_BLDCMD-rescue:PWR_DIODE-Miz D15
 U 1 1 5E571D6A
 P 19475 1625
@@
 Connection ~ 21500 2400
 $Comp
-L Miz:SI8274 U9
+L CAN_BLDCMD-rescue:SI8274-Miz U9
 U 1 1 5E6F3747
 P 15425 9600
@@
 	15725 10700 15625 10700
 $Comp
-L Miz:SI8274 U7
+L CAN_BLDCMD-rescue:SI8274-Miz U7
 U 1 1 5E7159FA
 P 15425 5150
@@
 $EndComp
 $Comp
-L Miz:LTC2644 U16
+L CAN_BLDCMD-rescue:LTC2644-Miz U16
 U 1 1 5EE0F6FD
 P 20125 6125
@@
 OUT_V_Analog
 $Comp
-L Miz:LTC2644 U17
+L CAN_BLDCMD-rescue:LTC2644-Miz U17
 U 1 1 5EF10A58
 P 20125 8075
