File: MotorDriver/Brushless-DCMotor-Driver/CAN_BLDCMD_type2/ver.0.1/CAN_BLDCMD.sch (KiCad schematic (older format))
At the start: 203 parts, among them J1 SWD, J10 BATT_IN, J11 OUT_U, J12 OUT_V, J13 OUT_W, J14 VALVE, J15 HALL_IN, J2 CAN, J3 CAN, J4 ENC, J5 I/O0, J6 I/O1, J7 SERIAL, J8 FAN, J9 BATT_IN, Q1 MOSFET_N, Q2 MOSFET_N, Q3 MOSFET_N, Q4 MOSFET_N, Q5 MOSFET_N, Q6 MOSFET_N, Q7 NPN, Q8 NPN, SW1 SW0, SW2 SW1, SW3 RST, SW4 MODE, U1 MAX3051, U10 LM339, U11 NJM78L05, U12 ACS758, U15 BD9G101G, U19 LOGO, U2 BD9G101G, U20 AQM0802, U3 STM32F405RG, U4 AZ1086H, U5 ADRESS, U6 POWER_ON, U7 SI8274, U8 SI8274, U9 SI8274, Y1 8MHz

Commit message: 推奨のほうにファイルを追加しました
Parts:
- D1, D10, D11, D12, D13, D14, D16, D17, D18, D2, D3, D4, D7, D8, D9: symbol Miz:DIODE_rev -> CAN_BLDCMD-rescue:DIODE_rev-Miz
- Q1, Q2, Q3, Q4, Q5, Q6: symbol Miz:MOSFET_N -> CAN_BLDCMD-rescue:MOSFET_N-Miz
- U12: symbol Miz:ACS758 -> CAN_BLDCMD-rescue:ACS758-Miz
- U15, U2: symbol Miz:BD9G101G -> CAN_BLDCMD-rescue:BD9G101G-Miz
- U19: symbol Miz:LOGO -> CAN_BLDCMD-rescue:LOGO-Miz
- U20: symbol Miz:AQM1602 -> CAN_BLDCMD-rescue:AQM1602-Miz
- U3: symbol Miz:STM32F405RG -> CAN_BLDCMD-rescue:STM32F405RG-Miz
- U4: symbol Miz:AZ1086H -> CAN_BLDCMD-rescue:AZ1086H-Miz
- U7, U8, U9: symbol Miz:SI8274 -> CAN_BLDCMD-rescue:SI8274-Miz
Changed lines of the file:
@@
 EESchema Schematic File Version 4
-LIBS:CAN_BLDCMD-cache
 EELAYER 30 0
 EELAYER END
@@
 $EndDescr
 $Comp
-L Miz:STM32F405RG U3
+L CAN_BLDCMD-rescue:STM32F405RG-Miz U3
 U 1 1 5E429697
 P 4425 5675
@@
 $EndComp
 $Comp
-L Miz:DIODE_rev D1
+L CAN_BLDCMD-rescue:DIODE_rev-Miz D1
 U 1 1 5E4321DC
 P 1575 3525
@@
 Connection ~ 8525 6300
 $Comp
-L Miz:SI8274 U8
+L CAN_BLDCMD-rescue:SI8274-Miz U8
 U 1 1 5E4619A5
 P 15425 7375
@@
 $EndComp
 $Comp
-L Miz:MOSFET_N Q3
+L CAN_BLDCMD-rescue:MOSFET_N-Miz Q3
 U 1 1 5E46258F
 P 16975 6975
@@
 $EndComp
 $Comp
-L Miz:DIODE_rev D10
+L CAN_BLDCMD-rescue:DIODE_rev-Miz D10
 U 1 1 5E464365
 P 16325 6825
@@
 $EndComp
 $Comp
-L Miz:DIODE_rev D11
+L CAN_BLDCMD-rescue:DIODE_rev-Miz D11
 U 1 1 5E466FB2
 P 16325 7575
@@
 $EndComp
 $Comp
-L Miz:MOSFET_N Q4
+L CAN_BLDCMD-rescue:MOSFET_N-Miz Q4
 U 1 1 5E468D66
 P 16975 7725
@@
 Connection ~ 16025 7875
 $Comp
-L Miz:BD9G101G U2
+L CAN_BLDCMD-rescue:BD9G101G-Miz U2
 U 1 1 5E4B1A3D
 P 3250 1550
@@
 $EndComp
 $Comp
-L Miz:DIODE_rev D2
+L CAN_BLDCMD-rescue:DIODE_rev-Miz D2
 U 1 1 5E4B3163
 P 3875 1025
@@
 $EndComp
 $Comp
-L Miz:DIODE_rev D3
+L CAN_BLDCMD-rescue:DIODE_rev-Miz D3
 U 1 1 5E4B3C8D
 P 4350 1550
@@
 FB_5V
 $Comp
-L Miz:DIODE_rev D4
+L CAN_BLDCMD-rescue:DIODE_rev-Miz D4
 U 1 1 5E4CB219
 P 4875 1450
@@
 $EndComp
 $Comp
-L Miz:AZ1086H U4
+L CAN_BLDCMD-rescue:AZ1086H-Miz U4
 U 1 1 5E4D541D
 P 5575 1600
@@
 $EndComp
 $Comp
-L Miz:LOGO_Monster #G1
+L CAN_BLDCMD-rescue:LOGO_Monster-Miz #G1
 U 1 1 5E54EFF7
 P 22000 1475
@@
 $EndComp
 $Comp
-L Miz:LOGO U19
+L CAN_BLDCMD-rescue:LOGO-Miz U19
 U 1 1 5E54F6C7
 P 22025 2375
@@
 	19225 1625 19275 1625
 $Comp
-L Miz:BD9G101G U15
+L CAN_BLDCMD-rescue:BD9G101G-Miz U15
 U 1 1 5E57EC0F
 P 18350 2500
@@
 FB_12P
 $Comp
-L Miz:DIODE_rev D14
+L CAN_BLDCMD-rescue:DIODE_rev-Miz D14
 U 1 1 5E5F28D7
 P 18950 1975
@@
 $EndComp
 $Comp
-L Miz:DIODE_rev D16
+L CAN_BLDCMD-rescue:DIODE_rev-Miz D16
 U 1 1 5E5FCAD7
 P 19875 2400
@@
 Connection ~ 21500 2850
 $Comp
-L Miz:SI8274 U9
+L CAN_BLDCMD-rescue:SI8274-Miz U9
 U 1 1 5E6F3747
 P 15425 9600
@@
 $EndComp
 $Comp
-L Miz:MOSFET_N Q5
+L CAN_BLDCMD-rescue:MOSFET_N-Miz Q5
 U 1 1 5E6F374D
 P 16975 9200
@@
 $EndComp
 $Comp
-L Miz:DIODE_rev D12
+L CAN_BLDCMD-rescue:DIODE_rev-Miz D12
 U 1 1 5E6F375F
 P 16325 9050
@@
 $EndComp
 $Comp
-L Miz:DIODE_rev D13
+L CAN_BLDCMD-rescue:DIODE_rev-Miz D13
 U 1 1 5E6F377D
 P 16325 9800
@@
 $EndComp
 $Comp
-L Miz:MOSFET_N Q6
+L CAN_BLDCMD-rescue:MOSFET_N-Miz Q6
 U 1 1 5E6F3783
 P 16975 9950
@@
 Connection ~ 16025 10100
 $Comp
-L Miz:SI8274 U7
+L CAN_BLDCMD-rescue:SI8274-Miz U7
 U 1 1 5E7159FA
 P 15425 5150
@@
 $EndComp
 $Comp
-L Miz:MOSFET_N Q1
+L CAN_BLDCMD-rescue:MOSFET_N-Miz Q1
 U 1 1 5E715A00
 P 16975 4750
@@
 $EndComp
 $Comp
-L Miz:DIODE_rev D8
+L CAN_BLDCMD-rescue:DIODE_rev-Miz D8
 U 1 1 5E715A12
 P 16325 4600
@@
 $EndComp
 $Comp
-L Miz:DIODE_rev D9
+L CAN_BLDCMD-rescue:DIODE_rev-Miz D9
 U 1 1 5E715A30
 P 16325 5350
@@
 $EndComp
 $Comp
-L Miz:MOSFET_N Q2
+L CAN_BLDCMD-rescue:MOSFET_N-Miz Q2
 U 1 1 5E715A36
 P 16975 5500
@@
 Connection ~ 16025 5650
 $Comp
-L Miz:ACS758 U12
+L CAN_BLDCMD-rescue:ACS758-Miz U12
 U 1 1 5E715A9B
 P 18475 11125
@@
 	7000 9675 7000 10100
 $Comp
-L Miz:DIODE_rev D7
+L CAN_BLDCMD-rescue:DIODE_rev-Miz D7
 U 1 1 5ED809AE
 P 6800 9350
@@
 $EndComp
 $Comp
-L Miz:AQM1602 U20
+L CAN_BLDCMD-rescue:AQM1602-Miz U20
 U 1 1 5E68D963
 P 10675 10875
@@
 $EndComp
 $Comp
-L Miz:DIODE_rev D17
+L CAN_BLDCMD-rescue:DIODE_rev-Miz D17
 U 1 1 5E664802
 P 4900 10650
@@
 $EndComp
 $Comp
-L Miz:DIODE_rev D18
+L CAN_BLDCMD-rescue:DIODE_rev-Miz D18
 U 1 1 5E6D5E1A
 P 5850 10850

Commit message: update main circuit:ver.3.1.1
Connections:
- no-connect marks 19 -> 21
Changed lines of the file:
@@
 	1    0    0    -1
 $EndComp
+NoConn ~ 6625 6975
+NoConn ~ 6625 7075
 $EndSCHEMATC
